File: supply.sch (KiCad schematic (older format))
At the start: 66 parts

Commit message: - final schematic
Parts:
- gave numbers to parts that had none: 66

Commit message: - init PCB - fix last things in schematic
Parts:
- added C199: 10u, Capacitor_SMD:C_0805_2012Metric_Pad1.15x1.40mm_HandSolder, symbol Device:C_Small
- added C200: 470u, Capacitor_THT:CP_Radial_D10.0mm_P2.50mm_P5.00mm, symbol Device:CP1_Small
- C86: footprint (none) -> Capacitor_THT:CP_Radial_D10.0mm_P2.50mm_P5.00mm
- U19: footprint (none) -> Package_SO:SOIC-8-1EP_3.9x4.9mm_P1.27mm_EP2.41x3.3mm_ThermalVias
Connections:
- net +12V: now also C199.1, C200.1
- net GND: now also C199.2, C200.2
Other:
- moved on the sheet: C86
Changed lines of the file:
@@
 L Device:CP1_Small C86
 U 1 1 5F63923B
-P 5750 3000
-F 0 "C86" H 5841 3046 50  0000 L CNN
-F 1 "470u" H 5841 2955 50  0000 L CNN
-F 2 "" H 5750 3000 50  0001 C CNN
-F 3 "~" H 5750 3000 50  0001 C CNN
-	1    5750 3000
+P 6150 3000
+F 0 "C86" H 6241 3046 50  0000 L CNN
+F 1 "470u" H 6241 2955 50  0000 L CNN
+F 2 "Capacitor_THT:CP_Radial_D10.0mm_P2.50mm_P5.00mm" H 6150 3000 50  0001 C CNN
+F 3 "~" H 6150 3000 50  0001 C CNN
+	1    6150 3000
 	1    0    0    -1
 $EndComp
@@
 	4350 3450 4350 3400
 Wire Wire Line
-	5750 2800 5750 2900
+	6150 2800 6150 2900
 Connection ~ 4350 2800
 $Comp
 L power:GND #PWR?
 U 1 1 5F63CE0F
-P 5750 3100
+P 6150 3100
 AR Path="/5F40DCB9/5F63CE0F" Ref="#PWR?"  Part="1"
 AR Path="/5F618AB9/5F63CE0F" Ref="#PWR?"  Part="1"
 AR Path="/5F63CE0F" Ref="#PWR?"  Part="1"
 AR Path="/5F620813/5F63CE0F" Ref="#PWR090"  Part="1"
-F 0 "#PWR090" H 5750 2940 50  0001 C CNN
-F 1 "GND" H 5750 3000 39  0000 C TNN
-F 2 "" H 5750 3100 50  0001 C CNN
-F 3 "" H 5750 3100 50  0001 C CNN
-	1    5750 3100
+F 0 "#PWR090" H 6150 2940 50  0001 C CNN
+F 1 "GND" H 6150 3000 39  0000 C TNN
+F 2 "" H 6150 3100 50  0001 C CNN
+F 3 "" H 6150 3100 50  0001 C CNN
+	1    6150 3100
 	1    0    0    -1
 $EndComp
@@
 L power:+12V #PWR?
 U 1 1 5F6422F0
-P 5750 2750
+P 6150 2750
 AR Path="/5F61C123/5F6422F0" Ref="#PWR?"  Part="1"
 AR Path="/5F620813/5F6422F0" Ref="#PWR082"  Part="1"
-F 0 "#PWR082" H 5750 2600 50  0001 C CNN
-F 1 "+12V" H 5750 2866 39  0000 C CNN
-F 2 "" H 5750 2750 50  0001 C CNN
-F 3 "" H 5750 2750 50  0001 C CNN
-	1    5750 2750
+F 0 "#PWR082" H 6150 2600 50  0001 C CNN
+F 1 "+12V" H 6150 2866 39  0000 C CNN
+F 2 "" H 6150 2750 50  0001 C CNN
+F 3 "" H 6150 2750 50  0001 C CNN
+	1    6150 2750
 	1    0    0    -1
 $EndComp
@@
 	1    0    0    -1
 $EndComp
-Connection ~ 5750 2800
+Connection ~ 6150 2800
 Wire Wire Line
 	4250 2800 4350 2800
@@
 Wire Wire Line
 	5100 2800 5450 2800
-Connection ~ 5450 2800
-Wire Wire Line
-	5450 2800 5750 2800
 Wire Wire Line
 	5200 4150 5300 4150
@@
 	8500 4550 8150 4550
 Wire Wire Line
-	5750 2750 5750 2800
+	6150 2750 6150 2800
 $Comp
 L power:GND #PWR?
@@
 F 0 "U19" H 3150 3800 50  0000 C CNN
 F 1 "PAM242x" H 3550 3800 50  0000 C CNN
-F 2 "" H 3400 3850 50  0001 C CNN
+F 2 "Package_SO:SOIC-8-1EP_3.9x4.9mm_P1.27mm_EP2.41x3.3mm_ThermalVias" H 3400 3850 50  0001 C CNN
 F 3 "" H 3400 3850 50  0001 C CNN
 	1    3400 3350
@@
 	0    1    1    0
 $EndComp
+$Comp
+L power:PWR_FLAG #FLG?
+U 1 1 5FA293B2
+P 2100 5900
+AR Path="/5F61C123/5FA293B2" Ref="#FLG?"  Part="1"
+AR Path="/5F620813/5FA293B2" Ref="#FLG0104"  Part="1"
+F 0 "#FLG0104" H 2100 5975 50  0001 C CNN
+F 1 "PWR_FLAG" H 2100 6074 50  0001 C CNN
+F 2 "" H 2100 5900 50  0001 C CNN
+F 3 "~" H 2100 5900 50  0001 C CNN
+	1    2100 5900
+	-1   0    0    1
+$EndComp
+$Comp
+L power:PWR_FLAG #FLG?
+U 1 1 5FA2FCE7
+P 6150 4550
+AR Path="/5F61C123/5FA2FCE7" Ref="#FLG?"  Part="1"
+AR Path="/5F620813/5FA2FCE7" Ref="#FLG0105"  Part="1"
+F 0 "#FLG0105" H 6150 4625 50  0001 C CNN
+F 1 "PWR_FLAG" H 6150 4724 50  0001 C CNN
+F 2 "" H 6150 4550 50  0001 C CNN
+F 3 "~" H 6150 4550 50  0001 C CNN
+	1    6150 4550
+	-1   0    0    1
+$EndComp
+$Comp
+L power:PWR_FLAG #FLG?
+U 1 1 5FA643D4
+P 4800 1350
+AR Path="/5F61C123/5FA643D4" Ref="#FLG?"  Part="1"
+AR Path="/5F620813/5FA643D4" Ref="#FLG0108"  Part="1"
+F 0 "#FLG0108" H 4800 1425 50  0001 C CNN
+F 1 "PWR_FLAG" H 4800 1524 50  0001 C CNN
+F 2 "" H 4800 1350 50  0001 C CNN
+F 3 "~" H 4800 1350 50  0001 C CNN
+	1    4800 1350
+	1    0    0    -1
+$EndComp
+$Comp
+L Device:C_Small C199
+U 1 1 5FB0C8D5
+P 5800 3000
+AR Path="/5F620813/5FB0C8D5" Ref="C199"  Part="1"
+AR Path="/5F7A93EE/5FB0C8D5" Ref="C?"  Part="1"
+F 0 "C199" H 5850 3050 50  0000 L BNN
+F 1 "10u" H 5850 2950 50  0000 L TNN
+F 2 "Capacitor_SMD:C_0805_2012Metric_Pad1.15x1.40mm_HandSolder" H 5800 3000 50  0001 C CNN
+F 3 "~" H 5800 3000 50  0001 C CNN
+	1    5800 3000
+	1    0    0    -1
+$EndComp
+Wire Wire Line
+	5800 2800 5800 2900
+$Comp
+L power:GND #PWR?
+U 1 1 5FB0C8DD
+P 5800 3100
+AR Path="/5F40DCB9/5FB0C8DD" Ref="#PWR?"  Part="1"
+AR Path="/5F618AB9/5FB0C8DD" Ref="#PWR?"  Part="1"
+AR Path="/5FB0C8DD" Ref="#PWR?"  Part="1"
+AR Path="/5F620813/5FB0C8DD" Ref="#PWR0248"  Part="1"
+F 0 "#PWR0248" H 5800 2940 50  0001 C CNN
+F 1 "GND" H 5800 3000 39  0000 C TNN
+F 2 "" H 5800 3100 50  0001 C CNN
+F 3 "" H 5800 3100 50  0001 C CNN
+	1    5800 3100
+	1    0    0    -1
+$EndComp
+Wire Wire Line
+	5450 2800 5800 2800
+Connection ~ 5450 2800
+Connection ~ 5800 2800
+Wire Wire Line
+	5800 2800 6150 2800
+$Comp
+L Device:CP1_Small C200
+U 1 1 5FB33D03
+P 6500 3000
+F 0 "C200" H 6591 3046 50  0000 L CNN
+F 1 "470u" H 6591 2955 50  0000 L CNN
+F 2 "Capacitor_THT:CP_Radial_D10.0mm_P2.50mm_P5.00mm" H 6500 3000 50  0001 C CNN
+F 3 "~" H 6500 3000 50  0001 C CNN
+	1    6500 3000
+	1    0    0    -1
+$EndComp
+Wire Wire Line
+	6500 2800 6500 2900
+$Comp
+L power:GND #PWR?
+U 1 1 5FB33D0B
+P 6500 3100
+AR Path="/5F40DCB9/5FB33D0B" Ref="#PWR?"  Part="1"
+AR Path="/5F618AB9/5FB33D0B" Ref="#PWR?"  Part="1"
+AR Path="/5FB33D0B" Ref="#PWR?"  Part="1"
+AR Path="/5F620813/5FB33D0B" Ref="#PWR0249"  Part="1"
+F 0 "#PWR0249" H 6500 2940 50  0001 C CNN
+F 1 "GND" H 6500 3000 39  0000 C TNN
+F 2 "" H 6500 3100 50  0001 C CNN
+F 3 "" H 6500 3100 50  0001 C CNN
+	1    6500 3100
+	1    0    0    -1
+$EndComp
+Wire Wire Line
+	6500 2800 6150 2800
 $EndSCHEMATC

Commit message: - PCB progress
Parts:
- removed C83: 100n, Capacitor_SMD:C_0603_1608Metric_Pad1.05x0.95mm_HandSolder, symbol Device:C_Small
- removed C96: 1u, Capacitor_SMD:C_0805_2012Metric_Pad1.15x1.40mm_HandSolder, symbol Device:C_Small
- removed D13, D15: PMEG4005EJ, miscellaneous_my:D_SOD-323-523_HandSoldering, symbol Diode:PMEG4005EJ
- removed R109: 1R, Resistor_SMD:R_0603_1608Metric_Pad1.05x0.95mm_HandSolder, symbol Device:R_Small
- C100, C101, C107, C199, C98, C99: footprint Capacitor_SMD:C_0805_2012Metric_Pad1.15x1.40mm_HandSolder -> Capacitor_SMD:C_0603_1608Metric_Pad1.05x0.95mm_HandSolder
- C102, C103, C104, C105, C106, C108, C109, C74, C76, C78, C81, C82, C84, C87, C88, C89, C90, C93, C94: footprint Capacitor_SMD:C_0603_1608Metric_Pad1.05x0.95mm_HandSolder -> Capacitor_SMD:C_0603_1608Metric
- C75, C77, C85, C95: footprint Capacitor_SMD:C_0805_2012Metric_Pad1.15x1.40mm_HandSolder -> Capacitor_SMD:C_0805_2012Metric
- C91, C97: footprint Capacitor_SMD:C_0805_2012Metric_Pad1.15x1.40mm_HandSolder -> Capacitor_SMD:C_0603_1608Metric
- R100, R101, R102, R103, R104, R105, R106, R107, R108: footprint Resistor_SMD:R_0603_1608Metric_Pad1.05x0.95mm_HandSolder -> Resistor_SMD:R_0603_1608Metric
Other:
- moved on the sheet: C199, C200, C84, C85, C86

Commit message: - PCB WiP - Pump output aligned
Parts:
- R102, R107: footprint Resistor_SMD:R_0603_1608Metric -> Resistor_SMD:R_0603_1608Metric_Pad1.05x0.95mm_HandSolder
Changed lines of the file:
@@
 F 0 "R107" V 5000 4150 50  0000 C BNN
 F 1 "1R" V 4800 4150 50  0000 C TNN
-F 2 "Resistor_SMD:R_0603_1608Metric" V 4830 4150 50  0001 C CNN
+F 2 "Resistor_SMD:R_0603_1608Metric_Pad1.05x0.95mm_HandSolder" V 4830 4150 50  0001 C CNN
 F 3 "~" H 4900 4150 50  0001 C CNN
 	1    4900 4150
@@
 F 0 "R102" V 4050 2050 50  0000 C BNN
 F 1 "1R" V 3850 2050 50  0000 C TNN
-F 2 "Resistor_SMD:R_0603_1608Metric" V 3880 2050 50  0001 C CNN
+F 2 "Resistor_SMD:R_0603_1608Metric_Pad1.05x0.95mm_HandSolder" V 3880 2050 50  0001 C CNN
 F 3 "~" H 3950 2050 50  0001 C CNN
 	1    3950 2050

Commit message: - PCB WiP
Parts:
- C200, C86: footprint Capacitor_THT:CP_Radial_D10.0mm_P2.50mm_P5.00mm -> Capacitor_THT:CP_Radial_D8.0mm_P3.50mm
- D12, D14, D5, D6: footprint Diode_SMD:D_SOD-323_HandSoldering -> miscellaneous_my:D_SOD-323-523_HandSoldering
Changed lines of the file:
@@
 $Descr A4 11693 8268
 encoding utf-8
-Sheet 6 11
+Sheet 6 10
 Title ""
 Date ""
@@
 F 0 "C86" H 5891 3046 50  0000 L CNN
 F 1 "470u" H 5891 2955 50  0000 L CNN
-F 2 "Capacitor_THT:CP_Radial_D10.0mm_P2.50mm_P5.00mm" H 5800 3000 50  0001 C CNN
+F 2 "Capacitor_THT:CP_Radial_D8.0mm_P3.50mm" H 5800 3000 50  0001 C CNN
 F 3 "~" H 5800 3000 50  0001 C CNN
 	1    5800 3000
@@
 F 0 "D5" H 5550 1150 50  0000 C BNN
 F 1 "1N4448" H 5550 1100 50  0000 C CNN
-F 2 "Diode_SMD:D_SOD-323_HandSoldering" V 5550 1000 50  0001 C CNN
+F 2 "miscellaneous_my:D_SOD-323-523_HandSoldering" V 5550 1000 50  0001 C CNN
 F 3 "~" V 5550 1000 50  0001 C CNN
 	1    5550 1000
@@
 F 0 "D14" H 6900 5050 50  0000 C BNN
 F 1 "1N4448" H 6900 5000 50  0000 C CNN
-F 2 "Diode_SMD:D_SOD-323_HandSoldering" V 6900 4900 50  0001 C CNN
+F 2 "miscellaneous_my:D_SOD-323-523_HandSoldering" V 6900 4900 50  0001 C CNN
 F 3 "~" V 6900 4900 50  0001 C CNN
 	1    6900 4900
@@
 F 0 "D12" V 7254 4470 50  0000 L CNN
 F 1 "1N4448" H 7300 4300 50  0000 C CNN
-F 2 "Diode_SMD:D_SOD-323_HandSoldering" V 7300 4400 50  0001 C CNN
+F 2 "miscellaneous_my:D_SOD-323-523_HandSoldering" V 7300 4400 50  0001 C CNN
 F 3 "~" V 7300 4400 50  0001 C CNN
 	1    7300 4400
@@
 F 0 "D6" V 5900 1550 50  0000 L BNN
 F 1 "1N4448" H 5950 1400 50  0000 C CNN
-F 2 "Diode_SMD:D_SOD-323_HandSoldering" V 5950 1500 50  0001 C CNN
+F 2 "miscellaneous_my:D_SOD-323-523_HandSoldering" V 5950 1500 50  0001 C CNN
 F 3 "~" V 5950 1500 50  0001 C CNN
 	1    5950 1500
@@
 F 0 "C200" H 6241 3046 50  0000 L CNN
 F 1 "470u" H 6241 2955 50  0000 L CNN
-F 2 "Capacitor_THT:CP_Radial_D10.0mm_P2.50mm_P5.00mm" H 6150 3000 50  0001 C CNN
+F 2 "Capacitor_THT:CP_Radial_D8.0mm_P3.50mm" H 6150 3000 50  0001 C CNN
 F 3 "~" H 6150 3000 50  0001 C CNN
 	1    6150 3000

Commit message: - PCB WiP
Parts:
- removed C108: 1u, Capacitor_SMD:C_0603_1608Metric, symbol Device:C_Small
- added C7: 100n, Capacitor_SMD:C_0603_1608Metric, symbol Device:C_Small
Connections:
- net +BATT: now also C7.1
- net GND: now also C7.2
Other:
- moved on the sheet: C109
Changed lines of the file:
@@
 $Descr A4 11693 8268
 encoding utf-8
-Sheet 6 10
+Sheet 5 10
 Title ""
 Date ""
@@
 	1    0    0    -1
 $EndComp
-Wire Wire Line
-	6550 5900 6550 6000
-$Comp
-L power:GND #PWR?
-U 1 1 5FB9CB46
+$Comp
+L power:GND #PWR?
+U 1 1 5FB9CB4C
 P 6550 6200
-AR Path="/5F40DCB9/5FB9CB46" Ref="#PWR?"  Part="1"
-AR Path="/5F618AB9/5FB9CB46" Ref="#PWR?"  Part="1"
-AR Path="/5FB9CB46" Ref="#PWR?"  Part="1"
-AR Path="/5F620813/5FB9CB46" Ref="#PWR0116"  Part="1"
-F 0 "#PWR0116" H 6550 6040 50  0001 C CNN
+AR Path="/5F40DCB9/5FB9CB4C" Ref="#PWR?"  Part="1"
+AR Path="/5F618AB9/5FB9CB4C" Ref="#PWR?"  Part="1"
+AR Path="/5FB9CB4C" Ref="#PWR?"  Part="1"
+AR Path="/5F620813/5FB9CB4C" Ref="#PWR0117"  Part="1"
+F 0 "#PWR0117" H 6550 6040 50  0001 C CNN
 F 1 "GND" H 6550 6100 39  0000 C TNN
 F 2 "" H 6550 6200 50  0001 C CNN
@@
 	1    0    0    -1
 $EndComp
-$Comp
-L power:GND #PWR?
-U 1 1 5FB9CB4C
-P 6850 6200
-AR Path="/5F40DCB9/5FB9CB4C" Ref="#PWR?"  Part="1"
-AR Path="/5F618AB9/5FB9CB4C" Ref="#PWR?"  Part="1"
-AR Path="/5FB9CB4C" Ref="#PWR?"  Part="1"
-AR Path="/5F620813/5FB9CB4C" Ref="#PWR0117"  Part="1"
-F 0 "#PWR0117" H 6850 6040 50  0001 C CNN
-F 1 "GND" H 6850 6100 39  0000 C TNN
-F 2 "" H 6850 6200 50  0001 C CNN
-F 3 "" H 6850 6200 50  0001 C CNN
-	1    6850 6200
-	1    0    0    -1
-$EndComp
-Wire Wire Line
-	6850 6000 6850 5900
+Wire Wire Line
+	6550 6000 6550 5900
 $Comp
 L Device:C_Small C109
 U 1 1 5FB9CB53
-P 6850 6100
-F 0 "C109" H 6900 6150 50  0000 L BNN
-F 1 "100n" H 6900 6050 50  0000 L TNN
-F 2 "Capacitor_SMD:C_0603_1608Metric" H 6850 6100 50  0001 C CNN
-F 3 "~" H 6850 6100 50  0001 C CNN
-	1    6850 6100
-	1    0    0    -1
-$EndComp
-$Comp
-L Device:C_Small C108
-U 1 1 5FB9CB5A
 P 6550 6100
-F 0 "C108" H 6600 6150 50  0000 L BNN
-F 1 "1u" H 6600 6050 50  0000 L TNN
+F 0 "C109" H 6600 6150 50  0000 L BNN
+F 1 "100n" H 6600 6050 50  0000 L TNN
 F 2 "Capacitor_SMD:C_0603_1608Metric" H 6550 6100 50  0001 C CNN
 F 3 "~" H 6550 6100 50  0001 C CNN
@@
 	5950 5900 6250 5900
 Connection ~ 6250 5900
-Wire Wire Line
-	6250 5900 6550 5900
-Connection ~ 6550 5900
-Wire Wire Line
-	6550 5900 6850 5900
 $Comp
 L power:+3V3 #PWR0105
 U 1 1 5FBA87C8
-P 6850 5850
-F 0 "#PWR0105" H 6850 5700 50  0001 C CNN
-F 1 "+3V3" H 6865 6023 50  0000 C CNN
-F 2 "" H 6850 5850 50  0001 C CNN
-F 3 "" H 6850 5850 50  0001 C CNN
-	1    6850 5850
-	1    0    0    -1
-$EndComp
-Wire Wire Line
-	6850 5900 6850 5850
-Connection ~ 6850 5900
+P 6550 5850
+F 0 "#PWR0105" H 6550 5700 50  0001 C CNN
+F 1 "+3V3" H 6565 6023 50  0000 C CNN
+F 2 "" H 6550 5850 50  0001 C CNN
+F 3 "" H 6550 5850 50  0001 C CNN
+	1    6550 5850
+	1    0    0    -1
+$EndComp
+Wire Wire Line
+	6550 5900 6550 5850
 $Comp
 L power:+BATT #PWR081
@@
 Wire Wire Line
 	4750 2800 5100 2800
+Wire Wire Line
+	6250 5900 6550 5900
+Connection ~ 6550 5900
+$Comp
+L power:GND #PWR?
+U 1 1 5FB9822C
+P 1300 6200
+AR Path="/5F40DCB9/5FB9822C" Ref="#PWR?"  Part="1"
+AR Path="/5F618AB9/5FB9822C" Ref="#PWR?"  Part="1"
+AR Path="/5FB9822C" Ref="#PWR?"  Part="1"
+AR Path="/5F620813/5FB9822C" Ref="#PWR0116"  Part="1"
+F 0 "#PWR0116" H 1300 6040 50  0001 C CNN
+F 1 "GND" H 1300 6100 39  0000 C TNN
+F 2 "" H 1300 6200 50  0001 C CNN
+F 3 "" H 1300 6200 50  0001 C CNN
+	1    1300 6200
+	1    0    0    -1
+$EndComp
+$Comp
+L Device:C_Small C7
+U 1 1 5FB98233
+P 1300 6100
+F 0 "C7" H 1350 6150 50  0000 L BNN
+F 1 "100n" H 1350 6050 50  0000 L TNN
+F 2 "Capacitor_SMD:C_0603_1608Metric" H 1300 6100 50  0001 C CNN
+F 3 "~" H 1300 6100 50  0001 C CNN
+	1    1300 6100
+	1    0    0    -1
+$EndComp
+Wire Wire Line
+	1300 5900 1600 5900
+Wire Wire Line
+	1300 5900 1300 6000
 $EndSCHEMATC

Commit message: - as-built changes - add custom library elements
Parts:
- added C? (x2): 100n*, symbol Device:C_Small
- added D? (x3): 4148*, symbol Diode:PMEG4005EJ
- added Q? (x2): SI2365*, symbol Transistor_FET:BSS84
- added Q?: BSS138*, symbol Transistor_FET:2N7002
- added R106b: 3k3, symbol Device:R_Small
- added R?: 33R*, Resistor_SMD:R_0603_1608Metric_Pad1.05x0.95mm_HandSolder, symbol Device:R_Small
- added R?: 51k*, symbol Device:R_Small
- C80: value 47u -> 470u*
- C87: value 10n -> 11uF*
- R106: value 3k6 -> 3k3
- R108: value 1k2 -> 560R
Connections:
- net +BATT: now also Q?.2 (S), Q?.2 (S), R?.1; no longer C80.1, C81.1, C82.1, L10.1, U19.2 (VIN), U19.3 (EN)
- net -5V: now also D?.2 (A)
- net GND: now also C?.1, D?.1 (K), Q?.2 (S), R106b.1
- net at C90.2, D12.1 (K), R106.2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: now also R106b.2
- net at D16.2 (A), L11.2, R110.1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: now also R?.1
- new net: C80.1, C81.1, C82.1, L10.1, Q?.3 (D), Q?.3 (D), U19.2 (VIN), U19.3 (EN)
- new net: C?.1, R?.2
- new net: C?.2, D?.1 (K), D?.2 (A) (x2)
- new net: Q?.1 (G), Q?.1 (G), Q?.3 (D), R?.2
- new net TP32: Q?.1 (G)
Other:
- note added: "Patch: additional pump circuit added to pull -5 V \nbelow GND, when 12 V converter is disabled.\n\n! It works on battery, but don't works when battery is charged \nand charger gives 5 V out - converter passes voltage without boosting."
- moved on the sheet: C199, C200, C74, C75, C76, C77, C78, C79, C80, C81, C82, C84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
