File: Battery_Charger.sch (KiCad schematic (older format))
At the start: 29 parts

Commit message: - W.i.P.
Parts:
- removed F?: Polyfuse, symbol Device:Polyfuse_Small
- removed Q? (x2): BSS138, Package_TO_SOT_SMD:SOT-23, symbol Transistor_FET:BSS138
- removed SW?: PWRON, symbol Switch:SW_MEC_5E
- added F?: 2.5A, Fuse:Fuse_1812_4532Metric_Pad1.30x3.40mm_HandSolder, symbol Device:Polyfuse_Small
- added NTC?: 10k, Resistor_SMD:R_1206_3216Metric_Pad1.42x1.75mm_HandSolder, symbol Device:Thermistor_NTC
- added Q? (x2): 2N7002, Package_TO_SOT_SMD:SOT-23, symbol Transistor_FET:2N7002
- added SW?: PWRON, Button_Switch_SMD:SW_Push_1P1T_NO_6x6mm_H9.5mm, symbol Switch:SW_MEC_5E
- F?: value Polyfuse -> 2.5A; footprint (none) -> Fuse:Fuse_1812_4532Metric_Pad1.30x3.40mm_HandSolder; Mfr. (none) -> Bel Fuse; Mfr. No (none) -> 0ZCG0125AF2B; Price [PLN] (none) -> 0.45
- J?: footprint Connector_USB:USB_Micro-B_Amphenol_10103594-0001LF_Horizontal -> Connector_USB:USB_Micro-B_Amphenol_10118194_Horizontal; Mfr. (none) -> Amphenol; Mfr. No (none) -> 10118194-0001LF
Connections:
- net GND: now also NTC?.2, Q?.2 (S), Q?.2 (S), SW?.1, SW?.2
- net PWRON_LOCK: now also Q?.1 (G)
- net SYSOFF: now also Q?.3 (D), Q?.3 (D), SW?.3 (K), SW?.4 (A)
- net Vusb: now also Q?.1 (G)
- net at U?.3 (2+): now also F?.1
- net at C?.2, C?.2, F?.2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: now also F?.2
- net at NTC?.1, U?.1 (TS): now also NTC?.1
Changed lines of the file:
@@
 $Descr A4 11693 8268
 encoding utf-8
-Sheet 8 8
+Sheet 7 10
 Title ""
 Date ""
@@
 F 0 "J?" H 3155 2917 50  0000 C CNN
 F 1 "USB_B_Micro" H 3155 2826 50  0000 C CNN
-F 2 "Connector_USB:USB_Micro-B_Amphenol_10103594-0001LF_Horizontal" H 3250 2400 50  0001 C CNN
-F 3 "~" H 3250 2400 50  0001 C CNN
+F 2 "Connector_USB:USB_Micro-B_Amphenol_10118194_Horizontal" H 3250 2400 50  0001 C CNN
+F 3 "https://www.amphenol-icc.com/micro-usb-101181940001lf.html" H 3250 2400 50  0001 C CNN
+F 4 "Amphenol" H 3100 2450 50  0001 C CNN "Mfr."
+F 5 "10118194-0001LF" H 3100 2450 50  0001 C CNN "Mfr. No"
 	1    3100 2450
 	1    0    0    -1
@@
 	5950 3250 5950 3300
 $Comp
-L Switch:SW_MEC_5E SW?
-U 1 1 5F7AA9DF
-P 7850 3900
-AR Path="/5F620813/5F7AA9DF" Ref="SW?"  Part="1"
-AR Path="/5F7A93EE/5F7AA9DF" Ref="SW?"  Part="1"
-F 0 "SW?" V 7900 3950 50  0000 R CNN
-F 1 "PWRON" V 7800 3950 50  0000 R CNN
-F 2 "" H 7850 4200 50  0001 C CNN
-F 3 "http://www.apem.com/int/index.php?controller=attachment&id_attachment=1371" H 7850 4200 50  0001 C CNN
-	1    7850 3900
-	0    -1   -1   0
-$EndComp
-$Comp
 L Device:R_Small R?
 U 1 1 5F7AA9E6
@@
 	7750 3700 7750 3550
 Connection ~ 7750 3550
-Wire Wire Line
-	7850 3700 7750 3700
 Connection ~ 7750 3700
 Wire Wire Line
@@
 	1    0    0    -1
 $EndComp
-Connection ~ 7750 4100
-$Comp
-L Transistor_FET:BSS138 Q?
-U 1 1 5F7AAA0C
-P 7200 4100
-AR Path="/5F620813/5F7AAA0C" Ref="Q?"  Part="1"
-AR Path="/5F7A93EE/5F7AAA0C" Ref="Q?"  Part="1"
-F 0 "Q?" H 7405 4146 50  0000 L CNN
-F 1 "BSS138" H 7405 4055 50  0000 L CNN
-F 2 "Package_TO_SOT_SMD:SOT-23" H 7400 4025 50  0001 L CIN
-F 3 "https://www.onsemi.com/pub/Collateral/BSS138-D.PDF" H 7200 4100 50  0001 L CNN
-	1    7200 4100
-	1    0    0    -1
-$EndComp
 Wire Wire Line
 	7300 3900 7300 3700
-Connection ~ 7850 3700
 Wire Wire Line
 	7750 4300 7750 4100
 Connection ~ 7750 4300
-$Comp
-L Transistor_FET:BSS138 Q?
-U 1 1 5F7AAA19
-P 8500 4100
-AR Path="/5F620813/5F7AAA19" Ref="Q?"  Part="1"
-AR Path="/5F7A93EE/5F7AAA19" Ref="Q?"  Part="1"
-F 0 "Q?" H 8705 4146 50  0000 L CNN
-F 1 "BSS138" H 8705 4055 50  0000 L CNN
-F 2 "Package_TO_SOT_SMD:SOT-23" H 8700 4025 50  0001 L CIN
-F 3 "https://www.onsemi.com/pub/Collateral/BSS138-D.PDF" H 8500 4100 50  0001 L CNN
-	1    8500 4100
-	-1   0    0    -1
-$EndComp
 Wire Wire Line
 	8400 3900 8400 3700
@@
 $Comp
 L Device:Polyfuse_Small F?
-U 1 1 5F6C212E
-P 6450 3400
-F 0 "F?" H 6518 3446 50  0000 L CNN
-F 1 "Polyfuse" H 6518 3355 50  0000 L CNN
-F 2 "" H 6500 3200 50  0001 L CNN
-F 3 "~" H 6450 3400 50  0001 C CNN
-	1    6450 3400
-	1    0    0    -1
-$EndComp
-$Comp
-L Device:Polyfuse_Small F?
 U 1 1 5F6C226D
 P 6250 3400
 F 0 "F?" H 6300 3350 50  0000 L CNN
-F 1 "Polyfuse" H 6300 3450 50  0000 L CNN
-F 2 "" H 6300 3200 50  0001 L CNN
+F 1 "2.5A" H 6300 3450 50  0000 L CNN
+F 2 "Fuse:Fuse_1812_4532Metric_Pad1.30x3.40mm_HandSolder" H 6300 3200 50  0001 L CNN
 F 3 "~" H 6250 3400 50  0001 C CNN
+F 4 "Bel Fuse" H 6250 3400 50  0001 C CNN "Mfr."
+F 5 "0ZCG0125AF2B " H 6250 3400 50  0001 C CNN "Mfr. No"
+F 6 "0.45" H 6250 3400 50  0001 C CNN "Price [PLN]"
 	1    6250 3400
 	-1   0    0    1
@@
 Connection ~ 6250 3300
 Wire Wire Line
-	6250 3300 6450 3300
-Connection ~ 6450 3300
-Wire Wire Line
-	6450 3300 7750 3300
-Wire Wire Line
-	5900 3900 5900 4000
-Wire Wire Line
-	5350 3500 5900 3500
+	5900 3900 5900 3950
+Wire Wire Line
+	5350 3500 5700 3500
 Wire Wire Line
 	5350 3300 5650 3300
@@
 	7750 4300 7300 4300
 Wire Wire Line
-	7850 3700 8400 3700
-Wire Wire Line
 	7750 4300 8400 4300
+Wire Wire Line
+	6250 3300 6450 3300
+$Comp
+L Device:Polyfuse_Small F?
+U 1 1 5F86532F
+P 6450 3400
+F 0 "F?" H 6500 3350 50  0000 L CNN
+F 1 "2.5A" H 6450 3500 50  0000 L CNN
+F 2 "Fuse:Fuse_1812_4532Metric_Pad1.30x3.40mm_HandSolder" H 6500 3200 50  0001 L CNN
+F 3 "~" H 6450 3400 50  0001 C CNN
+F 4 "Bel Fuse" H 6450 3400 50  0001 C CNN "Mfr."
+F 5 "0ZCG0125AF2B " H 6450 3400 50  0001 C CNN "Mfr. No"
+F 6 "0.45" H 6450 3400 50  0001 C CNN "Price [PLN]"
+	1    6450 3400
+	-1   0    0    1
+$EndComp
+Connection ~ 6450 3300
+Wire Wire Line
+	6450 3300 7750 3300
+$Comp
+L Transistor_FET:2N7002 Q?
+U 1 1 5F8658FF
+P 7200 4100
+F 0 "Q?" H 7405 4146 50  0000 L CNN
+F 1 "2N7002" H 7405 4055 50  0000 L CNN
+F 2 "Package_TO_SOT_SMD:SOT-23" H 7400 4025 50  0001 L CIN
+F 3 "https://www.onsemi.com/pub/Collateral/NDS7002A-D.PDF" H 7200 4100 50  0001 L CNN
+	1    7200 4100
+	1    0    0    -1
+$EndComp
+$Comp
+L Transistor_FET:2N7002 Q?
+U 1 1 5F865B17
+P 8500 4100
+F 0 "Q?" H 8705 4146 50  0000 L CNN
+F 1 "2N7002" H 8705 4055 50  0000 L CNN
+F 2 "Package_TO_SOT_SMD:SOT-23" H 8700 4025 50  0001 L CIN
+F 3 "https://www.onsemi.com/pub/Collateral/NDS7002A-D.PDF" H 8500 4100 50  0001 L CNN
+	1    8500 4100
+	-1   0    0    -1
+$EndComp
+$Comp
+L Switch:SW_MEC_5E SW?
+U 1 1 5F865F09
+P 7850 3900
+F 0 "SW?" V 7896 3812 50  0000 R CNN
+F 1 "PWRON" V 7805 3812 50  0000 R CNN
+F 2 "Button_Switch_SMD:SW_Push_1P1T_NO_6x6mm_H9.5mm" H 7850 4200 50  0001 C CNN
+F 3 "http://www.apem.com/int/index.php?controller=attachment&id_attachment=1371" H 7850 4200 50  0001 C CNN
+F 4 "TL3301TF160QG" V 7850 3900 50  0001 C CNN "Mfr. No"
+F 5 "1.27" V 7850 3900 50  0001 C CNN "Price [PLN]"
+	1    7850 3900
+	0    -1   -1   0
+$EndComp
+Wire Wire Line
+	7750 3700 7850 3700
+Connection ~ 7750 4100
+Wire Wire Line
+	8400 3700 7850 3700
+Connection ~ 7850 3700
+$Comp
+L Device:Thermistor_NTC NTC?
+U 1 1 5F869CC1
+P 5700 3750
+AR Path="/5F620813/5F869CC1" Ref="NTC?"  Part="1"
+AR Path="/5F7A93EE/5F869CC1" Ref="NTC?"  Part="1"
+F 0 "NTC?" H 5798 3796 50  0001 L CNN
+F 1 "10k" H 5798 3705 50  0001 L CNN
+F 2 "Resistor_SMD:R_1206_3216Metric_Pad1.42x1.75mm_HandSolder" H 5700 3800 50  0001 C CNN
+F 3 "~" H 5700 3800 50  0001 C CNN
+	1    5700 3750
+	1    0    0    -1
+$EndComp
+Wire Wire Line
+	5700 3600 5700 3500
+Connection ~ 5700 3500
+Wire Wire Line
+	5700 3500 5900 3500
+Wire Wire Line
+	5700 3900 5700 3950
+Wire Wire Line
+	5700 3950 5900 3950
+Connection ~ 5900 3950
+Wire Wire Line
+	5900 3950 5900 4000
 $EndSCHEMATC

Commit message: - connect things to MCUlow (DAC, screen, keys, debug) - improvement in charger (read PWR key)
Parts:
- removed SW?: PWRON, Button_Switch_SMD:SW_Push_1P1T_NO_6x6mm_H9.5mm, symbol Switch:SW_MEC_5E
- added C?: 100n, Capacitor_SMD:C_0603_1608Metric_Pad1.05x0.95mm_HandSolder, symbol Device:C_Small
- added C?: 10n, Capacitor_SMD:C_0603_1608Metric_Pad1.05x0.95mm_HandSolder, symbol Device:C_Small
- added D? (x3): 1N4448, Diode_SMD:D_SOD-323, symbol Device:D_Small
- added F?: 2.5A, Fuse:Fuse_1812_4532Metric_Pad1.30x3.40mm_HandSolder, symbol Device:Polyfuse_Small
- added Q?: BSS84, Package_TO_SOT_SMD:SOT-23, symbol Transistor_FET:BSS84
- added Q?: 2N7002, Package_TO_SOT_SMD:SOT-23, symbol Transistor_FET:2N7002
- added R? (x2): 47k, Resistor_SMD:R_0603_1608Metric_Pad1.05x0.95mm_HandSolder, symbol Device:R_Small
- added R? (x3): 10k, Resistor_SMD:R_0603_1608Metric_Pad1.05x0.95mm_HandSolder, symbol Device:R_Small
- added R?: 1M, Resistor_SMD:R_0603_1608Metric_Pad1.05x0.95mm_HandSolder, symbol Device:R_Small
- added SW?: PWRON, Button_Switch_SMD:SW_Push_1P1T_NO_6x6mm_H9.5mm, symbol Switch:SW_MEC_5E
- added TP? (x3): TestPoint, TestPoint:TestPoint_THTPad_D1.5mm_Drill0.7mm, symbol Connector:TestPoint
- SW?: value SW_DIP_x02 -> set_current
Connections:
- net GND: now also C?.1, C?.2, Q?.2 (S), R?.1, R?.1, R?.1, SW?.1, SW?.2
- net PWRON_LOCK: now also D?.2 (A); no longer Q?.1 (G)
- net Vusb: now also C?.1, F?.2, R?.2; no longer J?.1 (VBUS)
- net at C?.2, C?.2, F?.2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: now also Q?.2 (S), R?.1
- net at J?.2 (D-): now also TP?.1
- net at J?.3 (D+): now also TP?.1
- net at J?.4 (ID): now also TP?.1
- new net: F?.1, J?.1 (VBUS)
- new net: D?.1 (K), D?.1 (K), Q?.1 (G), R?.2
- new net: R?.1, R?.2, SW?.3 (K), SW?.4 (A)
- new net: C?.2, Q?.1 (G), R?.2
- new net: D?.2 (A), D?.2 (A), Q?.3 (D)
- new net: D?.1 (K), Q?.1 (G), R?.2
- new net +3V3: R?.1
- new net KEY_PWR: Q?.3 (D), R?.2
- no-connect marks 3 -> 0
Other:
- note added: "EN2 / EN1 setting:\n0 0 - 100 mA (USB mode)\n0 1 - 500 mA (USB mode)\n1 0 - 1 A (charger)\n1 1 - standby (suspend)"
- moved on the sheet: C?, Q?, R?

Commit message: - final schematic
Parts:
- gave numbers to parts that had none: 47
Connections:
- net PWRON_LOCK renamed PWR_LOCK

Commit message: - init PCB - fix last things in schematic
Parts:
- removed SW3: PWRON, Button_Switch_SMD:SW_Push_1P1T_NO_6x6mm_H9.5mm, symbol Switch:SW_MEC_5E
- added SW3: PWRON, Button_Switch_SMD:SW_Push_1P1T_NO_6x6mm_H9.5mm, symbol Switch:SW_Push
- added TP24: TestPoint, TestPoint:TestPoint_THTPad_D1.5mm_Drill0.7mm, symbol Connector:TestPoint
- Q12, Q13, Q14: value 2N7002 -> BSS138
- U24: footprint (none) -> Power_my:BatteryHolder_Eagle-12BHC186P
Connections:
- net GND: now also SW3.1
- net at U23.7 (~PGOOD): now also TP24.1
- net at R114.2, R115.1: now also SW3.2
Other:
- moved on the sheet: R114
Changed lines of the file:
@@
 F 0 "U24" H 6538 3796 50  0000 L CNN
 F 1 "Holder 2x18650" H 6538 3705 50  0000 L CNN
-F 2 "" H 6800 4550 50  0001 C CNN
+F 2 "Power_my:BatteryHolder_Eagle-12BHC186P" H 6800 4550 50  0001 C CNN
 F 3 "" H 6800 4550 50  0001 C CNN
 	1    6350 3750
@@
 P 7250 5050
 F 0 "Q12" H 7400 5300 50  0000 L CNN
-F 1 "2N7002" H 7400 5200 50  0000 L CNN
+F 1 "BSS138" H 7400 5200 50  0000 L CNN
 F 2 "Package_TO_SOT_SMD:SOT-23" H 7450 4975 50  0001 L CIN
 F 3 "https://www.onsemi.com/pub/Collateral/NDS7002A-D.PDF" H 7250 5050 50  0001 L CNN
@@
 P 7950 5050
 F 0 "Q13" H 8155 5096 50  0000 L CNN
-F 1 "2N7002" H 8155 5005 50  0000 L CNN
+F 1 "BSS138" H 8155 5005 50  0000 L CNN
 F 2 "Package_TO_SOT_SMD:SOT-23" H 8150 4975 50  0001 L CIN
 F 3 "https://www.onsemi.com/pub/Collateral/NDS7002A-D.PDF" H 7950 5050 50  0001 L CNN
@@
 	1    4200 2450
 	1    0    0    -1
-$EndComp
-$Comp
-L Switch:SW_MEC_5E SW3
-U 1 1 5FE2B309
-P 9450 3800
-F 0 "SW3" V 9500 3850 50  0000 R CNN
-F 1 "PWRON" V 9400 3850 50  0000 R CNN
-F 2 "Button_Switch_SMD:SW_Push_1P1T_NO_6x6mm_H9.5mm" H 9450 4100 50  0001 C CNN
-F 3 "http://www.apem.com/int/index.php?controller=attachment&id_attachment=1371" H 9450 4100 50  0001 C CNN
-F 4 "TL3301TF160QG" V 9450 3800 50  0001 C CNN "Mfr. No"
-F 5 "1.27" V 9450 3800 50  0001 C CNN "Price [PLN]"
-	1    9450 3800
-	0    -1   -1   0
 $EndComp
 $Comp
@@
 L Device:R_Small R?
 U 1 1 5FE31AB0
-P 9450 3450
+P 9350 3450
 AR Path="/5F7D6767/5FE31AB0" Ref="R?"  Part="1"
 AR Path="/5F7A93EE/5FE31AB0" Ref="R114"  Part="1"
-F 0 "R114" H 9509 3496 50  0000 L CNN
-F 1 "10k" H 9509 3405 50  0000 L CNN
-F 2 "Resistor_SMD:R_0603_1608Metric_Pad1.05x0.95mm_HandSolder" H 9450 3450 50  0001 C CNN
-F 3 "~" H 9450 3450 50  0001 C CNN
-	1    9450 3450
+F 0 "R114" H 9409 3496 50  0000 L CNN
+F 1 "10k" H 9409 3405 50  0000 L CNN
+F 2 "Resistor_SMD:R_0603_1608Metric_Pad1.05x0.95mm_HandSolder" H 9350 3450 50  0001 C CNN
+F 3 "~" H 9350 3450 50  0001 C CNN
+	1    9350 3450
 	1    0    0    -1
 $EndComp
@@
 P 9250 5050
 F 0 "Q14" H 9455 5096 50  0000 L CNN
-F 1 "2N7002" H 9455 5005 50  0000 L CNN
+F 1 "BSS138" H 9455 5005 50  0000 L CNN
 F 2 "Package_TO_SOT_SMD:SOT-23" H 9450 4975 50  0001 L CIN
 F 3 "https://www.onsemi.com/pub/Collateral/NDS7002A-D.PDF" H 9250 5050 50  0001 L CNN
@@
 $EndComp
 Wire Wire Line
-	9450 3300 9450 3350
+	9350 3300 9350 3350
 Wire Wire Line
 	8450 3400 8450 3300
 Connection ~ 8450 3300
 Wire Wire Line
-	8450 3300 9450 3300
+	8450 3300 9350 3300
 Wire Wire Line
 	8750 3650 8750 3600
@@
 	8750 3600 8950 3600
 Wire Wire Line
-	9450 3600 9450 3550
+	9350 3600 9350 3550
 Connection ~ 8750 3600
 $Comp
@@
 	1    0    0    -1
 $EndComp
-Wire Wire Line
-	9450 4000 9350 4000
-Connection ~ 9350 4000
 Connection ~ 9350 4850
 Wire Wire Line
@@
 Wire Wire Line
 	6450 3300 7350 3300
-Wire Wire Line
-	9150 3600 9350 3600
-Wire Wire Line
-	9350 3600 9450 3600
-Connection ~ 9350 3600
-Connection ~ 9450 3600
 Wire Wire Line
 	8550 5550 8450 5550
@@
 Text GLabel 8550 5550 2    50   Output ~ 0
 PWR_LOCK
+$Comp
+L Connector:TestPoint TP24
+U 1 1 5FA4C9CB
+P 5350 3700
+F 0 "TP24" V 5250 3750 50  0000 L CNN
+F 1 "TestPoint" V 5395 3888 50  0001 L CNN
+F 2 "TestPoint:TestPoint_THTPad_D1.5mm_Drill0.7mm" H 5550 3700 50  0001 C CNN
+F 3 "~" H 5550 3700 50  0001 C CNN
+	1    5350 3700
+	0    1    1    0
+$EndComp
+$Comp
+L power:PWR_FLAG #FLG?
+U 1 1 5FA3853B
+P 4500 2250
+AR Path="/5F61C123/5FA3853B" Ref="#FLG?"  Part="1"
+AR Path="/5F7A93EE/5FA3853B" Ref="#FLG0106"  Part="1"
+F 0 "#FLG0106" H 4500 2325 50  0001 C CNN
+F 1 "PWR_FLAG" H 4500 2424 50  0001 C CNN
+F 2 "" H 4500 2250 50  0001 C CNN
+F 3 "~" H 4500 2250 50  0001 C CNN
+	1    4500 2250
+	1    0    0    -1
+$EndComp
+$Comp
+L Switch:SW_Push SW?
+U 1 1 5FBC9B04
+P 9350 3800
+AR Path="/5F7D6767/5FBC9B04" Ref="SW?"  Part="1"
+AR Path="/5F7A93EE/5FBC9B04" Ref="SW3"  Part="1"
+F 0 "SW3" V 9400 3750 50  0000 R CNN
+F 1 "PWRON" V 9300 3750 50  0000 R CNN
+F 2 "Button_Switch_SMD:SW_Push_1P1T_NO_6x6mm_H9.5mm" H 9350 4000 50  0001 C CNN
+F 3 "~" H 9350 4000 50  0001 C CNN
+	1    9350 3800
+	0    -1   -1   0
+$EndComp
+Wire Wire Line
+	9150 3600 9350 3600
+Connection ~ 9350 3600
 $EndSCHEMATC
