File: uScope.sch (KiCad schematic (older format))
At the start: 9 parts, among them U1 K, U2 E, U3 F

Commit message: - W.i.P.
Parts:
- removed R?: VR25 470k, Resistor_THT:R_Axial_DIN0207_L6.3mm_D2.5mm_P10.16mm_Horizontal, symbol Device:R
- added R?: VR25 470k, Resistor_THT:R_Axial_DIN0207_L6.3mm_D2.5mm_P10.16mm_Horizontal, symbol Device:R_Small
- added U?: IL300, symbol Isolator_Analog:IL300
- added U?: NHD-0420H1Z, Display:NHD-0420H1Z, symbol Display_Character:NHD-0420H1Z
- added U?: NHD-C0220BIZ, Display:NHD-C0220BiZ, symbol Display_Character:NHD-C0220BIZ
- R?: symbol Device:R -> Device:R_Small; Mfr. (none) -> Vishay; Mfr. No (none) -> VR25000004703JA500; Price [PLN] (none) -> 0.6
Other:
- note added: "TODO:\n- battery fuse (reverse connection protection - nie ma sensu)\n- dla PAMxx dobrac tez mniejsza cewke (5u6? 4u7?)\nmoze byc potrzebna dla wiekszych pradow\n- zasilanie strony wysokiej przewidziec z baterii, miejsce zostawic (gdyby RECOM nie doszedl)\n- STM32G030K8 symbol dodac.. a moze 'F' bedzie ok? Porownac rozklad pinow\n- Nucleo dodac symbol connectorow, i wytrzasnac skads model 3D i fo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"
- note removed: "TODO:\n- tranzystory drivera, moc dobrac\n- battery fuse (reverse connection protection - nie ma sensu)\n- dla PAMxx dobrac tez mniejsza cewke (5u6? 4u7?)\nmoze byc potrzebna dla wiekszych pradow\n- ! polaczenie zrodel zasilania moze byc uwarunkowane tym, z ktorej strony wplywa prad. Bo nie sa to zrodla push-pull, tylko push."
Changed lines of the file:
@@
 $Descr A4 11693 8268
 encoding utf-8
-Sheet 1 8
+Sheet 1 10
 Title ""
 Date ""
@@
 S 5250 4800 1700 1250
 U 5F7D6767
-F0 "MCU" 50
-F1 "MCU.sch" 50
+F0 "MCU_low" 50
+F1 "MCU_low.sch" 50
 F2 "PWRON_MCU" O L 5250 5150 50
 F3 "BATT_SENSE" I L 5250 5550 50
@@
 $EndSheet
 Text Notes 7950 1600 0    100  ~ 20
-TODO:\n- tranzystory drivera, moc dobrac\n- battery fuse (reverse connection protection - nie ma sensu)\n- dla PAMxx dobrac tez mniejsza cewke (5u6? 4u7?)\nmoze byc potrzebna dla wiekszych pradow\n- ! polaczenie zrodel zasilania moze byc uwarunkowane tym, z ktorej strony wplywa prad. Bo nie sa to zrodla push-pull, tylko push.
+TODO:\n- battery fuse (reverse connection protection - nie ma sensu)\n- dla PAMxx dobrac tez mniejsza cewke (5u6? 4u7?)\nmoze byc potrzebna dla wiekszych pradow\n- zasilanie strony wysokiej przewidziec z baterii, miejsce zostawic (gdyby RECOM nie doszedl)\n- STM32G030K8 symbol dodac.. a moze 'F' bedzie ok? Porownac rozklad pinow\n- Nucleo dodac symbol connectorow, i wytrzasnac skads model 3D i footprint
 $Comp
 L power:-VDC #PWR?
@@
 $EndComp
 $Comp
-L Device:R R?
+L Device:R_Small R?
 U 1 1 5F7FDE7C
 P 1200 2600
@@
 F 2 "Resistor_THT:R_Axial_DIN0207_L6.3mm_D2.5mm_P10.16mm_Horizontal" V 1130 2600 50  0001 C CNN
 F 3 "~" H 1200 2600 50  0001 C CNN
+F 4 "Vishay" V 1200 2600 50  0001 C CNN "Mfr."
+F 5 "VR25000004703JA500" V 1200 2600 50  0001 C CNN "Mfr. No"
+F 6 "0.6" V 1200 2600 50  0001 C CNN "Price [PLN]"
 	1    1200 2600
-	0    -1   -1   0
-$EndComp
-$Comp
-L Device:R R?
-U 1 1 5F7FE032
-P 1800 2600
-AR Path="/5F40DCB9/5F7FE032" Ref="R?"  Part="1"
-AR Path="/5F479892/5F7FE032" Ref="R?"  Part="1"
-AR Path="/5F7FE032" Ref="R?"  Part="1"
-F 0 "R?" V 1900 2600 50  0000 C CNN
-F 1 "VR25 470k" V 1700 2600 50  0000 C CNN
-F 2 "Resistor_THT:R_Axial_DIN0207_L6.3mm_D2.5mm_P10.16mm_Horizontal" V 1730 2600 50  0001 C CNN
-F 3 "~" H 1800 2600 50  0001 C CNN
-	1    1800 2600
 	0    -1   -1   0
 $EndComp
@@
 	1500 3300 1500 3100
 Wire Wire Line
-	1350 2600 1500 2600
-Wire Wire Line
-	1950 2600 2100 2600
+	1300 2600 1500 2600
+Wire Wire Line
+	1900 2600 2100 2600
 Wire Wire Line
 	2100 2600 2100 2900
@@
 Connection ~ 1500 2600
 Wire Wire Line
-	1500 2600 1650 2600
+	1500 2600 1700 2600
 Wire Wire Line
 	900  2800 900  2600
 Wire Wire Line
-	900  2600 1050 2600
+	900  2600 1100 2600
 Connection ~ 2100 2600
 $Comp
@@
 	1    0    0    -1
 $EndComp
+$Comp
+L Device:R_Small R?
+U 1 1 5F82AF16
+P 1800 2600
+AR Path="/5F40DCB9/5F82AF16" Ref="R?"  Part="1"
+AR Path="/5F479892/5F82AF16" Ref="R?"  Part="1"
+AR Path="/5F82AF16" Ref="R?"  Part="1"
+F 0 "R?" V 1900 2600 50  0000 C CNN
+F 1 "VR25 470k" V 1700 2600 50  0000 C CNN
+F 2 "Resistor_THT:R_Axial_DIN0207_L6.3mm_D2.5mm_P10.16mm_Horizontal" V 1730 2600 50  0001 C CNN
+F 3 "~" H 1800 2600 50  0001 C CNN
+F 4 "Vishay" V 1800 2600 50  0001 C CNN "Mfr."
+F 5 "VR25000004703JA500" V 1800 2600 50  0001 C CNN "Mfr. No"
+F 6 "0.6" V 1800 2600 50  0001 C CNN "Price [PLN]"
+	1    1800 2600
+	0    -1   -1   0
+$EndComp
+$Sheet
+S 3800 3700 600  900
+U 5F82F010
+F0 "communication" 50
+F1 "communication.sch" 50
+F2 "UART_TX" I R 4400 4400 50
+F3 "UART_RX" O R 4400 4500 50
+F4 "HV_UART_RX" O L 3800 3750 50
+F5 "HV_UART_TX" I L 3800 3850 50
+$EndSheet
+$Sheet
+S 2850 900  900  600
+U 5F8337DC
+F0 "MCU_high" 50
+F1 "MCU_high.sch" 50
+F2 "UART_RX" I L 2850 1150 50
+F3 "UART_TX" O L 2850 1250 50
+$EndSheet
+$Comp
+L Isolator_Analog:IL300 U?
+U 1 1 5F862EA9
+P 10100 2750
+F 0 "U?" H 10100 3275 50  0000 C CNN
+F 1 "IL300" H 10100 3184 50  0000 C CNN
+F 2 "" H 9800 3050 50  0001 L CNN
+F 3 "http://www.vishay.com/docs/83622/il300.pdf" H 9900 3150 50  0001 L CNN
+	1    10100 2750
+	1    0    0    -1
+$EndComp
+$Comp
+L Display_Character:NHD-0420H1Z U?
+U 1 1 5F873B78
+P 9600 4150
+F 0 "U?" H 9600 3264 50  0000 C CNN
+F 1 "NHD-0420H1Z" H 9600 3173 50  0000 C CNN
+F 2 "Display:NHD-0420H1Z" H 9600 3250 50  0001 C CNN
+F 3 "http://www.newhavendisplay.com/specs/NHD-0420H1Z-FSW-GBW-33V3.pdf" H 9700 4050 50  0001 C CNN
+	1    9600 4150
+	1    0    0    -1
+$EndComp
+$Comp
+L Display_Character:NHD-C0220BIZ U?
+U 1 1 5F873C49
+P 10600 4350
+F 0 "U?" H 10600 5028 50  0000 C CNN
+F 1 "NHD-C0220BIZ" H 10600 4937 50  0000 C CNN
+F 2 "Display:NHD-C0220BiZ" H 10600 3750 50  0001 C CNN
+F 3 "http://www.newhavendisplay.com/specs/NHD-C0220BiZ-FSW-FBW-3V3M.pdf" H 10300 4950 50  0001 C CNN
+	1    10600 4350
+	1    0    0    -1
+$EndComp

Commit message: - MCU_Low: added encoder, DAC, alternate MCU
Parts:
- removed U?: NHD-0420H1Z, Display:NHD-0420H1Z, symbol Display_Character:NHD-0420H1Z
- removed U?: NHD-C0220BIZ, Display:NHD-C0220BiZ, symbol Display_Character:NHD-C0220BIZ
Other:
- note added: "TODO:\n- dla PAMxx dobrac tez mniejsza cewke (5u6? 4u7?)\nmoze byc potrzebna dla wiekszych pradow\n- zasilanie strony wysokiej przewidziec z baterii, miejsce zostawic (gdyby RECOM nie doszedl)\n- STM32G030K8 symbol dodac.. a moze 'F' bedzie ok? Porownac rozklad pinow\n- Nucleo dodac symbol connectorow, i wytrzasnac skads model 3D i footprint\n- ADS'y dodac symbole, rozpisac piny CPU (CubeMX) i wy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"
- note removed: "TODO:\n- battery fuse (reverse connection protection - nie ma sensu)\n- dla PAMxx dobrac tez mniejsza cewke (5u6? 4u7?)\nmoze byc potrzebna dla wiekszych pradow\n- zasilanie strony wysokiej przewidziec z baterii, miejsce zostawic (gdyby RECOM nie doszedl)\n- STM32G030K8 symbol dodac.. a moze 'F' bedzie ok? Porownac rozklad pinow\n- Nucleo dodac symbol connectorow, i wytrzasnac skads model 3D i fo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"
Changed lines of the file:
@@
 $EndSheet
 Text Notes 7950 1600 0    100  ~ 20
-TODO:\n- battery fuse (reverse connection protection - nie ma sensu)\n- dla PAMxx dobrac tez mniejsza cewke (5u6? 4u7?)\nmoze byc potrzebna dla wiekszych pradow\n- zasilanie strony wysokiej przewidziec z baterii, miejsce zostawic (gdyby RECOM nie doszedl)\n- STM32G030K8 symbol dodac.. a moze 'F' bedzie ok? Porownac rozklad pinow\n- Nucleo dodac symbol connectorow, i wytrzasnac skads model 3D i footprint
+TODO:\n- dla PAMxx dobrac tez mniejsza cewke (5u6? 4u7?)\nmoze byc potrzebna dla wiekszych pradow\n- zasilanie strony wysokiej przewidziec z baterii, miejsce zostawic (gdyby RECOM nie doszedl)\n- STM32G030K8 symbol dodac.. a moze 'F' bedzie ok? Porownac rozklad pinow\n- Nucleo dodac symbol connectorow, i wytrzasnac skads model 3D i footprint\n- ADS'y dodac symbole, rozpisac piny CPU (CubeMX) i wybrac proce.\n- IL300 moze byc zasilane z baterii, a jej zalaczanie zrobie przez transoptor
 $Comp
 L power:-VDC #PWR?
@@
 	1    0    0    -1
 $EndComp
-$Comp
-L Display_Character:NHD-0420H1Z U?
-U 1 1 5F873B78
-P 9600 4150
-F 0 "U?" H 9600 3264 50  0000 C CNN
-F 1 "NHD-0420H1Z" H 9600 3173 50  0000 C CNN
-F 2 "Display:NHD-0420H1Z" H 9600 3250 50  0001 C CNN
-F 3 "http://www.newhavendisplay.com/specs/NHD-0420H1Z-FSW-GBW-33V3.pdf" H 9700 4050 50  0001 C CNN
-	1    9600 4150
-	1    0    0    -1
-$EndComp
-$Comp
-L Display_Character:NHD-C0220BIZ U?
-U 1 1 5F873C49
-P 10600 4350
-F 0 "U?" H 10600 5028 50  0000 C CNN
-F 1 "NHD-C0220BIZ" H 10600 4937 50  0000 C CNN
-F 2 "Display:NHD-C0220BiZ" H 10600 3750 50  0001 C CNN
-F 3 "http://www.newhavendisplay.com/specs/NHD-C0220BiZ-FSW-FBW-3V3M.pdf" H 10300 4950 50  0001 C CNN
-	1    10600 4350
-	1    0    0    -1
-$EndComp

Commit message: - drivers modified - MCU replaced
Parts:
- removed U?: IL300, symbol Isolator_Analog:IL300
- added U?: Pump, Library_uScope:APD_P2_single, symbol uScope:APD_P2_single
Other:
- note added: "NOTE:\n* ADS131M06 pin-to-pin compatible with: -M08"
Changed lines of the file:
@@
 $EndComp
 $Sheet
-S 7500 4750 1200 600
+S 7500 4750 1200 1250
 U 5F61C123
 F0 "drivers" 50
 F1 "drivers.sch" 50
-F2 "dac_K" I L 7500 4900 50
-F3 "dac_F" I L 7500 5200 50
-F4 "dac_E" I L 7500 5050 50
+F2 "TIM_CH1" I L 7500 4850 50
+F3 "TIM_CH2" I L 7500 4950 50
+F4 "TIM_CH3" I L 7500 5050 50
+F5 "TIM_CH4" I L 7500 5150 50
+F6 "loadDAC" I L 7500 5350 50
+F7 "DAC_SPI_DIN" I L 7500 5450 50
+F8 "DAC_SPI_CLK" I L 7500 5550 50
+F9 "~DAC_SPI_CS" I L 7500 5650 50
+F10 "~DAC_SPI_SYNC" I L 7500 5750 50
 $EndSheet
 Text Notes 4750 2300 0    50   ~ 0
@@
 	5800 3900 5800 3750
 $Sheet
-S 2900 5000 950  700
+S 2450 6250 950  700
 U 5F620813
 F0 "supply" 50
 F1 "supply.sch" 50
-F2 "BATT_IN" I L 2900 5350 50
-$EndSheet
-$Sheet
-S 1350 5000 950  700
+F2 "BATT_IN" I L 2450 6600 50
+$EndSheet
+$Sheet
+S 900  6250 950  700
 U 5F7A93EE
 F0 "Battery_Charger" 50
 F1 "Battery_Charger.sch" 50
-F2 "V_BATT" O R 2300 5350 50
-F3 "PWRON_LOCK" I L 1350 5450 50
-$EndSheet
-Wire Wire Line
-	2300 5350 2900 5350
-$Sheet
-S 5250 4800 1700 1250
+F2 "V_BATT" O R 1850 6600 50
+F3 "PWRON_LOCK" I L 900 6700 50
+$EndSheet
+Wire Wire Line
+	1850 6600 2450 6600
+$Sheet
+S 4700 5750 1700 1250
 U 5F7D6767
 F0 "MCU_low" 50
 F1 "MCU_low.sch" 50
-F2 "PWRON_MCU" O L 5250 5150 50
-F3 "BATT_SENSE" I L 5250 5550 50
-F4 "dac_K" O R 6950 5150 50
-F5 "dac_F" O R 6950 5300 50
-F6 "dac_E" O R 6950 5550 50
+F2 "PWRON_MCU" O L 4700 6100 50
+F3 "BATT_SENSE" I L 4700 6500 50
+F4 "dac_K" O R 6400 6100 50
+F5 "dac_F" O R 6400 6250 50
+F6 "dac_E" O R 6400 6500 50
 $EndSheet
 Text Notes 7950 1600 0    100  ~ 20
@@
 F3 "UART_TX" O L 2850 1250 50
 $EndSheet
-$Comp
-L Isolator_Analog:IL300 U?
-U 1 1 5F862EA9
-P 10100 2750
-F 0 "U?" H 10100 3275 50  0000 C CNN
-F 1 "IL300" H 10100 3184 50  0000 C CNN
-F 2 "" H 9800 3050 50  0001 L CNN
-F 3 "http://www.vishay.com/docs/83622/il300.pdf" H 9900 3150 50  0001 L CNN
-	1    10100 2750
-	1    0    0    -1
-$EndComp
+Text Notes 850  7650 0    50   ~ 0
+NOTE:\n* ADS131M06 pin-to-pin compatible with: -M08
+$Comp
+L uScope:APD_P2_single U?
+U 2 1 5FA4EFC3
+P 5600 4250
+AR Path="/5FA4EFC3" Ref="U?"  Part="2"
+AR Path="/5F61C123/5FA4EFC3" Ref="U?"  Part="2"
+F 0 "U?" H 5828 4301 50  0000 L CNN
+F 1 "Pump" H 5828 4210 50  0000 L CNN
+F 2 "Library_uScope:APD_P2_single" H 5600 4250 50  0001 C CNN
+F 3 "" H 5600 4250 50  0001 C CNN
+	2    5600 4250
+	1    0    0    -1
+$EndComp

Commit message: - connect things to MCUlow (DAC, screen, keys, debug) - improvement in charger (read PWR key)
Connections:
- wire segments 20 -> 19
Other:
- note added: "TODO:\n- dla PAMxx dobrac tez mniejsza cewke (5u6? 4u7?)\nmoze byc potrzebna dla wiekszych pradow"
- note removed: "TODO:\n- dla PAMxx dobrac tez mniejsza cewke (5u6? 4u7?)\nmoze byc potrzebna dla wiekszych pradow\n- zasilanie strony wysokiej przewidziec z baterii, miejsce zostawic (gdyby RECOM nie doszedl)\n- STM32G030K8 symbol dodac.. a moze 'F' bedzie ok? Porownac rozklad pinow\n- Nucleo dodac symbol connectorow, i wytrzasnac skads model 3D i footprint\n- ADS'y dodac symbole, rozpisac piny CPU (CubeMX) i wy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"
Changed lines of the file:
@@
 $EndComp
 $Sheet
-S 7500 4750 1200 1250
+S 7500 4750 800  1100
 U 5F61C123
 F0 "drivers" 50
@@
 F0 "supply" 50
 F1 "supply.sch" 50
-F2 "BATT_IN" I L 2450 6600 50
 $EndSheet
 $Sheet
@@
 F0 "Battery_Charger" 50
 F1 "Battery_Charger.sch" 50
-F2 "V_BATT" O R 1850 6600 50
 F3 "PWRON_LOCK" I L 900 6700 50
 $EndSheet
-Wire Wire Line
-	1850 6600 2450 6600
 $Sheet
 S 4700 5750 1700 1250
@@
 F1 "MCU_low.sch" 50
 F2 "PWRON_MCU" O L 4700 6100 50
-F3 "BATT_SENSE" I L 4700 6500 50
-F4 "dac_K" O R 6400 6100 50
-F5 "dac_F" O R 6400 6250 50
-F6 "dac_E" O R 6400 6500 50
 $EndSheet
 Text Notes 7950 1600 0    100  ~ 20
-TODO:\n- dla PAMxx dobrac tez mniejsza cewke (5u6? 4u7?)\nmoze byc potrzebna dla wiekszych pradow\n- zasilanie strony wysokiej przewidziec z baterii, miejsce zostawic (gdyby RECOM nie doszedl)\n- STM32G030K8 symbol dodac.. a moze 'F' bedzie ok? Porownac rozklad pinow\n- Nucleo dodac symbol connectorow, i wytrzasnac skads model 3D i footprint\n- ADS'y dodac symbole, rozpisac piny CPU (CubeMX) i wybrac proce.\n- IL300 moze byc zasilane z baterii, a jej zalaczanie zrobie przez transoptor
+TODO:\n- dla PAMxx dobrac tez mniejsza cewke (5u6? 4u7?)\nmoze byc potrzebna dla wiekszych pradow
 $Comp
 L power:-VDC #PWR?

Commit message: - high side (supply, MCU) - low side MCU - much small changes
Parts:
- removed C?: 10n, Capacitor_moja:C_Disc_D18.0_W5.0_P10.0mm, symbol Device:C_Small
- removed U?: ElectronGun_MEMS, symbol uScope:ElectronGun_MEMS
- added C? (x5): 10n, Capacitor_THT:C_Rect_L26.5mm_W10.5mm_P22.50mm_MKS4, symbol Device:C_Small
- added GD?: GDT_75V, miscellaneous_my:Arrester_Axial_L6mm_D6mm_P8.89mm_Horizontal, symbol Device:GDT_2pin
- added J?: Pump-, miscellaneous_my:Terminal_Amp_HB0101, symbol Connector:Screw_Terminal_01x01
- added J?: Conn_01x02, symbol Connector_Generic:Conn_01x02
- added J?: Pump+, miscellaneous_my:Terminal_Amp_HB0101, symbol Connector:Screw_Terminal_01x01
- added J?: U_K, miscellaneous_my:Terminal_Amp_HB0101, symbol Connector:Screw_Terminal_01x01
- added J?: U_F, miscellaneous_my:Terminal_Amp_HB0101, symbol Connector:Screw_Terminal_01x01
- added J?: U_E, miscellaneous_my:Terminal_Amp_HB0101, symbol Connector:Screw_Terminal_01x01
- added J?: Anode, miscellaneous_my:Terminal_Amp_HB0101, symbol Connector:Screw_Terminal_01x01
- added R? (x3): VR37 30M, Resistor_THT:R_Axial_DIN0411_L9.9mm_D3.6mm_P12.70mm_Horizontal, symbol Device:R_Small
- added R? (x4): VR25 470k, Resistor_THT:R_Axial_DIN0207_L6.3mm_D2.5mm_P10.16mm_Horizontal, symbol Device:R_Small
- added TP?: Volt+, miscellaneous_my:Socket_banana4mm, symbol Connector:TestPoint
- added TP?: Volt-, miscellaneous_my:Socket_banana4mm, symbol Connector:TestPoint
- added TP?: Amp+, miscellaneous_my:Socket_banana4mm, symbol Connector:TestPoint
- added TP?: Amp-, miscellaneous_my:Socket_banana4mm, symbol Connector:TestPoint
- C?: footprint Capacitor_moja:C_Disc_D18.0_W5.0_P10.0mm -> Capacitor_THT:C_Rect_L26.5mm_W10.5mm_P22.50mm_MKS4; Voltage 6kV cer. -> 6kV
Connections:
- net labels removed: -VDC
- wire segments 19 -> 59
Other:
- note removed: "(optional\nU_K-E filter)"
- note removed: "Napiecie E: takie polaczenie jest dobre\nze wzgledu na moc, ale tez na eliminacje ripple (nie wplywaja na prad).\nAle co z Focus, moze F tez lepiej podczepic pod katode?\nTo zalezy, czy bedzie tylko dodatnie czy +/- od katody"
- moved on the sheet: C?, R?, U1B, U2B, U3B, U?, U?B

Commit message: - final schematic
Parts:
- gave numbers to parts that had none: 29
Connections:
- net U_E: now also C3.2, J3.1 (Pin_1), R5.2
- net U_F: now also C4.2, J4.1 (Pin_1), R7.2
- net ammeter/in renamed ammeter/current_in
Other:
- moved on the sheet: C1, C2, C3, C4, J3, J4, J7, R4, R5, R6, R7, U2B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

Commit message: - init PCB - fix last things in schematic
Parts:
- J5: footprint (none) -> Connector_PinHeader_2.54mm:PinHeader_1x02_P2.54mm_Vertical
- U1, U2, U3: footprint Library_uScope:APD_P2_single -> Power_my:DCDC_APD_P2_single
- U4: renamed from U5; footprint Library_uScope:APD_P2_single -> Power_my:DCDC_APD_P2_single
- U6: footprint (none) -> Power_my:SIP16_RECOM
Other:
- note added: ""High" side:\nHazardous voltage\nNegative voltage up to -6 kV"
- note added: ""Low" side:\nground / touch / interface potential"
- note added: "Separate circuit.\nNot part of the project,\nbut useful at testing."
Changed lines of the file:
@@
 $EndDescr
 $Sheet
-S 9950 3500 1000 400
+S 5850 7200 1000 400
 U 5F463F4C
 F0 "rippleMeas" 50
@@
 F 0 "U2" H 1600 1600 50  0000 R CNN
 F 1 "E" H 1550 1700 50  0000 R CNN
-F 2 "Library_uScope:APD_P2_single" H 1300 1700 50  0001 C CNN
+F 2 "Power_my:DCDC_APD_P2_single" H 1300 1700 50  0001 C CNN
 F 3 "" H 1300 1700 50  0001 C CNN
 	2    1300 1700
@@
 F 0 "U3" H 3728 1746 50  0000 L CNN
 F 1 "F" H 3728 1655 50  0000 L CNN
-F 2 "Library_uScope:APD_P2_single" H 3550 1700 50  0001 C CNN
+F 2 "Power_my:DCDC_APD_P2_single" H 3550 1700 50  0001 C CNN
 F 3 "" H 3550 1700 50  0001 C CNN
 	2    3550 1700
@@
 F0 "MCU_low" 50
 F1 "MCU_low.sch" 50
-F3 "TIM1_CH1" O R 9500 5150 50
-F4 "TIM1_CH2" O R 9500 5250 50
-F5 "TIM1_CH3" O R 9500 5350 50
-F6 "TIM1_CH4" O R 9500 5450 50
-F7 "DAC_load" O R 9500 5700 50
-F8 "DAC_NSS" O R 9500 6150 50
-F9 "DAC_CS" O R 9500 6050 50
-F10 "DAC_SCK" O R 9500 5950 50
-F11 "DAC_MOSI" O R 9500 5850 50
-F12 "UART_TX" O L 7800 5250 50
-F13 "UART_RX" I L 7800 5150 50
-F14 "ADC_CH0" I L 7800 5500 50
-F15 "ADC_CH1" I L 7800 5600 50
+F2 "TIM1_CH1" O R 9500 5150 50
+F3 "TIM1_CH2" O R 9500 5250 50
+F4 "TIM1_CH3" O R 9500 5350 50
+F5 "TIM1_CH4" O R 9500 5450 50
+F6 "DAC_load" O R 9500 5700 50
+F7 "DAC_NSS" O R 9500 6150 50
+F8 "DAC_CS" O R 9500 6050 50
+F9 "DAC_SCK" O R 9500 5950 50
+F10 "DAC_MOSI" O R 9500 5850 50
+F11 "UART_TX" O L 7800 5250 50
+F12 "UART_RX" I L 7800 5150 50
+F13 "ADC_CH0" I L 7800 5500 50
+F14 "ADC_CH1" I L 7800 5600 50
 $EndSheet
 Text Notes 12000 1100 0    100  ~ 20
@@
 F 0 "U1" H 700 4050 50  0000 R CNN
 F 1 "K" H 650 4150 50  0000 R CNN
-F 2 "Library_uScope:APD_P2_single" H 750 4300 50  0001 C CNN
+F 2 "Power_my:DCDC_APD_P2_single" H 750 4300 50  0001 C CNN
 F 3 "" H 750 4300 50  0001 C CNN
 	2    750  4300
@@
 F 0 "U6" H 3050 4650 50  0000 L CNN
 F 1 "RHV2-1212S/R20" V 3100 3850 50  0000 L CNN
-F 2 "" H 1100 5500 50  0001 C CNN
+F 2 "Power_my:SIP16_RECOM" H 1100 5500 50  0001 C CNN
 F 3 "" H 1100 5500 50  0001 C CNN
 	1    2750 4250
@@
 L power:+12V #PWR?
 U 1 1 5F812227
-P 2600 4800
+P 2600 4850
 AR Path="/5F61C123/5F812227" Ref="#PWR?"  Part="1"
 AR Path="/5F620813/5F812227" Ref="#PWR?"  Part="1"
 AR Path="/5F812227" Ref="#PWR010"  Part="1"
-F 0 "#PWR010" H 2600 4650 50  0001 C CNN
-F 1 "+12V" H 2600 4916 39  0000 C CNN
-F 2 "" H 2600 4800 50  0001 C CNN
-F 3 "" H 2600 4800 50  0001 C CNN
-	1    2600 4800
+F 0 "#PWR010" H 2600 4700 50  0001 C CNN
+F 1 "+12V" H 2600 4966 39  0000 C CNN
+F 2 "" H 2600 4850 50  0001 C CNN
+F 3 "" H 2600 4850 50  0001 C CNN
+	1    2600 4850
 	-1   0    0    1
 $EndComp
@@
 NOTE:\n* ADS131M06 pin-to-pin compatible with: -M08
 $Comp
-L uScope:APD_P2_single U5
+L uScope:APD_P2_single U4
 U 2 1 5FA4EFC3
 P 8700 1100
-AR Path="/5FA4EFC3" Ref="U5"  Part="2"
+AR Path="/5FA4EFC3" Ref="U4"  Part="2"
 AR Path="/5F61C123/5FA4EFC3" Ref="U?"  Part="2"
-F 0 "U5" H 8928 1151 50  0000 L CNN
+F 0 "U4" H 8928 1151 50  0000 L CNN
 F 1 "Pump" H 8928 1060 50  0000 L CNN
-F 2 "Library_uScope:APD_P2_single" H 8700 1100 50  0001 C CNN
+F 2 "Power_my:DCDC_APD_P2_single" H 8700 1100 50  0001 C CNN
 F 3 "" H 8700 1100 50  0001 C CNN
 	2    8700 1100
@@
 F 0 "J5" V 10023 2180 50  0000 L CNN
 F 1 "Conn_01x02" V 10114 2180 50  0000 L CNN
-F 2 "" H 10150 2100 50  0001 C CNN
+F 2 "Connector_PinHeader_2.54mm:PinHeader_1x02_P2.54mm_Vertical" H 10150 2100 50  0001 C CNN
 F 3 "~" H 10150 2100 50  0001 C CNN
 	1    10150 2100
@@
 Wire Wire Line
 	5950 4650 6100 4650
+Wire Wire Line
+	2600 4850 2600 4800
+Text Notes 8200 4100 0    100  ~ 0
+"High" side:\nHazardous voltage\nNegative voltage up to -6 kV
+Text Notes 8200 4650 0    100  ~ 0
+"Low" side:\nground / touch / interface potential
+Wire Notes Line
+	5700 7000 6950 7000
+Text Notes 5900 7500 0    50   ~ 0
+Separate circuit.\nNot part of the project,\nbut useful at testing.
+Wire Notes Line
+	5700 7750 5700 7000
 $EndSCHEMATC

Commit message: - pcb placement, add 3dShapes
Parts:
- TP1, TP4: footprint miscellaneous_my:Socket_banana4mm -> miscellaneous_my:Banana4mmSocket_black
- TP2, TP3: footprint miscellaneous_my:Socket_banana4mm -> miscellaneous_my:Banana4mmSocket_red
Changed lines of the file:
@@
 F 0 "TP3" V 9254 1688 50  0000 L CNN
 F 1 "Volt+" V 9345 1688 50  0000 L CNN
-F 2 "miscellaneous_my:Socket_banana4mm" H 9500 1500 50  0001 C CNN
+F 2 "miscellaneous_my:Banana4mmSocket_red" H 9500 1500 50  0001 C CNN
 F 3 "~" H 9500 1500 50  0001 C CNN
 	1    9300 1500
@@
 F 0 "TP4" V 9254 1888 50  0000 L CNN
 F 1 "Volt-" V 9345 1888 50  0000 L CNN
-F 2 "miscellaneous_my:Socket_banana4mm" H 9500 1700 50  0001 C CNN
+F 2 "miscellaneous_my:Banana4mmSocket_black" H 9500 1700 50  0001 C CNN
 F 3 "~" H 9500 1700 50  0001 C CNN
 	1    9300 1700
@@
 F 0 "TP2" H 10358 1420 50  0000 L CNN
 F 1 "Amp+" H 10358 1329 50  0000 L CNN
-F 2 "miscellaneous_my:Socket_banana4mm" H 10500 1300 50  0001 C CNN
+F 2 "miscellaneous_my:Banana4mmSocket_red" H 10500 1300 50  0001 C CNN
 F 3 "~" H 10500 1300 50  0001 C CNN
 	1    10300 1300
@@
 F 0 "TP1" H 9958 1420 50  0000 L CNN
 F 1 "Amp-" H 9958 1329 50  0000 L CNN
-F 2 "miscellaneous_my:Socket_banana4mm" H 10100 1300 50  0001 C CNN
+F 2 "miscellaneous_my:Banana4mmSocket_black" H 10100 1300 50  0001 C CNN
 F 3 "~" H 10100 1300 50  0001 C CNN
 	1    9900 1300
