File: uScope.sch (KiCad schematic (older format))
At the start: 32 parts, among them J1 Pump+, J2 Pump-, J3 U_E, J4 U_F, J5 Conn_01x02, J6 U_K, J7 Anode, U1 K, U2 E, U3 F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

Commit message: - PCB progress
Parts:
- C1, C2, C3, C4, C5, C6: value 10n -> 3n3
Changed lines of the file:
@@
 AR Path="/5F7FE5C6" Ref="C5"  Part="1"
 F 0 "C5" H 1250 4300 50  0000 R CNN
-F 1 "10n" H 1250 4200 50  0000 R CNN
+F 1 "3n3" H 1250 4200 50  0000 R CNN
 F 2 "Capacitor_THT:C_Rect_L26.5mm_W10.5mm_P22.50mm_MKS4" H 1300 4250 50  0001 C CNN
 F 3 "~" H 1300 4250 50  0001 C CNN
@@
 AR Path="/5F9EAC48" Ref="C6"  Part="1"
 F 0 "C6" H 1750 4300 50  0000 R CNN
-F 1 "10n" H 1750 4200 50  0000 R CNN
+F 1 "3n3" H 1750 4200 50  0000 R CNN
 F 2 "Capacitor_THT:C_Rect_L26.5mm_W10.5mm_P22.50mm_MKS4" H 1800 4250 50  0001 C CNN
 F 3 "~" H 1800 4250 50  0001 C CNN
@@
 AR Path="/5F9F6366" Ref="C2"  Part="1"
 F 0 "C2" H 3950 1750 50  0000 R CNN
-F 1 "10n" H 3950 1650 50  0000 R CNN
+F 1 "3n3" H 3950 1650 50  0000 R CNN
 F 2 "Capacitor_THT:C_Rect_L26.5mm_W10.5mm_P22.50mm_MKS4" H 4000 1700 50  0001 C CNN
 F 3 "~" H 4000 1700 50  0001 C CNN
@@
 AR Path="/5F9F643C" Ref="C4"  Part="1"
 F 0 "C4" H 4500 1800 50  0000 R CNN
-F 1 "10n" H 4500 1700 50  0000 R CNN
+F 1 "3n3" H 4500 1700 50  0000 R CNN
 F 2 "Capacitor_THT:C_Rect_L26.5mm_W10.5mm_P22.50mm_MKS4" H 4550 1750 50  0001 C CNN
 F 3 "~" H 4550 1750 50  0001 C CNN
@@
 AR Path="/5FA157B5" Ref="C1"  Part="1"
 F 0 "C1" H 1700 1750 50  0000 R CNN
-F 1 "10n" H 1700 1650 50  0000 R CNN
+F 1 "3n3" H 1700 1650 50  0000 R CNN
 F 2 "Capacitor_THT:C_Rect_L26.5mm_W10.5mm_P22.50mm_MKS4" H 1750 1700 50  0001 C CNN
 F 3 "~" H 1750 1700 50  0001 C CNN
@@
 AR Path="/5FA157C7" Ref="C3"  Part="1"
 F 0 "C3" H 2250 1800 50  0000 R CNN
-F 1 "10n" H 2250 1700 50  0000 R CNN
+F 1 "3n3" H 2250 1700 50  0000 R CNN
 F 2 "Capacitor_THT:C_Rect_L26.5mm_W10.5mm_P22.50mm_MKS4" H 2300 1750 50  0001 C CNN
 F 3 "~" H 2300 1750 50  0001 C CNN

Commit message: - PCB WiP
Connections:
- net HVGND: now also R9.2; no longer R9.1
- net at U1.4 (-): now also R8.1; no longer R8.2
- new net: C5.1, R8.2, R9.1
Changed lines of the file:
@@
 F 6 "0.6" V 1050 3750 50  0001 C CNN "Price [PLN]"
 	1    1050 3750
-	0    1    1    0
+	0    -1   -1   0
 $EndComp
 $Comp
@@
 F 6 "0.6" V 1550 3750 50  0001 C CNN "Price [PLN]"
 	1    1550 3750
-	0    1    1    0
+	0    -1   -1   0
 $EndComp
 $Sheet

Commit message: - PCB WiP
Other:
- note removed: "Separate circuit.\nNot part of the project,\nbut useful at testing."
Changed lines of the file:
@@
 $Descr A4 11693 8268
 encoding utf-8
-Sheet 1 11
+Sheet 1 10
 Title ""
 Date ""
@@
 Comment4 ""
 $EndDescr
-$Sheet
-S 5850 7200 1000 400
-U 5F463F4C
-F0 "rippleMeas" 50
-F1 "rippleMeas.sch" 50
-$EndSheet
 $Sheet
 S 6100 3700 1200 1100
@@
 Text Notes 8200 4650 0    100  ~ 0
 "Low" side:\nground / touch / interface potential
-Wire Notes Line
-	5700 7000 6950 7000
-Text Notes 5900 7500 0    50   ~ 0
-Separate circuit.\nNot part of the project,\nbut useful at testing.
-Wire Notes Line
-	5700 7750 5700 7000
 $EndSCHEMATC

Commit message: - as-built changes - add custom library elements
Other:
- note added: "NOTE:\n* ADS131M06 pin-to-pin compatible with: -M08\nERRORS/problems on PCB rev 2050:\n- H3 pin (BOOT0) of both MCU's should be connected to GND (problem with startup)\n- need large capacitor between BMS input and battery fuses. Large dropout on fuses caused UVLO at startup. 2700 uF works fine.\n- designators of Testpads on silcscreen\n- more testpoints: Vusb, Vbat, \n- more control of supply: tu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"
- note removed: "NOTE:\n* ADS131M06 pin-to-pin compatible with: -M08"
- note removed: "TODO:\n- dla PAMxx dobrac tez mniejsza cewke (5u6? 4u7?)\nmoze byc potrzebna dla wiekszych pradow"
Changed lines of the file:
@@
 encoding utf-8
 Sheet 1 10
-Title ""
-Date ""
-Rev ""
-Comp ""
+Title "Schemat główny"
+Date "2021-01-18"
+Rev "1.0"
+Comp "Łukasz Sitarek"
 Comment1 ""
 Comment2 ""
@@
 $EndSheet
 $Sheet
-S 2450 6250 950  700
+S 2450 5650 950  700
 U 5F620813
 F0 "supply" 50
@@
 $EndSheet
 $Sheet
-S 900  6250 950  700
+S 900  5650 950  700
 U 5F7A93EE
 F0 "Battery_Charger" 50
@@
 F14 "ADC_CH1" I L 7800 5600 50
 $EndSheet
-Text Notes 12000 1100 0    100  ~ 20
-TODO:\n- dla PAMxx dobrac tez mniejsza cewke (5u6? 4u7?)\nmoze byc potrzebna dla wiekszych pradow
 $Comp
 L Device:R_Small R?
@@
 F5 "ADC_CH1" I L 6050 1750 50
 $EndSheet
-Text Notes 850  7650 0    50   ~ 0
-NOTE:\n* ADS131M06 pin-to-pin compatible with: -M08
+Text Notes 850  7550 0    50   ~ 0
+NOTE:\n* ADS131M06 pin-to-pin compatible with: -M08\nERRORS/problems on PCB rev 2050:\n- H3 pin (BOOT0) of both MCU's should be connected to GND (problem with startup)\n- need large capacitor between BMS input and battery fuses. Large dropout on fuses caused UVLO at startup. 2700 uF works fine.\n- designators of Testpads on silcscreen\n- more testpoints: Vusb, Vbat, \n- more control of supply: turn-off ability (at least of Recom and high side) is useful at charging\nPOSSIBLE IMPROVEMENTS:\n- current measurement on each output\n- current and/or voltage measurement on pump (use rather IL300 and isolated DC-DC than separate ADC)\n- add buzzer to warn about High Voltage output, overload, etc.
 $Comp
 L uScope:APD_P2_single U4
