File: ammeter.sch (KiCad schematic (older format))
At the start: 12 parts

Commit message: - added supply sch draft
Changed lines of the file:
@@
 $Descr A4 11693 8268
 encoding utf-8
-Sheet 8 8
+Sheet 7 9
 Title ""
 Date ""
@@
 $Comp
 L power:GND #PWR?
-U 1 1 5F618E9F
-P 4350 4300
-AR Path="/5F40DCB9/5F618E9F" Ref="#PWR?"  Part="1"
-AR Path="/5F618AB9/5F618E9F" Ref="#PWR?"  Part="1"
-F 0 "#PWR?" H 4350 4140 50  0001 C CNN
-F 1 "GND" V 4350 4223 39  0000 R CNN
-F 2 "" H 4350 4300 50  0001 C CNN
-F 3 "" H 4350 4300 50  0001 C CNN
-	1    4350 4300
-	1    0    0    -1
-$EndComp
-$Comp
-L power:GND #PWR?
 U 1 1 5F618EA5
 P 5000 3800
 AR Path="/5F40DCB9/5F618EA5" Ref="#PWR?"  Part="1"
 AR Path="/5F618AB9/5F618EA5" Ref="#PWR?"  Part="1"
+AR Path="/5F618EA5" Ref="#PWR?"  Part="1"
 F 0 "#PWR?" H 5000 3640 50  0001 C CNN
 F 1 "GND" V 5000 3723 39  0000 R CNN
@@
 Wire Wire Line
 	4200 4000 4500 4000
-Wire Wire Line
-	4500 4300 4350 4300
-Connection ~ 4350 4300
-Wire Wire Line
-	4350 4300 4200 4300
 $Comp
 L Device:C_Small C?
@@
 AR Path="/5F40DCB9/5F618F1D" Ref="#PWR?"  Part="1"
 AR Path="/5F618AB9/5F618F1D" Ref="#PWR?"  Part="1"
+AR Path="/5F618F1D" Ref="#PWR?"  Part="1"
 F 0 "#PWR?" H 6950 3540 50  0001 C CNN
 F 1 "GND" V 6950 3623 39  0000 R CNN
@@
 Text HLabel 7900 3800 2    50   Output ~ 0
 outAdc
+$Comp
+L power:GND #PWR?
+U 1 1 5F626D4A
+P 4350 4300
+AR Path="/5F40DCB9/5F626D4A" Ref="#PWR?"  Part="1"
+AR Path="/5F618AB9/5F626D4A" Ref="#PWR?"  Part="1"
+AR Path="/5F626D4A" Ref="#PWR?"  Part="1"
+F 0 "#PWR?" H 4350 4140 50  0001 C CNN
+F 1 "GND" H 4350 4200 39  0000 C TNN
+F 2 "" H 4350 4300 50  0001 C CNN
+F 3 "" H 4350 4300 50  0001 C CNN
+	1    4350 4300
+	1    0    0    -1
+$EndComp
+Wire Wire Line
+	4200 4300 4350 4300
+Connection ~ 4350 4300
+Wire Wire Line
+	4350 4300 4500 4300
 $EndSCHEMATC

Commit message: - changes..
Parts:
- removed Q?: NPN, symbol Device:Q_NPN_BCE
- removed Q?: PNP, symbol Device:Q_PNP_BCE
- added C?: 1n, symbol Device:C_Small
- added Q?: BC817, Package_TO_SOT_SMD:SOT-23, symbol Transistor_BJT:BC817
- added Q?: BC807, Package_TO_SOT_SMD:SOT-23, symbol Transistor_BJT:BC807
Connections:
- wire segments 28 -> 34
Other:
- moved on the sheet: C?, R?, U?A, U?B, U?C

Commit message: - connect things to MCUlow (DAC, screen, keys, debug) - improvement in charger (read PWR key)
Parts:
- removed D? (x2): 1N4148, Diode_THT:D_DO-35_SOD27_P7.62mm_Horizontal, symbol Diode:1N4148
- added D? (x2): 1N4448WS, Diode_SMD:D_SOD-323, symbol Diode:1N4448WS
Changed lines of the file:
@@
 $Descr A4 11693 8268
 encoding utf-8
-Sheet 5 10
+Sheet 4 10
 Title ""
 Date ""
@@
 	3400 4000 3450 4000
 $Comp
-L Diode:1N4148 D?
-U 1 1 5F618EEA
-P 2950 4150
-AR Path="/5F40DCB9/5F618EEA" Ref="D?"  Part="1"
-AR Path="/5F618AB9/5F618EEA" Ref="D?"  Part="1"
-F 0 "D?" V 2904 4229 50  0000 L CNN
-F 1 "1N4148" V 2995 4229 50  0000 L CNN
-F 2 "Diode_THT:D_DO-35_SOD27_P7.62mm_Horizontal" H 2950 3975 50  0001 C CNN
-F 3 "http://www.nxp.com/documents/data_sheet/1N4148_1N4448.pdf" H 2950 4150 50  0001 C CNN
-	1    2950 4150
-	0    1    1    0
-$EndComp
-$Comp
-L Diode:1N4148 D?
-U 1 1 5F618EF1
-P 2650 4150
-AR Path="/5F40DCB9/5F618EF1" Ref="D?"  Part="1"
-AR Path="/5F618AB9/5F618EF1" Ref="D?"  Part="1"
-F 0 "D?" V 2696 4071 50  0000 R CNN
-F 1 "1N4148" V 2605 4071 50  0001 R CNN
-F 2 "Diode_THT:D_DO-35_SOD27_P7.62mm_Horizontal" H 2650 3975 50  0001 C CNN
-F 3 "http://www.nxp.com/documents/data_sheet/1N4148_1N4448.pdf" H 2650 4150 50  0001 C CNN
-	1    2650 4150
-	0    -1   -1   0
-$EndComp
-Connection ~ 2950 4000
-Wire Wire Line
-	2950 4000 3400 4000
-Wire Wire Line
-	2650 4000 2950 4000
-$Comp
 L Device:C_Small C?
 U 1 1 5F618EFF
@@
 Text Label 6550 3800 0    50   ~ 0
 I_adc
-Wire Wire Line
-	2650 4000 2450 4000
-Connection ~ 2650 4000
 Text HLabel 2450 4000 0    50   Input ~ 0
 in
@@
 Wire Wire Line
 	4900 3950 4900 3900
+$Comp
+L Diode:1N4448WS D?
+U 1 1 5FE19E0E
+P 2950 4150
+F 0 "D?" V 2904 4230 50  0000 L CNN
+F 1 "1N4448WS" V 2995 4230 50  0000 L CNN
+F 2 "Diode_SMD:D_SOD-323" H 2950 3975 50  0001 C CNN
+F 3 "https://www.vishay.com/docs/81387/1n4448ws.pdf" H 2950 4150 50  0001 C CNN
+	1    2950 4150
+	0    1    1    0
+$EndComp
+Wire Wire Line
+	2450 4000 2650 4000
+Connection ~ 2950 4000
+Wire Wire Line
+	2950 4000 3400 4000
+$Comp
+L Diode:1N4448WS D?
+U 1 1 5FE19EDD
+P 2650 4150
+F 0 "D?" V 2650 4070 50  0000 R CNN
+F 1 "1N4448WS" V 2605 4070 50  0001 R CNN
+F 2 "Diode_SMD:D_SOD-323" H 2650 3975 50  0001 C CNN
+F 3 "https://www.vishay.com/docs/81387/1n4448ws.pdf" H 2650 4150 50  0001 C CNN
+	1    2650 4150
+	0    -1   -1   0
+$EndComp
+Connection ~ 2650 4000
+Wire Wire Line
+	2650 4000 2950 4000
 $EndSCHEMATC

Commit message: - high side (supply, MCU) - low side MCU - much small changes
Parts:
- removed C?: 1n, symbol Device:C_Small
- added C? (x2): 100p, Capacitor_SMD:C_0603_1608Metric_Pad1.05x0.95mm_HandSolder, symbol Device:C_Small
- added R?: 100k, Resistor_SMD:R_0603_1608Metric_Pad1.05x0.95mm_HandSolder, symbol Device:R_Small
- added R?: 1k, Resistor_SMD:R_0603_1608Metric_Pad1.05x0.95mm_HandSolder, symbol Device:R_Small
- C?: value 100n -> 100p; footprint (none) -> Capacitor_SMD:C_0603_1608Metric_Pad1.05x0.95mm_HandSolder
- R? (x3): footprint (none) -> Resistor_SMD:R_0603_1608Metric_Pad1.05x0.95mm_HandSolder; symbol Device:R -> Device:R_Small
- R?: value 100R -> 1k; footprint (none) -> Resistor_SMD:R_0603_1608Metric_Pad1.05x0.95mm_HandSolder; symbol Device:R -> Device:R_Small
Connections:
- net in: now also R?.1; no longer U?.2 (-)
- net outAdc: now also R?.2; no longer R?.2, U?.7
- net at R?.1, U?.1: now also C?.1
- net at C?.1, Q?.2 (E), Q?.2 (E)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: now also C?.1
- net at Q?.1 (B), Q?.1 (B), R?.2: now also C?.2
- new net: C?.2, R?.2, U?.2 (-)
- new net I_adc: R?.1, R?.2, U?.7
Other:
- moved on the sheet: D?, Q?, R?, U?B, U?C

Commit message: - final schematic
Parts:
- added C25, C28: 100n, Capacitor_SMD:C_0603_1608Metric_Pad1.05x0.95mm_HandSolder, symbol Device:C_Small
- added L7, L8: BLM18RK102, Resistor_SMD:R_0805_2012Metric_Pad1.15x1.40mm_HandSolder, symbol Device:L_Core_Ferrite_Small
- D3, D4: renamed from D?; footprint Diode_SMD:D_SOD-323 -> miscellaneous_my:D_SOD-323-523-SMA_Universal_Handsoldering
- U12: renamed from U?; footprint (none) -> miscellaneous_my:SO8-MSOP8_3x3mm_P0.65mm
- gave numbers to parts that had none: 12
Connections:
- net +5V: now also L7.2; no longer U12.8 (V+)
- net -5V: now also L8.1; no longer U12.4 (V-)
- net GND: now also C25.1, C28.2
- net in renamed current_in
- new net: C28.1, L8.2, U12.4 (V-)
- new net: C25.2, L7.1, U12.8 (V+)
Other:
- moved on the sheet: U12C

Commit message: - init PCB - fix last things in schematic
Parts:
- added C201, C202: 100n, Capacitor_SMD:C_0603_1608Metric_Pad1.05x0.95mm_HandSolder, symbol Device:C_Small
- added R14, R196, R197, R198, R200: 100k, Resistor_SMD:R_0603_1608Metric_Pad1.05x0.95mm_HandSolder, symbol Device:R_Small
- added R199: 0R, Resistor_SMD:R_0603_1608Metric_Pad1.05x0.95mm_HandSolder, symbol Device:R_Small
- added R201: 100k, Resistor_THT:R_Axial_DIN0207_L6.3mm_D2.5mm_P10.16mm_Horizontal, symbol Device:R_Small
- added U5: INA128, Package_SO:SO-8_3.9x4.9mm_P1.27mm, symbol Amplifier_Instrumentation:INA128
- U12: footprint (none) -> miscellaneous_my:SO8-MSOP8_3x3mm_P0.65mm
Connections:
- net +5V: no longer Q3.3 (C)
- net -5V: no longer Q4.3 (C)
- net GND: now also C201.2, C202.1, U5.5 (Ref)
- net I_adc: now also R199.2
- net current_in: now also R198.2, R200.2, R201.2; no longer C29.2, D3.2 (A), D4.1 (K), R32.1, R34.1
- net VEE: now reaches C28.1, L8.2, U12.4 (V-)
- net VEE: now also Q4.3 (C), C202.2, U5.4 (V-)
- net VCC: now reaches C25.2, L7.1, U12.8 (V+)
- net VCC: now also Q3.3 (C), C201.1, U5.7 (V+)
- new net: C29.2, D3.2 (A), D4.1 (K), R14.2, R200.1, R201.1, R32.1, R34.1
- new net: R196.1, R197.1, U5.1 (Rg)
- new net: R198.1, U5.2 (-)
- new net: R14.1, U5.3 (+)
- new net: R199.1, U5.6
- new net: R196.2, R197.2, U5.8 (Rg)
Other:
- note added: "Alternate circuit"
- note added: "Primary circuit"

Commit message: - PCB progress
Parts:
- added R204: 10k, Resistor_SMD:R_1206_3216Metric, symbol Device:R_Small
- C201, C202, C25, C26, C27, C28: footprint Capacitor_SMD:C_0603_1608Metric_Pad1.05x0.95mm_HandSolder -> Capacitor_SMD:C_0603_1608Metric
- L7, L8: footprint Resistor_SMD:R_0805_2012Metric_Pad1.15x1.40mm_HandSolder -> Inductor_SMD:L_0603_1608Metric
- R14, R29, R30, R31, R33: footprint Resistor_SMD:R_0603_1608Metric_Pad1.05x0.95mm_HandSolder -> Resistor_SMD:R_0603_1608Metric
Connections:
- net at C29.2, D3.2 (A), D4.1 (K)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: now also R204.1
- net at C26.1, C29.1, Q3.2 (E)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: now also R204.2
Changed lines of the file:
@@
 F 0 "R30" V 4550 3900 50  0000 C CNN
 F 1 "1k" V 4350 3900 50  0000 C CNN
-F 2 "Resistor_SMD:R_0603_1608Metric_Pad1.05x0.95mm_HandSolder" V 4380 3900 50  0001 C CNN
+F 2 "Resistor_SMD:R_0603_1608Metric" V 4380 3900 50  0001 C CNN
 F 3 "~" H 4450 3900 50  0001 C CNN
 	1    4450 3900
@@
 F 0 "R31" V 5950 3900 50  0000 C CNN
 F 1 "47k" V 5750 3900 50  0000 C CNN
-F 2 "Resistor_SMD:R_0603_1608Metric_Pad1.05x0.95mm_HandSolder" V 5780 3900 50  0001 C CNN
+F 2 "Resistor_SMD:R_0603_1608Metric" V 5780 3900 50  0001 C CNN
 F 3 "~" H 5850 3900 50  0001 C CNN
 	1    5850 3900
@@
 F 0 "R33" V 6550 4150 50  0000 C CNN
 F 1 "47k" V 6350 4150 50  0000 C CNN
-F 2 "Resistor_SMD:R_0603_1608Metric_Pad1.05x0.95mm_HandSolder" V 6380 4150 50  0001 C CNN
+F 2 "Resistor_SMD:R_0603_1608Metric" V 6380 4150 50  0001 C CNN
 F 3 "~" H 6450 4150 50  0001 C CNN
 	1    6450 4150
@@
 F 0 "C27" V 3750 4150 50  0000 R CNN
 F 1 "100p" V 3750 4250 50  0000 L CNN
-F 2 "Capacitor_SMD:C_0603_1608Metric_Pad1.05x0.95mm_HandSolder" H 3800 4200 50  0001 C CNN
+F 2 "Capacitor_SMD:C_0603_1608Metric" H 3800 4200 50  0001 C CNN
 F 3 "~" H 3800 4200 50  0001 C CNN
 	1    3800 4200
@@
 F 0 "C26" V 4850 3850 50  0000 R CNN
 F 1 "100p" V 4850 3950 50  0000 L CNN
-F 2 "Capacitor_SMD:C_0603_1608Metric_Pad1.05x0.95mm_HandSolder" H 4900 3900 50  0001 C CNN
+F 2 "Capacitor_SMD:C_0603_1608Metric" H 4900 3900 50  0001 C CNN
 F 3 "~" H 4900 3900 50  0001 C CNN
 	1    4900 3900
@@
 F 0 "R29" V 7300 3800 50  0000 C CNN
 F 1 "1k" V 7100 3800 50  0000 C CNN
-F 2 "Resistor_SMD:R_0603_1608Metric_Pad1.05x0.95mm_HandSolder" V 7130 3800 50  0001 C CNN
+F 2 "Resistor_SMD:R_0603_1608Metric" V 7130 3800 50  0001 C CNN
 F 3 "~" H 7200 3800 50  0001 C CNN
 	1    7200 3800
@@
 F 0 "C25" H 8350 3900 50  0000 L CNN
 F 1 "100n" H 8350 3800 50  0000 L CNN
-F 2 "Capacitor_SMD:C_0603_1608Metric_Pad1.05x0.95mm_HandSolder" H 8250 3850 50  0001 C CNN
+F 2 "Capacitor_SMD:C_0603_1608Metric" H 8250 3850 50  0001 C CNN
 F 3 "~" H 8250 3850 50  0001 C CNN
 	1    8250 3850
@@
 F 0 "L7" V 8855 3750 50  0000 C CNN
 F 1 "BLM18RK102" V 8764 3750 50  0000 C CNN
-F 2 "Resistor_SMD:R_0805_2012Metric_Pad1.15x1.40mm_HandSolder" H 8650 3750 50  0001 C CNN
+F 2 "Inductor_SMD:L_0603_1608Metric" H 8650 3750 50  0001 C CNN
 F 3 "~" H 8650 3750 50  0001 C CNN
 	1    8650 3750
@@
 F 0 "C28" H 8350 4300 50  0000 L CNN
 F 1 "100n" H 8350 4200 50  0000 L CNN
-F 2 "Capacitor_SMD:C_0603_1608Metric_Pad1.05x0.95mm_HandSolder" H 8250 4250 50  0001 C CNN
+F 2 "Capacitor_SMD:C_0603_1608Metric" H 8250 4250 50  0001 C CNN
 F 3 "~" H 8250 4250 50  0001 C CNN
 	1    8250 4250
@@
 F 0 "L8" V 8855 4350 50  0000 C CNN
 F 1 "BLM18RK102" V 8764 4350 50  0000 C CNN
-F 2 "Resistor_SMD:R_0805_2012Metric_Pad1.15x1.40mm_HandSolder" H 8650 4350 50  0001 C CNN
+F 2 "Inductor_SMD:L_0603_1608Metric" H 8650 4350 50  0001 C CNN
 F 3 "~" H 8650 4350 50  0001 C CNN
 	1    8650 4350
@@
 F 0 "C201" H 4750 1600 50  0000 L CNN
 F 1 "100n" H 4750 1500 50  0000 L CNN
-F 2 "Capacitor_SMD:C_0603_1608Metric_Pad1.05x0.95mm_HandSolder" H 4650 1550 50  0001 C CNN
+F 2 "Capacitor_SMD:C_0603_1608Metric" H 4650 1550 50  0001 C CNN
 F 3 "~" H 4650 1550 50  0001 C CNN
 	1    4650 1550
@@
 F 0 "C202" H 4500 2550 50  0000 L CNN
 F 1 "100n" H 4500 2450 50  0000 L CNN
-F 2 "Capacitor_SMD:C_0603_1608Metric_Pad1.05x0.95mm_HandSolder" H 4400 2500 50  0001 C CNN
+F 2 "Capacitor_SMD:C_0603_1608Metric" H 4400 2500 50  0001 C CNN
 F 3 "~" H 4400 2500 50  0001 C CNN
 	1    4400 2500
@@
 F 0 "R14" V 2800 1800 50  0000 C CNN
 F 1 "100k" V 2600 1800 50  0000 C CNN
-F 2 "Resistor_SMD:R_0603_1608Metric_Pad1.05x0.95mm_HandSolder" V 2630 1800 50  0001 C CNN
+F 2 "Resistor_SMD:R_0603_1608Metric" V 2630 1800 50  0001 C CNN
 F 3 "~" H 2700 1800 50  0001 C CNN
 	1    2700 1800
@@
 Wire Wire Line
 	6800 3300 6800 3800
+$Comp
+L Device:R_Small R?
+U 1 1 5FA9EA22
+P 4200 5000
+AR Path="/5F40DCB9/5FA9EA22" Ref="R?"  Part="1"
+AR Path="/5F618AB9/5FA9EA22" Ref="R204"  Part="1"
+F 0 "R204" V 4300 5000 50  0000 C CNN
+F 1 "10k" V 4100 5000 50  0000 C CNN
+F 2 "Resistor_SMD:R_1206_3216Metric" V 4130 5000 50  0001 C CNN
+F 3 "~" H 4200 5000 50  0001 C CNN
+	1    4200 5000
+	0    -1   -1   0
+$EndComp
+Wire Wire Line
+	4100 5000 4000 5000
+Wire Wire Line
+	4000 4700 4000 5000
+Wire Wire Line
+	4400 5000 4400 4700
+Wire Wire Line
+	4300 5000 4400 5000
 $EndSCHEMATC
