File: rippleMeas.sch (KiCad schematic (older format))
At the start: 32 parts, among them U10 LMC6482

Commit message: - final schematic
Parts:
- gave numbers to parts that had none: 30
- renumbered DMM to DMM1

Commit message: - init PCB - fix last things in schematic
Parts:
- removed DMM1: (10M), miscellaneous_my:Virtual_noFootprint, symbol Device:Voltmeter_DC
- removed Liion1, Liion2: 4.0V, miscellaneous_my:Virtual_noFootprint, symbol Device:Battery_Cell
- removed Load1: 17M, miscellaneous_my:Virtual_noFootprint, symbol Device:R
- removed R14: 68M, miscellaneous_my:Virtual_noFootprint, symbol Device:R
- removed SW1: RST, Button_Switch_SMD:SW_Push_1P1T_NO_6x6mm_H9.5mm, symbol Switch:SW_MEC_5E
- removed TP12: TestPoint_Probe, miscellaneous_my:Virtual_noFootprint, symbol Connector:TestPoint_Probe
- removed U7: HVDC, miscellaneous_my:Virtual_noFootprint, symbol uScope:APD_P2_single
- added SW1: RST, Button_Switch_SMD:SW_Push_1P1T_NO_6x6mm_H9.5mm, symbol Switch:SW_Push
- C7, C9: footprint (none) -> Capacitor_SMD:C_0603_1608Metric_Pad1.05x0.95mm_HandSolder
- U10: footprint (none) -> Package_SO:SO-8_3.9x4.9mm_P1.27mm
Connections:
- net at C10.2, C12.1, D1.1 (K)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: now also SW1.1
- net at R16.1: now also SW1.2
Changed lines of the file:
@@
 Wire Wire Line
 	5200 4600 4900 4600
-Wire Wire Line
-	4400 4950 4400 4850
 Connection ~ 4400 4600
 Wire Wire Line
@@
 F 0 "U10" H 9050 4267 50  0000 C CNN
 F 1 "LMC6482" H 9050 4176 50  0000 C CNN
-F 2 "" H 9050 3900 50  0001 C CNN
+F 2 "Package_SO:SO-8_3.9x4.9mm_P1.27mm" H 9050 3900 50  0001 C CNN
 F 3 "http://www.ti.com/lit/ds/symlink/lmc6482.pdf" H 9050 3900 50  0001 C CNN
 	2    9050 3900
@@
 F 0 "U10" H 6850 3900 50  0000 R CNN
 F 1 "LMC6482" H 6850 3800 50  0001 R CNN
-F 2 "" H 7000 3850 50  0001 C CNN
+F 2 "Package_SO:SO-8_3.9x4.9mm_P1.27mm" H 7000 3850 50  0001 C CNN
 F 3 "http://www.ti.com/lit/ds/symlink/lmc6482.pdf" H 7000 3850 50  0001 C CNN
 	3    7000 3850
-	1    0    0    -1
-$EndComp
-$Comp
-L Device:Battery_Cell Liion1
-U 1 1 5F71611B
-P 7600 3750
-F 0 "Liion1" H 7718 3846 50  0000 L CNN
-F 1 "4.0V" H 7718 3755 50  0000 L CNN
-F 2 "miscellaneous_my:Virtual_noFootprint" V 7600 3810 50  0001 C CNN
-F 3 "~" V 7600 3810 50  0001 C CNN
-	1    7600 3750
-	1    0    0    -1
-$EndComp
-$Comp
-L Device:Battery_Cell Liion2
-U 1 1 5F716305
-P 7600 4050
-F 0 "Liion2" H 7718 4146 50  0000 L CNN
-F 1 "4.0V" H 7718 4055 50  0000 L CNN
-F 2 "miscellaneous_my:Virtual_noFootprint" V 7600 4110 50  0001 C CNN
-F 3 "~" V 7600 4110 50  0001 C CNN
-	1    7600 4050
 	1    0    0    -1
 $EndComp
@@
 $EndComp
 Wire Wire Line
-	7950 3850 7600 3850
-Connection ~ 7600 3850
-Wire Wire Line
 	7600 4150 7500 4150
 Wire Wire Line
@@
 F 0 "C7" H 7250 3600 50  0000 R CNN
 F 1 "100n" H 7250 3800 50  0000 R CNN
-F 2 "" H 7250 3700 50  0001 C CNN
+F 2 "Capacitor_SMD:C_0603_1608Metric_Pad1.05x0.95mm_HandSolder" H 7250 3700 50  0001 C CNN
 F 3 "~" H 7250 3700 50  0001 C CNN
 	1    7250 3700
@@
 F 0 "C9" H 7250 3900 50  0000 R CNN
 F 1 "100n" H 7250 4100 50  0000 R CNN
-F 2 "" H 7250 4000 50  0001 C CNN
+F 2 "Capacitor_SMD:C_0603_1608Metric_Pad1.05x0.95mm_HandSolder" H 7250 4000 50  0001 C CNN
 F 3 "~" H 7250 4000 50  0001 C CNN
 	1    7250 4000
 	1    0    0    -1
 $EndComp
-Wire Wire Line
-	7600 3850 7250 3850
 Wire Wire Line
 	7250 3850 7250 3800
@@
 	4950 3650 4950 3750
 Connection ~ 5200 4600
-$Comp
-L Connector:TestPoint_Probe TP12
-U 1 1 5F76997E
-P 6850 4600
-F 0 "TP12" H 7003 4702 50  0000 L CNN
-F 1 "TestPoint_Probe" H 7003 4611 50  0000 L CNN
-F 2 "miscellaneous_my:Virtual_noFootprint" H 7050 4600 50  0001 C CNN
-F 3 "~" H 7050 4600 50  0001 C CNN
-	1    6850 4600
-	1    0    0    -1
-$EndComp
 Connection ~ 6500 4600
-$Comp
-L uScope:APD_P2_single U?
-U 2 1 5F76F947
-P 2800 4450
-AR Path="/5F76F947" Ref="U?"  Part="2"
-AR Path="/5F463F4C/5F76F947" Ref="U7"  Part="2"
-F 0 "U7" H 2650 4500 50  0000 R CNN
-F 1 "HVDC" H 2650 4400 50  0000 R CNN
-F 2 "miscellaneous_my:Virtual_noFootprint" H 2800 4450 50  0001 C CNN
-F 3 "" H 2800 4450 50  0001 C CNN
-	2    2800 4450
-	1    0    0    -1
-$EndComp
-$Comp
-L power:GND #PWR?
-U 1 1 5F76F94E
-P 2800 4900
-AR Path="/5F40DCB9/5F76F94E" Ref="#PWR?"  Part="1"
-AR Path="/5F463F4C/5F76F94E" Ref="#PWR015"  Part="1"
-AR Path="/5F76F94E" Ref="#PWR?"  Part="1"
-F 0 "#PWR015" H 2800 4740 50  0001 C CNN
-F 1 "GND" V 2800 4823 39  0000 R CNN
-F 2 "" H 2800 4900 50  0001 C CNN
-F 3 "" H 2800 4900 50  0001 C CNN
-	1    2800 4900
-	1    0    0    -1
-$EndComp
-$Comp
-L Device:R R?
-U 1 1 5F76F954
-P 3650 4350
-AR Path="/5F40DCB9/5F76F954" Ref="R?"  Part="1"
-AR Path="/5F463F4C/5F76F954" Ref="Load1"  Part="1"
-F 0 "Load1" H 3600 4400 50  0000 R CNN
-F 1 "17M" H 3600 4300 50  0000 R CNN
-F 2 "miscellaneous_my:Virtual_noFootprint" V 3580 4350 50  0001 C CNN
-F 3 "~" H 3650 4350 50  0001 C CNN
-	1    3650 4350
-	1    0    0    -1
-$EndComp
-$Comp
-L power:GND #PWR?
-U 1 1 5F76F95B
-P 3650 4900
-AR Path="/5F40DCB9/5F76F95B" Ref="#PWR?"  Part="1"
-AR Path="/5F463F4C/5F76F95B" Ref="#PWR017"  Part="1"
-AR Path="/5F76F95B" Ref="#PWR?"  Part="1"
-F 0 "#PWR017" H 3650 4740 50  0001 C CNN
-F 1 "GND" V 3650 4823 39  0000 R CNN
-F 2 "" H 3650 4900 50  0001 C CNN
-F 3 "" H 3650 4900 50  0001 C CNN
-	1    3650 4900
-	1    0    0    -1
-$EndComp
-Wire Wire Line
-	3650 4500 3650 4900
-$Comp
-L Device:Voltmeter_DC DMM1
-U 1 1 5F776F80
-P 3200 4700
-F 0 "DMM1" H 3353 4746 50  0000 L CNN
-F 1 "(10M)" H 3353 4655 50  0000 L CNN
-F 2 "miscellaneous_my:Virtual_noFootprint" V 3200 4800 50  0001 C CNN
-F 3 "~" V 3200 4800 50  0001 C CNN
-	1    3200 4700
-	1    0    0    -1
-$EndComp
-$Comp
-L Device:R Load?
-U 1 1 5F77AA20
-P 3200 4350
-AR Path="/5F40DCB9/5F77AA20" Ref="Load?"  Part="1"
-AR Path="/5F463F4C/5F77AA20" Ref="R14"  Part="1"
-F 0 "R14" H 3150 4400 50  0001 R CNN
-F 1 "68M" H 3150 4300 50  0000 R CNN
-F 2 "miscellaneous_my:Virtual_noFootprint" V 3130 4350 50  0001 C CNN
-F 3 "~" H 3200 4350 50  0001 C CNN
-	1    3200 4350
-	1    0    0    -1
-$EndComp
-$Comp
-L power:GND #PWR?
-U 1 1 5F77E720
-P 3200 4900
-AR Path="/5F40DCB9/5F77E720" Ref="#PWR?"  Part="1"
-AR Path="/5F463F4C/5F77E720" Ref="#PWR016"  Part="1"
-AR Path="/5F77E720" Ref="#PWR?"  Part="1"
-F 0 "#PWR016" H 3200 4740 50  0001 C CNN
-F 1 "GND" V 3200 4823 39  0000 R CNN
-F 2 "" H 3200 4900 50  0001 C CNN
-F 3 "" H 3200 4900 50  0001 C CNN
-	1    3200 4900
-	1    0    0    -1
-$EndComp
-Wire Wire Line
-	2800 4900 2800 4700
-Wire Wire Line
-	2800 4200 3200 4200
-Connection ~ 3200 4200
-Wire Wire Line
-	3200 4200 3650 4200
 Wire Wire Line
 	3750 4050 3650 4050
-Wire Wire Line
-	3650 4050 3650 4200
-Connection ~ 3650 4200
 Connection ~ 4400 3650
 Connection ~ 4550 3650
@@
 Wire Wire Line
 	3950 4050 4400 4050
-Wire Wire Line
-	6500 4600 6850 4600
 $Comp
 L Connector:TestPoint TP?
@@
 	1    0    0    -1
 $EndComp
-Connection ~ 3650 4050
 $Comp
 L Device:C_Small C?
@@
 Wire Wire Line
 	5900 3850 5850 3850
-$Comp
-L Switch:SW_MEC_5E SW?
-U 1 1 5FA40568
-P 4600 4950
-AR Path="/5F7A93EE/5FA40568" Ref="SW?"  Part="1"
-AR Path="/5F7D6767/5FA40568" Ref="SW?"  Part="1"
-AR Path="/5F463F4C/5FA40568" Ref="SW1"  Part="1"
-F 0 "SW1" V 4650 5000 50  0000 R CNN
-F 1 "RST" V 4550 5000 50  0000 R CNN
-F 2 "Button_Switch_SMD:SW_Push_1P1T_NO_6x6mm_H9.5mm" H 4600 5250 50  0001 C CNN
-F 3 "http://www.apem.com/int/index.php?controller=attachment&id_attachment=1371" H 4600 5250 50  0001 C CNN
-F 4 "TL3301TF160QG" V 4600 4950 50  0001 C CNN "Mfr. No"
-F 5 "1.27" V 4600 4950 50  0001 C CNN "Price [PLN]"
-	1    4600 4950
-	1    0    0    -1
-$EndComp
-Wire Wire Line
-	4400 4600 4400 4850
-Connection ~ 4400 4850
 Wire Wire Line
 	4800 4950 4900 4950
-Wire Wire Line
-	4800 4950 4800 4850
-Connection ~ 4800 4950
 $Comp
 L Connector:TestPoint TP?
@@
 	1    0    0    -1
 $EndComp
-Connection ~ 7600 3550
 $Comp
 L Device:R_Small R?
@@
 	-1   0    0    1
 $EndComp
-Connection ~ 7600 4150
 $Comp
 L Connector:TestPoint TP?
@@
 $EndComp
 Connection ~ 7950 3850
+$Comp
+L power:PWR_FLAG #FLG0101
+U 1 1 5FA25CAA
+P 6900 3550
+F 0 "#FLG0101" H 6900 3625 50  0001 C CNN
+F 1 "PWR_FLAG" H 6900 3724 50  0001 C CNN
+F 2 "" H 6900 3550 50  0001 C CNN
+F 3 "~" H 6900 3550 50  0001 C CNN
+	1    6900 3550
+	0    -1   -1   0
+$EndComp
+Connection ~ 6900 3550
+$Comp
+L power:PWR_FLAG #FLG0102
+U 1 1 5FA25F10
+P 6900 4150
+F 0 "#FLG0102" H 6900 4225 50  0001 C CNN
+F 1 "PWR_FLAG" H 6900 4324 50  0001 C CNN
+F 2 "" H 6900 4150 50  0001 C CNN
+F 3 "~" H 6900 4150 50  0001 C CNN
+	1    6900 4150
+	0    -1   -1   0
+$EndComp
+Connection ~ 6900 4150
+Wire Wire Line
+	7250 3850 7950 3850
+$Comp
+L Switch:SW_Push SW?
+U 1 1 5FBF43A4
+P 4600 4950
+AR Path="/5F7D6767/5FBF43A4" Ref="SW?"  Part="1"
+AR Path="/5F463F4C/5FBF43A4" Ref="SW1"  Part="1"
+F 0 "SW1" V 4650 4900 50  0000 R CNN
+F 1 "RST" V 4550 4900 50  0000 R CNN
+F 2 "Button_Switch_SMD:SW_Push_1P1T_NO_6x6mm_H9.5mm" H 4600 5150 50  0001 C CNN
+F 3 "~" H 4600 5150 50  0001 C CNN
+	1    4600 4950
+	1    0    0    -1
+$EndComp
+Wire Wire Line
+	4400 4600 4400 4950
 $EndSCHEMATC

Commit message: - PCB progress
Parts:
- added C203, C204: 1u, Capacitor_SMD:C_0603_1608Metric, symbol Device:C_Small
- added R127: 6M8, Resistor_SMD:R_1206_3216Metric_Pad1.42x1.75mm_HandSolder, symbol Device:R_Small
- added R179, R202, R203: 1M, Resistor_SMD:R_0603_1608Metric_Pad1.05x0.95mm_HandSolder, symbol Device:R_Small
- added R205: 100R, Resistor_SMD:R_0603_1608Metric, symbol Device:R_Small
- added R206, R207: 47k, Resistor_SMD:R_0603_1608Metric, symbol Device:R_Small
- added TP12: TestPoint, TestPoint:TestPoint_THTPad_D1.5mm_Drill0.7mm, symbol Connector:TestPoint
- C11, C7, C8, C9: footprint Capacitor_SMD:C_0603_1608Metric_Pad1.05x0.95mm_HandSolder -> Capacitor_SMD:C_0603_1608Metric
- C12: value 346n -> 100n
- R10, R11, R12, R13, R16: footprint Resistor_SMD:R_0603_1608Metric_Pad1.05x0.95mm_HandSolder -> Resistor_SMD:R_0603_1608Metric
Connections:
- net GND: now also C203.2, C204.1
- net at C10.2, C12.1, D1.1 (K)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: now also R179.1
- net at C12.2, C8.1, Q1.2 (E)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: now also R127.2, R203.2, R206.1; no longer R15.2
- net at U10.6 (-): now also R206.2, R207.1; no longer U10.7
- net at C9.2, Q2.3 (C), R13.1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: now also C204.2
- net at C7.1, Q1.3 (C), R10.1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: now also C203.1
- new net: R127.1, R15.2
- new net: R205.1, R207.2, U10.7
- new net: R179.2, R202.1
- new net: R202.2, R203.1
- new net: R205.2, TP12.1
Other:
- moved on the sheet: C12, R10, R13, R15, R16, SW1, TP10, TP5, U10B
