File: uScope.kicad_pcb (KiCad board)
At the start: 2 copper layers, 595 parts, among them J1 Pump+, J10 Nucleo_SWD, J11 STLinkV2, J12 Nucleo_SWD, J2 Pump-, J3 U_E, J4 U_F, J5 Conn_01x02, J6 U_K, J7 Anode, J8 USB_B_Micro, J9 STLinkV2, Q1 BC817, Q10 BC817, Q11 BC807, Q12 BSS138, Q13 BSS138, Q14 BSS138, Q15 BSS138, Q16 BSS138, Q17 BSS138, Q18 BSS138, Q19 BSS138, Q2 MMST3906, Q20 BSS138, Q21 BC817, Q3 BC817, Q4 BC807, Q5 BUK98150-55A, Q6 BUK98150-55A, Q7 BUK98150-55A, Q8 BUK98150-55A, Q9 BSS84, SW1 RST, SW10 ESC, SW11 RST, SW2 set_current, SW3 PWRON, SW4 RST, SW5 Encoder, SW6 X, SW7 UP, SW8 DOWN, SW9 ENTER, U1 K, U10 LMC6482, U11 LMC6482, U12 LMC6482, U13 LM321, U14 DAC8564, U15 LM321, U16 LM321, U17 LM321, U18 LM317L_SOT89, U19 PAM242x, U2 E, U20 LM337L_SO8, U21 TPS613222ADBV, U22 LP2985-3.3, U23 BQ24079RGT, U24 Holder 2x18650, U25 LCD_I2C, U26 STM32L431RBTx, U27 ADS131M06, U28 OPTI128, U29 QSE159, U3 F, U30 SN74LVC1G14DRL, U31 QSE159, U32 SN74LVC1G14DRL, U33 ADS131M06, U34 STM32L431RBTx, U35 LM317L_SOT89, U36 LP2985-3.3, U37 TL432, U38 TC7660S, U39 LM337L_SO8, U4 Pump, U5 INA128, U6 RHV2-1212S/R20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

Commit message: - first segregation on pcb
Parts:
- C30, C39, C43, C52, C54, C63, C64, C73: footprint Capacitor_SMD:C_0805_2012Metric_Pad1.15x1.40mm_HandSolder -> Capacitor_SMD:C_0603_1608Metric_Pad1.05x0.95mm_HandSolder
- moved R3 564.1 mm to (550.4, -54.4)
- moved GD1 563.3 mm to (537.9, -59.5)
- moved R2 563.3 mm to (533.9, -54.2)
- moved J5 557.0 mm to (539.2, -65.3), turned to 270 degrees
- moved TP1 527.5 mm to (527.6, -79.8)
- moved TP2 475.9 mm to (540.5, -76.5)
- moved TP4 439.2 mm to (529.1, -38.6)
- moved TP3 438.4 mm to (546.1, -39.4)
- moved R1 426.2 mm to (514.6, -54.4)
- moved J1 423.9 mm to (503.5, -61.8)
- moved J2 423.9 mm to (497.4, -61.8)
- moved R6 401.6 mm to (442.5, 51.1), turned to 90 degrees
- moved R7 393.2 mm to (442.5, 37.6), turned to 90 degrees
- moved U3 388.7 mm to (445.8, 52.8), turned to 90 degrees
- moved J4 374.3 mm to (442.5, 17.8), turned to 180 degrees
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
Commit message: - pcb placement, add 3dShapes
Parts:
- TP1, TP4: footprint miscellaneous_my:Socket_banana4mm -> miscellaneous_my:Banana4mmSocket_black
- TP2, TP3: footprint miscellaneous_my:Socket_banana4mm -> miscellaneous_my:Banana4mmSocket_red
- Y3, Y4: footprint Crystal:Crystal_AT310_D3.0mm_L10.0mm_Horizontal_1EP_style2 -> Crystal:Crystal_HC49-4H_Vertical
- moved R128 219.9 mm to (45.7, 23.6), turned to 90 degrees
- moved TP17 215.9 mm to (-56.6, 193.5)
- moved R129 215.3 mm to (39.6, 23.6), turned to 270 degrees
- moved Q16 214.4 mm to (42.7, 18.5), turned to 180 degrees
- moved TP18 213.3 mm to (-56.6, 196.1)
- moved Q15 210.4 mm to (42.7, 23.6), turned to 180 degrees
- moved C137 200.0 mm to (-45.7, 186.9), turned to 180 degrees
- moved R138 199.6 mm to (-36.8, 123.2)
- moved TP16 196.8 mm to (-56.6, 191.0)
- moved R160 194.6 mm to (-49.5, 193.0)
- moved C139 190.2 mm to (-45.7, 191.0), turned to 180 degrees
- moved J10 188.4 mm to (37.6, 46.7)
- moved C131 182.5 mm to (-38.6, 198.9), turned to 270 degrees
- moved C138 176.7 mm to (-45.7, 189.0), turned to 180 degrees
- moved L13 176.5 mm to (-32.5, 199.4), turned to 180 degrees
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Routing:
- net Net-(C137-Pad2): track 0.00 -> 12.7 mm
- net Net-(C138-Pad2): track 0.00 -> 9.67 mm
- net Net-(C147-Pad2): track 0.00 -> 8.58 mm
- net Net-(C146-Pad2): track 0.00 -> 8.51 mm
- net Net-(C139-Pad2): track 0.00 -> 7.95 mm
- net Net-(C140-Pad2): track 0.00 -> 7.88 mm
- net Net-(R162-Pad1): track 0.00 -> 6.87 mm
- net Net-(R161-Pad1): track 0.00 -> 6.66 mm
- net Net-(R160-Pad1): track 0.00 -> 6.45 mm
- net Net-(R154-Pad1): track 0.00 -> 6.24 mm
Other:
- board text added: "+Amp-"
- board text added: "- Volt+"
- board text added: "Pump+"
- board text added: "Pump-"

Commit message: - PCB progress
Parts:
- removed C83: 100n, Capacitor_SMD:C_0603_1608Metric_Pad1.05x0.95mm_HandSolder
- removed C96: 1u, Capacitor_SMD:C_0805_2012Metric_Pad1.15x1.40mm_HandSolder
- removed D13, D15: PMEG4005EJ, miscellaneous_my:D_SOD-323-523_HandSoldering
- removed R109: 1R, Resistor_SMD:R_0603_1608Metric_Pad1.05x0.95mm_HandSolder
- added C203: 1u, Capacitor_SMD:C_0603_1608Metric, F.Cu at (18.8, -28.2)
- added C204: 1u, Capacitor_SMD:C_0603_1608Metric, F.Cu at (15.7, -28.2)
- added R202: 1M, Resistor_SMD:R_0603_1608Metric_Pad1.05x0.95mm_HandSolder, F.Cu at (6.35, -27.2)
- added R203: 1M, Resistor_SMD:R_0603_1608Metric_Pad1.05x0.95mm_HandSolder, F.Cu at (9.65, -27.2)
- added R204: 10k, Resistor_SMD:R_1206_3216Metric, F.Cu at (122.3, 154.4)
- added R205: 100R, Resistor_SMD:R_0603_1608Metric, F.Cu at (25.1, -17.5)
- added R206: 47k, Resistor_SMD:R_0603_1608Metric, F.Cu at (23.6, -20.8)
- added R207: 47k, Resistor_SMD:R_0603_1608Metric, F.Cu at (23.6, -17.5)
- added TP12: TestPoint, TestPoint:TestPoint_THTPad_D1.5mm_Drill0.7mm, F.Cu at (28.7, -22.4)
- C1, C2, C3, C4, C5, C6: value 10n -> 3n3
- C100, C101, C184, C192, C198, C98, C99: footprint Capacitor_SMD:C_0805_2012Metric_Pad1.15x1.40mm_HandSolder -> Capacitor_SMD:C_0603_1608Metric_Pad1.05x0.95mm_HandSolder
- C102, C103, C104, C105, C106, C108, C109, C117, C118, C119, C120, C121, C122, C81, C82, C84, C87, C88, C89, C90: footprint Capacitor_SMD:C_0603_1608Metric_Pad1.05x0.95mm_HandSolder -> Capacitor_SMD:C_0603_1608Metric; moved to B.Cu
- C107, C199: footprint Capacitor_SMD:C_0805_2012Metric_Pad1.15x1.40mm_HandSolder -> Capacitor_SMD:C_0603_1608Metric_Pad1.05x0.95mm_HandSolder; moved to B.Cu
- C11, C110, C111, C116, C123, C124, C125, C126, C127, C128, C129, C13, C130, C131, C132, C133, C134, C135, C136, C137, C138, C139, C14, C140, C141, C142, C143, C144, C145, C146, C147, C148, C149, C150, C151, C152, C153, C154, C155, C156, C157, C158, C159, C160, C161, C162, C163, C164, C165, C166, C167, C168, C169, C17, C170, C171, C172, C173, C174, C175, C176, C177, C179, C18, C181, C182, C183, C185, C186, C187, C188, C189, C190, C191, C194, C195, C197, C201, C202, C21, C22, C25, C26, C27, C28, C30, C39, C40, C41, C42, C43, C52, C53, C54, C63, C64, C7, C73, C74, C76, C78, C8, C9, C93, C94: footprint Capacitor_SMD:C_0603_1608Metric_Pad1.05x0.95mm_HandSolder -> Capacitor_SMD:C_0603_1608Metric
- C112, C113, C114, C115, C178, C180, C193, C196, C75, C77, C95: footprint Capacitor_SMD:C_0805_2012Metric_Pad1.15x1.40mm_HandSolder -> Capacitor_SMD:C_0805_2012Metric
- C12: value 346n -> 100n
- C15, C16, C19, C20, C23, C24, C91: footprint Capacitor_SMD:C_0805_2012Metric_Pad1.15x1.40mm_HandSolder -> Capacitor_SMD:C_0603_1608Metric
- C85: footprint Capacitor_SMD:C_0805_2012Metric_Pad1.15x1.40mm_HandSolder -> Capacitor_SMD:C_0805_2012Metric; moved to B.Cu
- C97: footprint Capacitor_SMD:C_0805_2012Metric_Pad1.15x1.40mm_HandSolder -> Capacitor_SMD:C_0603_1608Metric; moved to B.Cu
- D12, D9, F2, F3, L10, R110, U19, U22: moved to B.Cu
- L1, L2, L3, L4, L5, L6, L7, L8, L9: footprint Resistor_SMD:R_0805_2012Metric_Pad1.15x1.40mm_HandSolder -> Inductor_SMD:L_0603_1608Metric
- L12, L13, L14, L15: footprint Resistor_SMD:R_0603_1608Metric_Pad1.05x0.95mm_HandSolder -> Inductor_SMD:L_0603_1608Metric
- R10, R100, R101, R102, R103, R104, R107, R11, R111, R112, R114, R115, R116, R117, R12, R120, R121, R122, R123, R124, R125, R126, R13, R14, R16, R18, R19, R20, R22, R23, R24, R26, R27, R28, R29, R30, R31, R33: footprint Resistor_SMD:R_0603_1608Metric_Pad1.05x0.95mm_HandSolder -> Resistor_SMD:R_0603_1608Metric
- R105, R106, R108: footprint Resistor_SMD:R_0603_1608Metric_Pad1.05x0.95mm_HandSolder -> Resistor_SMD:R_0603_1608Metric; moved to B.Cu
- R127: value 0R -> 6M8; footprint Resistor_SMD:R_0603_1608Metric_Pad1.05x0.95mm_HandSolder -> Resistor_SMD:R_1206_3216Metric_Pad1.42x1.75mm_HandSolder
- R179: value 0R -> 1M
- moved R179 413.0 mm to (3.05, -27.2)
- moved R15 381.4 mm to (3.81, -29.7)
- moved R13 373.4 mm to (15.7, -29.7)
- moved C12 370.0 mm to (2.29, -24.1)
- moved R12 367.6 mm to (9.65, -15.5), turned to 90 degrees
- moved TP6 367.6 mm to (23.6, -24.9)
- moved Q2 367.5 mm to (15.5, -25.7), turned to 90 degrees
- moved TP5 367.5 mm to (26.2, -27.4)
- moved R11 367.3 mm to (12.4, -23.1)
- moved R10 366.1 mm to (21.8, -28.2)
- moved TP7 364.3 mm to (26.2, -24.9)
- moved R16 364.1 mm to (8.89, -20.3), turned to 90 degrees
- moved C9 363.6 mm to (16.9, -14.0), turned to 180 degrees
- moved C7 363.6 mm to (20.3, -21.1), turned to 180 degrees
- moved TP11 362.8 mm to (26.2, -22.4)
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Connections:
- C152 pad 1: GND -> HVGND
- J12 pad 3: GND -> HVGND
- Q19 pad 2: GND -> HVGND
- Q20 pad 2: HVGND -> GND
- R127 pad 2: +3V3 -> Net-(C12-Pad2)
- R15 pad 2: Net-(C12-Pad2) -> Net-(R127-Pad1)
- R179 pad 1: Net-(R179-Pad1) -> Net-(C10-Pad2)
- R179 pad 2: HV+3V3 -> Net-(R179-Pad2)
- U10 pad 6: Net-(U10-Pad6) -> Net-(R206-Pad2)
- U10 pad 7: Net-(U10-Pad6) -> Net-(R205-Pad1)
- U26 pad 1: Net-(R127-Pad1) -> +3V3
- U34 pad 1: Net-(R179-Pad1) -> HV+3V3
Routing:
- net Net-(C10-Pad2): track 0.00 -> 38.2 mm
- net +12V: track 0.00 -> 26.5 mm, vias 0 -> 1
- net /MCU_high/SWD_IO: track 0.00 -> 24.6 mm
- net Net-(D30-Pad2): track 0.00 -> 24.0 mm
- net /MCU_high/SWD_CLK: track 0.00 -> 22.2 mm
- net HVGND: track 0.00 -> 19.9 mm
- net GND: track 0.00 -> 19.8 mm, vias 0 -> 6
- net Net-(C92-Pad1): track 0.00 -> 17.4 mm
- net Net-(C12-Pad2): track 0.00 -> 17.2 mm
- net +3V3: track 0.00 -> 15.7 mm, vias 0 -> 5
- net /MCU_high/SWD_SWO: track 0.00 -> 12.9 mm
- net +BATT: track 0.00 -> 12.9 mm
- net Net-(C15-Pad1): track 0.00 -> 10.5 mm
- net Net-(D9-Pad1): track 0.00 -> 10.2 mm
- net Net-(R16-Pad1): track 0.00 -> 10.0 mm
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Other:
- rule via_min_size: 0.4 -> 0.6

Commit message: - PCB WiP - Pump output aligned
Parts:
- added C83: 10u, Capacitor_SMD:C_0603_1608Metric_Pad1.05x0.95mm_HandSolder, F.Cu at (174.1, 104.5)
- added C96: 1n, Capacitor_SMD:C_0603_1608Metric, F.Cu at (101.5, 142.0)
- added R109: 10k, Resistor_SMD:R_0603_1608Metric_Pad1.05x0.95mm_HandSolder, F.Cu at (101.6, 140.5)
- added REF**: MountingHole_3.2mm_M3, MountingHole:MountingHole_3.2mm_M3, F.Cu at (446.5, 111.5)
- added REF**: MountingHole_3.2mm_M3, MountingHole:MountingHole_3.2mm_M3, F.Cu at (111.5, 18.5)
- added REF**: MountingHole_3.2mm_M3, MountingHole:MountingHole_3.2mm_M3, F.Cu at (18.5, 18.5)
- added REF**: MountingHole_3.2mm_M3, MountingHole:MountingHole_3.2mm_M3, F.Cu at (18.5, 111.5)
- added REF**: MountingHole_3.2mm_M3, MountingHole:MountingHole_3.2mm_M3, F.Cu at (138.5, 111.5)
- added REF**: MountingHole_3.2mm_M3, MountingHole:MountingHole_3.2mm_M3, F.Cu at (231.5, 111.5)
- added REF**: MountingHole_3.2mm_M3, MountingHole:MountingHole_3.2mm_M3, F.Cu at (138.5, 18.5)
- added REF**: MountingHole_3.2mm_M3, MountingHole:MountingHole_3.2mm_M3, F.Cu at (231.5, 18.5)
- added REF**: MountingHole_3.2mm_M3, MountingHole:MountingHole_3.2mm_M3, F.Cu at (446.5, 18.5)
- added REF**: MountingHole_3.2mm_M3, MountingHole:MountingHole_3.2mm_M3, F.Cu at (353.5, 18.5)
- added REF**: MountingHole_3.2mm_M3, MountingHole:MountingHole_3.2mm_M3, F.Cu at (353.5, 111.5)
- added REF**: MountingHole_3.2mm_M3, MountingHole:MountingHole_3.2mm_M3, F.Cu at (346.5, 111.5)
- added REF**: MountingHole_3.2mm_M3, MountingHole:MountingHole_3.2mm_M3, F.Cu at (346.5, 18.5)
- added REF**: MountingHole_3.2mm_M3, MountingHole:MountingHole_3.2mm_M3, F.Cu at (253.5, 18.5)
- added REF**: MountingHole_3.2mm_M3, MountingHole:MountingHole_3.2mm_M3, F.Cu at (253.5, 111.5)
- added REF**: MountingHole_3.2mm_M3, MountingHole:MountingHole_3.2mm_M3, F.Cu at (111.5, 111.5)
- C160, C161, C162, C163, C164, C181, C182, C183, C184, C185, C186, C189, C193, C194, C195, C196, D37, D38, GD1, R192, R194, U36, U39: moved to B.Cu
- C90, D12, R106, R108: moved to F.Cu
- R102, R107: footprint Resistor_SMD:R_0603_1608Metric -> Resistor_SMD:R_0603_1608Metric_Pad1.05x0.95mm_HandSolder
- R113, R128, R129, R130, R131, R132, R133, R135, R136, R139, R140, R141, R142, R143, R144, R145, R146, R147, R148, R149, R150, R151, R152, R153, R154, R155, R156, R157, R158, R159, R160, R161, R162, R163, R164, R165, R166, R167, R168, R169, R170, R171, R172, R173, R174, R175, R176, R177, R178, R180, R181, R182, R183, R184, R185, R186, R189, R190, R191, R198, R199, R45, R47, R50, R51, R61, R62, R63, R64, R66, R82, R84, R96, R98: footprint Resistor_SMD:R_0603_1608Metric_Pad1.05x0.95mm_HandSolder -> Resistor_SMD:R_0603_1608Metric
- R134, R137, R138: footprint Resistor_SMD:R_0603_1608Metric_Pad1.05x0.95mm_HandSolder -> Resistor_SMD:R_0603_1608Metric; moved to B.Cu
- moved SW3 264.9 mm to (53.5, 92.5), turned to 90 degrees
- moved U4 263.6 mm to (272.7, 86.2)
- moved J1 257.0 mm to (296.7, -30.0)
- moved J2 257.0 mm to (284.5, -30.0)
- moved TP2 256.8 mm to (275.6, -30.6)
- moved J5 252.0 mm to (268.6, -32.1)
- moved GD1 252.0 mm to (267.3, -26.3)
- moved R1 251.7 mm to (297.7, -7.24)
- moved R2 251.7 mm to (293.6, -11.3)
- moved TP4 251.7 mm to (258.6, -11.0)
- moved R3 251.7 mm to (289.6, -15.4)
- moved TP3 251.7 mm to (271.3, -11.0)
- moved TP1 248.6 mm to (259.0, -30.6)
- moved R8 219.2 mm to (486.4, 41.0)
- moved C5 218.3 mm to (490.3, 46.7)
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Connections:
- R32 pad 1: Net-(C29-Pad2) -> Net-(C96-Pad1)
Routing:
- net Net-(C191-Pad1): track 0.00 -> 30.1 mm
- net Net-(J1-Pad1): track 0.00 -> 26.2 mm
- net HV+3V3: track 0.00 -> 25.7 mm, vias 0 -> 5
- net Net-(GD1-Pad2): track 0.00 -> 20.9 mm
- net HV+5V: track 0.00 -> 20.7 mm
- net -5V: track 0.00 -> 17.0 mm
- net HV-5V: track 0.00 -> 16.8 mm
- net Net-(C189-Pad2): track 0.00 -> 14.4 mm
- net HVGND: track 19.9 -> 33.7 mm, vias 0 -> 5
- net Net-(C90-Pad2): track 0.00 -> 13.8 mm
- net HV+12V: track 0.00 -> 13.2 mm
- net Net-(Q15-Pad3): track 0.00 -> 11.6 mm
- net Net-(C187-Pad1): track 0.00 -> 11.6 mm
- net Net-(C188-Pad2): track 0.00 -> 10.3 mm
- net +5V: track 8.33 -> 18.5 mm
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Other:
- board text added: "-Pump+"
- board text added: "10MOhm multimeter 1:10 out"
- board text added: "DOWN"
- board text added: "ENTER"
- board text added: "ESC"
- board text added: "POWER"
- board text added: "UP"
- board text added: "X"
- board text added: "shortcircuit when n.c."
- board text removed: "Pump+"
- board text removed: "Pump-"

Commit message: - PCB WiP
Parts:
- C13, C14, C141, C143, C145, C15, C150, C151, C152, C16, C17, C18, C19, C20, C21, C22, C23, C24, L1, L2, L3, L4, L5, L6, R122, R131, R155, R157, R159, R163, R164, R165, R169, R18, R19, R20, R22, R23, R24, R26, R27, R28, U11, U24, U30, U32, U8, U9: moved to B.Cu
- D18, D19, D21, D23: footprint Diode_SMD:D_SOD-323 -> miscellaneous_my:D_SOD-323-523_HandSoldering
- R109, R32: footprint Resistor_SMD:R_0603_1608Metric_Pad1.05x0.95mm_HandSolder -> Resistor_SMD:R_0603_1608Metric
- R113: value 1k -> 47k
- moved C10 518.8 mm to (502.7, 48.0)
- moved C11 518.8 mm to (490.5, 36.1)
- moved C12 518.8 mm to (479.0, 31.2)
- moved C203 518.8 mm to (495.6, 27.2)
- moved C204 518.8 mm to (492.5, 27.2)
- moved C7 518.8 mm to (497.1, 34.3)
- moved C8 518.8 mm to (492.3, 32.3)
- moved C9 518.8 mm to (493.6, 41.4)
- moved D1 518.8 mm to (488.2, 39.9)
- moved D2 518.8 mm to (490.2, 39.9)
- moved Q1 518.8 mm to (495.8, 29.7)
- moved Q2 518.8 mm to (492.3, 29.7)
- moved R10 518.8 mm to (498.6, 27.2)
- moved R11 518.8 mm to (489.2, 32.3)
- moved R12 518.8 mm to (486.4, 39.9)
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Connections:
- net Net-(NTC1-Pad1) renamed /Battery_Charger/NTC
- Q12 pad 1: /Battery_Charger/Vusb -> Net-(Q12-Pad1)
- R113 pad 1: /Battery_Charger/Vusb -> Net-(Q12-Pad1)
- R113 pad 2: Net-(R113-Pad2) -> /Battery_Charger/Vusb
- R116 pad 1: Net-(R116-Pad1) -> /Battery_Charger/EN1
- R116 pad 2: GND -> /Battery_Charger/Vusb
- R117 pad 1: Net-(R117-Pad1) -> /Battery_Charger/Vusb
- R117 pad 2: GND -> /Battery_Charger/EN2
- R8 pad 1: Net-(C5-Pad1) -> Net-(R8-Pad1)
- R8 pad 2: Net-(R8-Pad2) -> Net-(C5-Pad1)
- R9 pad 1: HVGND -> Net-(C5-Pad1)
- R9 pad 2: Net-(C5-Pad1) -> HVGND
- SW2 pad 1: Net-(R113-Pad2) -> /Battery_Charger/EN2
- SW2 pad 2: Net-(R113-Pad2) -> /Battery_Charger/EN1
- SW2 pad 3: Net-(R117-Pad1) -> GND
- SW2 pad 4: Net-(R116-Pad1) -> GND
- U1 pad 4: Net-(R8-Pad2) -> Net-(R8-Pad1)
- U23 pad 5: Net-(R117-Pad1) -> /Battery_Charger/EN2
- U23 pad 6: Net-(R116-Pad1) -> /Battery_Charger/EN1
Routing:
- net Net-(GD1-Pad1): track 7.71 -> 80.8 mm
- net Net-(J1-Pad1): track 26.2 -> 72.9 mm
- net GND: track 19.8 -> 59.1 mm, vias 6 -> 11
- net Net-(GD1-Pad2): track 20.9 -> 47.9 mm
- net Net-(Q19-Pad1): track 0.00 -> 12.8 mm, vias 0 -> 1
- net /communication/RX_LV: track 0.00 -> 12.1 mm, vias 0 -> 1
- net /communication/A_HV: track 0.00 -> 11.4 mm
- net /communication/K_HV: track 0.00 -> 11.2 mm
- net Net-(C20-Pad2): track 0.00 -> 10.6 mm
- net Net-(C24-Pad2): track 0.00 -> 10.3 mm
- net /Battery_Charger/SYSOFF: track 0.00 -> 9.92 mm
- net /LV_UART_RX: track 0.00 -> 8.61 mm, vias 0 -> 1
- net Net-(C19-Pad1): track 0.00 -> 8.46 mm
- net Net-(Q10-Pad3): track 0.00 -> 8.31 mm
- net +5V: track 18.5 -> 26.5 mm
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Other:
- board outline added: 555 x 100 mm
- board text added: "1 2 ---- 0 0 OFF 1 0 1A 0 1 500mA 1 1 100mA"
- board text added: "GND Anode"
- board text added: "UE Extract."
- board text added: "UF Focus"
- board text added: "UK (HVGND) Kathode"

Commit message: - PCB WiP
Parts:
- added C205: 1u, Capacitor_SMD:C_0603_1608Metric, B.Cu at (423.4, 76.3)
- added C206: 1u, Capacitor_SMD:C_0603_1608Metric, B.Cu at (378.3, 76.5)
- added C207: 1u, Capacitor_SMD:C_0603_1608Metric, B.Cu at (334.0, 76.3)
- added C208: 1u, Capacitor_SMD:C_0603_1608Metric, B.Cu at (281.3, 76.7)
- added REF**: MountingHole_3.2mm_M3, MountingHole:MountingHole_3.2mm_M3, F.Cu at (138.5, 73.5)
- added REF**: SO8_to_MSOP8_3x3mm_P0.65mm, miscellaneous_my:SO8_to_MSOP8_3x3mm_P0.65mm, F.Cu at (515.5, 80.0)
- added REF**: SO8_to_MSOP8_3x3mm_P0.65mm, miscellaneous_my:SO8_to_MSOP8_3x3mm_P0.65mm, F.Cu at (498.5, 80.0)
- added REF**: SO8_to_MSOP8_3x3mm_P0.65mm, miscellaneous_my:SO8_to_MSOP8_3x3mm_P0.65mm, F.Cu at (524.0, 71.0)
- added REF**: SO8_to_MSOP8_3x3mm_P0.65mm, miscellaneous_my:SO8_to_MSOP8_3x3mm_P0.65mm, F.Cu at (515.5, 71.0)
- added REF**: SO8_to_MSOP8_3x3mm_P0.65mm, miscellaneous_my:SO8_to_MSOP8_3x3mm_P0.65mm, F.Cu at (507.0, 71.0)
- added REF**: SO8_to_MSOP8_3x3mm_P0.65mm, miscellaneous_my:SO8_to_MSOP8_3x3mm_P0.65mm, F.Cu at (490.0, 80.0)
- added REF**: SO8_to_MSOP8_3x3mm_P0.65mm, miscellaneous_my:SO8_to_MSOP8_3x3mm_P0.65mm, F.Cu at (498.5, 71.0)
- added REF**: MountingHole_3.2mm_M3, MountingHole:MountingHole_3.2mm_M3, F.Cu at (231.5, 73.5)
- added REF**: SO8_to_MSOP8_3x3mm_P0.65mm, miscellaneous_my:SO8_to_MSOP8_3x3mm_P0.65mm, F.Cu at (524.0, 89.0)
- added REF**: SO8_to_MSOP8_3x3mm_P0.65mm, miscellaneous_my:SO8_to_MSOP8_3x3mm_P0.65mm, F.Cu at (490.0, 71.0)
- added REF**: SO8_to_MSOP8_3x3mm_P0.65mm, miscellaneous_my:SO8_to_MSOP8_3x3mm_P0.65mm, F.Cu at (515.5, 89.0)
- added REF**: SO8_to_MSOP8_3x3mm_P0.65mm, miscellaneous_my:SO8_to_MSOP8_3x3mm_P0.65mm, F.Cu at (498.5, 89.0)
- added REF**: SO8_to_MSOP8_3x3mm_P0.65mm, miscellaneous_my:SO8_to_MSOP8_3x3mm_P0.65mm, F.Cu at (507.0, 89.0)
- added REF**: SO8_to_MSOP8_3x3mm_P0.65mm, miscellaneous_my:SO8_to_MSOP8_3x3mm_P0.65mm, F.Cu at (490.0, 89.0)
- added REF**: SO8_to_MSOP8_3x3mm_P0.65mm, miscellaneous_my:SO8_to_MSOP8_3x3mm_P0.65mm, F.Cu at (507.0, 80.0)
- added REF**: SO8_to_MSOP8_3x3mm_P0.65mm, miscellaneous_my:SO8_to_MSOP8_3x3mm_P0.65mm, F.Cu at (524.0, 80.0)
- C129, C130, C131, C132, C148, C149, C201, C202, C30, C31, C32, C33, C34, C35, C36, C37, C38, C39, C43, C44, C45, C46, C47, C48, C49, C50, C51, C52, C54, C55, C56, C57, C58, C59, C60, C61, C62, C63, C64, C65, C66, C67, C68, C69, C70, C71, C72, C73, L12, L13, Q5, Q6, Q7, Q8, R14, R196, R197, R198, R199, R35, R36, R37, R38, R39, R40, R41, R42, R43, R44, R45, R46, R47, R48, R49, R52, R53, R54, R55, R56, R57, R58, R59, R60, R62, R65, R66, R67, R72, R73, R74, R75, R76, R77, R78, R79, R80, R81, R82, R83, R84, R85, R86, R87, R88, R89, R90, R91, R92, R93, R94, R95, R96, R97, R98, R99, U13, U15, U16, U17, U5, Y3: moved to B.Cu
- F2, F3: moved to F.Cu
- moved TP16 499.1 mm to (443.6, 61.7), turned to 270 degrees
- moved TP17 497.5 mm to (441.8, 63.9), turned to 270 degrees
- moved TP18 496.9 mm to (440.1, 61.7), turned to 270 degrees
- moved TP19 495.3 mm to (438.3, 63.9), turned to 270 degrees
- moved R146 493.4 mm to (447.2, 67.1), turned to 270 degrees
- moved R148 492.1 mm to (445.4, 67.1), turned to 270 degrees
- moved R154 490.9 mm to (443.6, 67.1), turned to 270 degrees
- moved R160 489.7 mm to (441.8, 67.1), turned to 270 degrees
- moved C137 488.9 mm to (447.2, 70.4), turned to 90 degrees
- moved R161 488.4 mm to (440.1, 67.1), turned to 270 degrees
- moved C138 487.7 mm to (445.4, 70.4), turned to 90 degrees
- moved R162 487.2 mm to (438.3, 67.1), turned to 270 degrees
- moved C139 486.4 mm to (443.6, 70.4), turned to 90 degrees
- moved C140 485.2 mm to (441.8, 70.4), turned to 90 degrees
- moved C146 483.9 mm to (440.1, 70.4), turned to 90 degrees
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Routing:
- net GND: track 59.1 -> 129.6 mm, vias 11 -> 19
- net /ammeter/VCC: track 0.00 -> 23.6 mm, vias 0 -> 2
- net /ammeter/VEE: track 0.00 -> 14.4 mm
- net Net-(C23-Pad2): track 4.04 -> 17.5 mm
- net Net-(C15-Pad2): track 3.75 -> 15.3 mm
- net Net-(C19-Pad2): track 4.08 -> 15.6 mm
- net +3V3: track 30.6 -> 41.1 mm, vias 5 -> 6
- net Net-(C135-Pad1): track 0.00 -> 9.70 mm
- net Net-(R196-Pad1): track 0.00 -> 7.69 mm
- net Net-(C27-Pad1): track 0.00 -> 7.02 mm
- net Net-(R162-Pad1): track 6.87 -> 0.00 mm
- net Net-(R161-Pad1): track 6.66 -> 0.00 mm
- net Net-(R160-Pad1): track 6.45 -> 0.00 mm
- net Net-(C149-Pad1): track 0.00 -> 6.25 mm, vias 0 -> 1
- net Net-(R154-Pad1): track 6.24 -> 0.00 mm
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