File: uScope.kicad_pcb (KiCad board)
At the start: 2 copper layers, 555 x 100 mm, 639 parts, among them J1 Pump+, J10 Nucleo_SWD, J11 STLinkV2, J12 Nucleo_SWD, J2 Pump-, J3 U_E, J4 U_F, J5 Conn_01x02, J6 U_K, J7 Anode, J8 USB_B_Micro, J9 STLinkV2, Q1 BC817, Q10 BC817, Q11 BC807, Q12 BSS138, Q13 BSS138, Q14 BSS138, Q15 BSS138, Q16 BSS138, Q17 BSS138, Q18 BSS138, Q19 BSS138, Q2 MMST3906, Q20 BSS138, Q21 BC817, Q3 BC817, Q4 BC807, Q5 BUK98150-55A, Q6 BUK98150-55A, Q7 BUK98150-55A, Q8 BUK98150-55A, Q9 BSS84, SW1 RST, SW10 ESC, SW11 RST, SW2 set_current, SW3 PWRON, SW4 RST, SW5 Encoder, SW6 X, SW7 UP, SW8 DOWN, SW9 ENTER, U1 K, U10 LMC6482, U11 LMC6482, U12 LMC6482, U13 LM321, U14 DAC8564, U15 LM321, U16 LM321, U17 LM321, U18 LM317L_SOT89, U19 PAM242x, U2 E, U20 LM337L_SO8, U21 TPS613222ADBV, U22 LP2985-3.3, U23 BQ24079RGT, U24 Holder 2x18650, U25 LCD_I2C, U26 STM32L431RBTx, U27 ADS131M06, U28 OPTI128, U29 QSE159, U3 F, U30 SN74LVC1G14DRL, U31 QSE159, U32 SN74LVC1G14DRL, U33 ADS131M06, U34 STM32L431RBTx, U35 LM317L_SOT89, U36 LP2985-3.3, U37 TL432, U38 TC7660S, U39 LM337L_SO8, U4 Pump, U5 INA128, U6 RHV2-1212S/R20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

Commit message: - PCB WiP
Parts:
- removed C141: 10n, Capacitor_SMD:C_0603_1608Metric
- removed R149, R155: 10k, Resistor_SMD:R_0603_1608Metric
- removed R68, R69, R70, R71: 10k, Resistor_SMD:R_0603_1608Metric_Pad1.05x0.95mm_HandSolder
- removed the REF** at (524.0, 71.0)
- removed the REF** at (515.5, 71.0)
- removed SW6: X, Button_Switch_SMD:SW_Push_1P1T_NO_6x6mm_H9.5mm
- removed TP27, TP39, TP40: TestPoint, TestPoint:TestPoint_THTPad_D1.5mm_Drill0.7mm
- added JP1: 10k, miscellaneous_my:Jumper_3P_0603_1608Metric_open, F.Cu at (370.1, 96.5)
- added JP2: 10k, miscellaneous_my:Jumper_3P_0603_1608Metric_open, F.Cu at (371.6, 96.5)
- added L16: BLM18TG102, Inductor_SMD:L_0603_1608Metric, F.Cu at (441.1, 93.5)
- added L17: BLM18TG102, Inductor_SMD:L_0603_1608Metric, F.Cu at (438.4, 90.4)
- added L18: BLM18TG102, Inductor_SMD:L_0603_1608Metric, F.Cu at (439.3, 93.5)
- added L19: BLM18TG102, Inductor_SMD:L_0603_1608Metric, F.Cu at (442.0, 90.4)
- added L20: BLM18TG102, Inductor_SMD:L_0603_1608Metric, F.Cu at (437.5, 93.5)
- added L21: BLM18TG102, Inductor_SMD:L_0603_1608Metric, F.Cu at (440.2, 90.4)
- added L22: BLM18TG102, Inductor_SMD:L_0603_1608Metric, F.Cu at (159.0, -25.4)
- added L23: BLM18TG102, Inductor_SMD:L_0603_1608Metric, F.Cu at (162.0, -26.9)
- added L24: BLM18TG102, Inductor_SMD:L_0603_1608Metric, F.Cu at (162.0, -25.4)
- added L25: BLM18TG102, Inductor_SMD:L_0603_1608Metric, F.Cu at (162.0, -28.5)
- added L26: BLM18TG102, Inductor_SMD:L_0603_1608Metric, F.Cu at (159.0, -28.5)
- added L27: BLM18TG102, Inductor_SMD:L_0603_1608Metric, F.Cu at (159.0, -26.9)
- added REF**: SO8_to_MSOP8_3x3mm_P0.65mm, miscellaneous_my:SO8_to_MSOP8_3x3mm_P0.65mm, F.Cu at (97.2, 89.7)
- added REF**: SO8_to_MSOP8_3x3mm_P0.65mm, miscellaneous_my:SO8_to_MSOP8_3x3mm_P0.65mm, F.Cu at (88.7, 89.7)
- C126, C133, C134, C153, C154, C155, C156, C169, C171, C172, C175, C176, D23, L14, L15, NTC1, R136, R143, R180, R50, R51, R61, R63, R64, U14, U6, Y1, Y4, Y5: moved to B.Cu
- Y2, Y6: footprint Crystal:Crystal_AT310_D3.0mm_L10.0mm_Horizontal_1EP_style2 -> Crystal:Crystal_C38-LF_D3.0mm_L8.0mm_Horizontal_1EP_style1; moved to B.Cu
- moved C8 458.2 mm to (38.2, 94.0)
- moved D2 458.2 mm to (36.2, 101.6)
- moved Q2 458.2 mm to (38.2, 91.4)
- moved R12 458.2 mm to (32.4, 101.6)
- moved R127 458.2 mm to (31.6, 87.4)
- moved R16 458.2 mm to (31.6, 96.8)
- moved R203 458.2 mm to (32.4, 89.9)
- moved TP11 458.2 mm to (48.9, 94.7)
- moved TP5 458.2 mm to (48.9, 89.7)
- moved TP7 458.2 mm to (48.9, 92.2)
- moved U10 458.2 mm to (41.3, 99.6)
- moved C10 458.2 mm to (48.6, 109.7)
- moved C11 458.2 mm to (36.4, 97.8)
- moved C12 458.2 mm to (25.0, 93.0)
- moved C203 458.2 mm to (41.5, 88.9)
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Connections:
- net /MCU_low/KEY_DOWN renamed /MCU_low/KEY_RIGHT
- net /MCU_low/KEY_UP renamed /MCU_low/KEY_LEFT
- C133 pad 1: GND -> Net-(C133-Pad1)
- C133 pad 2: Net-(C133-Pad2) -> GND
- C175 pad 1: HVGND -> Net-(C175-Pad1)
- C175 pad 2: Net-(C175-Pad2) -> HVGND
- D24 pad 1: Net-(D24-Pad1) -> GND
- D24 pad 2: /MCU_low/LED_GRN -> Net-(D24-Pad2)
- D25 pad 1: Net-(D25-Pad1) -> GND
- D25 pad 2: /MCU_low/LED_ORG -> Net-(D25-Pad2)
- D26 pad 1: Net-(D26-Pad1) -> GND
- D26 pad 2: /MCU_low/LED_RED -> Net-(D26-Pad2)
- D27 pad 1: Net-(D27-Pad1) -> GND
- D27 pad 2: /MCU_low/LED_BLU -> Net-(D27-Pad2)
- D31 pad 1: Net-(D31-Pad1) -> HVGND
- D31 pad 2: /MCU_high/LED_GRN -> Net-(D31-Pad2)
- D32 pad 1: Net-(D32-Pad1) -> HVGND
- D32 pad 2: /MCU_high/LED_ORG -> Net-(D32-Pad2)
- D33 pad 1: Net-(D33-Pad1) -> HVGND
- D33 pad 2: /MCU_high/LED_RED -> Net-(D33-Pad2)
- D34 pad 1: Net-(D34-Pad1) -> HVGND
- D34 pad 2: /MCU_high/LED_BLU -> Net-(D34-Pad2)
- R139 pad 1: Net-(D24-Pad1) -> /MCU_low/LED_GRN
- R139 pad 2: GND -> Net-(D24-Pad2)
- R140 pad 1: Net-(D25-Pad1) -> /MCU_low/LED_ORG
- R140 pad 2: GND -> Net-(D25-Pad2)
- R141 pad 1: Net-(D26-Pad1) -> /MCU_low/LED_RED
- R141 pad 2: GND -> Net-(D26-Pad2)
- R142 pad 1: Net-(D27-Pad1) -> /MCU_low/LED_BLU
- R142 pad 2: GND -> Net-(D27-Pad2)
- R183 pad 1: Net-(D31-Pad1) -> /MCU_high/LED_GRN
- R183 pad 2: HVGND -> Net-(D31-Pad2)
- R184 pad 1: Net-(D32-Pad1) -> /MCU_high/LED_ORG
- R184 pad 2: HVGND -> Net-(D32-Pad2)
- R185 pad 1: Net-(D33-Pad1) -> /MCU_high/LED_RED
- R185 pad 2: HVGND -> Net-(D33-Pad2)
- R186 pad 1: Net-(D34-Pad1) -> /MCU_high/LED_BLU
- R186 pad 2: HVGND -> Net-(D34-Pad2)
- U26 pad 3: Net-(C133-Pad2) -> Net-(C133-Pad1)
- U26 pad 36: /MCU_low/KEY_5 -> Net-(U26-Pad36)
- U27 pad 16: /MCU_low/ADC_RESET -> Net-(L16-Pad1)
- U27 pad 17: /MCU_low/ADC_CS -> Net-(L21-Pad2)
- U27 pad 18: /MCU_low/ADC_DRDY -> Net-(L20-Pad1)
- U27 pad 19: /MCU_low/ADC_SCK -> Net-(L19-Pad1)
- U27 pad 20: /MCU_low/ADC_MISO -> Net-(L18-Pad1)
- U27 pad 21: /MCU_low/ADC_MOSI -> Net-(L17-Pad1)
- U33 pad 16: /MCU_high/ADC_RESET -> Net-(L22-Pad1)
- U33 pad 17: /MCU_high/ADC_CS -> Net-(L27-Pad2)
- U33 pad 18: /MCU_high/ADC_DRDY -> Net-(L26-Pad1)
- U33 pad 19: /MCU_high/ADC_SCK -> Net-(L25-Pad1)
- U33 pad 20: /MCU_high/ADC_MISO -> Net-(L24-Pad1)
- U33 pad 21: /MCU_high/ADC_MOSI -> Net-(L23-Pad1)
- U34 pad 3: Net-(C175-Pad2) -> Net-(C175-Pad1)
- Y2 pad 1: Net-(C133-Pad2) -> Net-(C134-Pad2)
- Y2 pad 2: Net-(C134-Pad2) -> Net-(C133-Pad1)
- Y2 pad 3: (no net) -> GND
- Y6 pad 1: Net-(C175-Pad2) -> Net-(C175-Pad1)
- Y6 pad 3: (no net) -> HVGND
Routing:
- net /drivers/DAC_D: track 0.00 -> 99.4 mm
- net /drivers/DAC_A: track 0.00 -> 61.4 mm
- net /MCU_low/DAC_load: track 0.00 -> 58.8 mm, vias 0 -> 1
- net /MCU_low/DAC_CS: track 0.00 -> 58.3 mm, vias 0 -> 1
- net /MCU_low/DAC_MOSI: track 0.00 -> 57.0 mm, vias 0 -> 1
- net /MCU_low/DAC_NSS: track 0.00 -> 55.3 mm, vias 0 -> 1
- net /MCU_low/DAC_SCK: track 0.00 -> 54.9 mm, vias 0 -> 1
- net /drivers/DAC_C: track 0.00 -> 46.8 mm
- net /MCU_low/SWD_IO: track 0.00 -> 42.8 mm, vias 0 -> 2
- net /MCU_low/NRST: track 3.96 -> 42.5 mm, vias 1 -> 3
- net /MCU_low/SWD_CLK: track 0.00 -> 37.7 mm
- net /MCU_low/SWD_SWO: track 0.00 -> 34.8 mm, vias 0 -> 2
- net /MCU_low/MCO: track 0.00 -> 27.5 mm, vias 0 -> 2
- net /MCU_low/LED_RED: track 0.00 -> 23.7 mm
- net /MCU_low/ADC_SCK: track 0.00 -> 23.4 mm
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Other:
- board size 555 x 100 mm -> 435 x 100 mm
- board text added: "LEFT"
- board text added: "RIGHT"
- board text removed: "DOWN"
- board text removed: "UP"
- board text removed: "X"

Commit message: - PCB WiP
Parts:
- removed C10: 1n5 6kV, Capacitor_THT:C_Rect_L26.5mm_W7.0mm_P22.50mm_MKS4
- removed C11, C8: 100p, Capacitor_SMD:C_0603_1608Metric
- removed C12: 100n, Capacitor_THT:C_Rect_L7.0mm_W3.5mm_P5.00mm
- removed C186, C7, C9: 100n, Capacitor_SMD:C_0603_1608Metric
- removed C193: 2u2, Capacitor_SMD:C_0805_2012Metric
- removed C203, C204: 1u, Capacitor_SMD:C_0603_1608Metric
- removed D1, D2: 1SS355, miscellaneous_my:D_SOD-323-523_HandSoldering
- removed Q1: BC817, Package_TO_SOT_SMD:SOT-23
- removed Q2: MMST3906, Package_TO_SOT_SMD:SOT-23
- removed R10, R11, R13, R16, R205: 100R, Resistor_SMD:R_0603_1608Metric
- removed R12: 10k, Resistor_SMD:R_0603_1608Metric
- removed R127, R15: 6M8, Resistor_SMD:R_1206_3216Metric_Pad1.42x1.75mm_HandSolder
- removed R179, R202, R203: 1M, Resistor_SMD:R_0603_1608Metric_Pad1.05x0.95mm_HandSolder
- removed R206, R207: 47k, Resistor_SMD:R_0603_1608Metric
- removed the REF** at (138.5, 73.5)
- removed the REF** at (88.7, 98.7)
- removed the REF** at (71.7, 98.7)
- removed the REF** at (97.2, 89.7)
- removed the REF** at (88.7, 89.7)
- removed the REF** at (80.2, 89.7)
- removed the REF** at (63.2, 98.7)
- removed the REF** at (71.7, 89.7)
- removed the REF** at (446.5, 111.5)
- removed the REF** at (446.5, 18.5)
- removed the REF** at (353.5, 18.5)
- removed the REF** at (231.5, 73.5)
- removed the REF** at (353.5, 111.5)
- removed the REF** at (346.5, 111.5)
- removed the REF** at (346.5, 18.5)
- removed the REF** at (253.5, 18.5)
- removed the REF** at (253.5, 111.5)
- removed the REF** at (111.5, 18.5)
- removed the REF** at (138.5, 111.5)
- removed the REF** at (97.2, 107.7)
- removed the REF** at (231.5, 111.5)
- removed the REF** at (138.5, 18.5)
- removed the REF** at (63.2, 89.7)
- removed the REF** at (88.7, 107.7)
- removed the REF** at (71.7, 107.7)
- removed the REF** at (80.2, 107.7)
- removed the REF** at (63.2, 107.7)
- removed the REF** at (80.2, 98.7)
- removed the REF** at (97.2, 98.7)
- removed SW1: RST, Button_Switch_SMD:SW_Push_1P1T_NO_6x6mm_H9.5mm
- removed TP10, TP11, TP12, TP42, TP5, TP6, TP7, TP8, TP9: TestPoint, TestPoint:TestPoint_THTPad_D1.5mm_Drill0.7mm
- removed U10: LMC6482, Package_SO:SO-8_3.9x4.9mm_P1.27mm
- added D13: 1N4448, miscellaneous_my:D_SOD-323-523_HandSoldering, F.Cu at (92.7, 22.5)
- added J13: Conn_02x09_Odd_Even, Connector_PinSocket_2.54mm:PinSocket_2x09_P2.54mm_Vertical, B.Cu at (110.2, 84.8)
- added J14: Conn_02x09_Odd_Even, Connector_PinSocket_2.54mm:PinSocket_2x09_P2.54mm_Vertical, F.Cu at (334.5, 84.8)
- added J15: Conn_02x03_Odd_Even, Connector_PinSocket_2.54mm:PinSocket_2x03_P2.54mm_Vertical, B.Cu at (24.0, 17.2)
- added J16: Conn_02x03_Odd_Even, Connector_PinSocket_2.54mm:PinSocket_2x03_P2.54mm_Vertical, F.Cu at (241.5, 17.2)
- added REF**: PinSocket_2x05_P2.54mm_Vertical, Connector_PinSocket_2.54mm:PinSocket_2x05_P2.54mm_Vertical, F.Cu at (327.8, 95.0)
- added REF**: MountingHole_3.2mm_M3, MountingHole:MountingHole_3.2mm_M3, F.Cu at (133.5, 18.5)
- added REF**: MountingHole_3.2mm_M3, MountingHole:MountingHole_3.2mm_M3, F.Cu at (133.5, 111.5)
- added REF**: MountingHole_3.2mm_M3, MountingHole:MountingHole_3.2mm_M3, F.Cu at (18.5, 73.5)
- added REF**: MountingHole_3.2mm_M3, MountingHole:MountingHole_3.2mm_M3, F.Cu at (111.5, 73.5)
- added REF**: MountingHole_3.2mm_M3, MountingHole:MountingHole_3.2mm_M3, F.Cu at (326.5, 111.5)
- added REF**: MountingHole_3.2mm_M3, MountingHole:MountingHole_3.2mm_M3, F.Cu at (326.5, 18.5)
- added REF**: MountingHole_3.2mm_M3, MountingHole:MountingHole_3.2mm_M3, F.Cu at (233.5, 18.5)
- added REF**: MountingHole_3.2mm_M3, MountingHole:MountingHole_3.2mm_M3, F.Cu at (233.5, 111.5)
- added REF**: MountingHole_3.2mm_M3, MountingHole:MountingHole_3.2mm_M3, F.Cu at (226.5, 111.5)
- added REF**: MountingHole_3.2mm_M3, MountingHole:MountingHole_3.2mm_M3, F.Cu at (226.5, 18.5)
- added TP27: TestPoint, TestPoint:TestPoint_THTPad_D1.5mm_Drill0.7mm, F.Cu at (326.9, 61.7)
- added TP39: TestPoint, TestPoint:TestPoint_THTPad_D1.5mm_Drill0.7mm, F.Cu at (325.3, 63.9)
- added TP40: TestPoint, TestPoint:TestPoint_THTPad_D1.5mm_Drill0.7mm, B.Cu at (17.7, 27.1)
- C116, C157, C158, C159, C165, C166, C167, C168, C170, C80, D18, D19, D21, F1, J8, L22, L25, L27, Q10, Q11, Q12, Q13, Q14, Q9, R103, R104, R111, R113, R114, R115, R120, R121, R123, R124, R125, R126, R174, R175, R176, R177, R178, R181, R182, SW11, TP13, TP14, TP15, TP20, TP21, TP22, TP23, TP41, U28, U33: moved to B.Cu
- C150, C153, C154, C155, C156, C171, C172, C181, C182, C183, C184, C185, C189, C194, C195, C196, C199, C81, C82, C84, C85, C87, C88, C89, D9, L10, L14, L15, R105, R192, R194, U19, U36, U39, Y4: moved to F.Cu
- C200, C86: footprint Capacitor_THT:CP_Radial_D10.0mm_P2.50mm_P5.00mm -> Capacitor_THT:CP_Radial_D8.0mm_P3.50mm; moved to B.Cu
- D12, D14, D35, D36, D5, D6: footprint Diode_SMD:D_SOD-323_HandSoldering -> miscellaneous_my:D_SOD-323-523_HandSoldering
- D37, D38: footprint Diode_SMD:D_SOD-323_HandSoldering -> miscellaneous_my:D_SOD-323-523_HandSoldering; moved to F.Cu
- U25: footprint miscellaneous_my:HD44780_20x4_wPCF8574 -> Connector_PinHeader_2.54mm:PinHeader_1x04_P2.54mm_Vertical
- U38: footprint Package_SO:SOP-8_3.9x4.9mm_P1.27mm -> Package_SO:SOIC-8_3.9x4.9mm_P1.27mm
- moved U25 277.5 mm to (331.7, 122.4)
- moved J11 184.2 mm to (70.8, 25.9), turned to 270 degrees
- moved R185 174.5 mm to (48.8, 21.2), turned to 90 degrees
- moved J12 174.5 mm to (75.8, 31.0), turned to 270 degrees
- moved D30 174.3 mm to (78.5, 26.5), turned to 90 degrees
- moved C179 172.7 mm to (97.4, 19.9), turned to 90 degrees
- moved R184 171.8 mm to (51.1, 21.2), turned to 90 degrees
- moved R173 171.8 mm to (78.5, 30.1), turned to 90 degrees
- moved C180 170.9 mm to (99.2, 19.2), turned to 90 degrees
- moved D33 170.5 mm to (48.8, 17.8), turned to 270 degrees
- moved C181 170.2 mm to (89.2, 23.7)
- moved C184 169.5 mm to (93.1, 24.3)
- moved R183 169.2 mm to (53.4, 21.2), turned to 90 degrees
- moved R186 168.3 mm to (55.6, 21.2), turned to 90 degrees
- moved D32 167.8 mm to (51.1, 17.8), turned to 270 degrees
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Connections:
- TP41 pad 1: Net-(TP41-Pad1) -> /ADC_UF
- U34 pad 29: Net-(TP41-Pad1) -> Net-(U34-Pad29)
Routing:
- net /Battery_Charger/Vusb: track 5.91 -> 92.7 mm, vias 0 -> 4
- net Net-(Q10-Pad1): track 5.16 -> 58.4 mm, vias 0 -> 1
- net /Battery_Charger/EN1: track 0.00 -> 51.8 mm, vias 0 -> 2
- net /Battery_Charger/EN2: track 0.00 -> 49.6 mm, vias 0 -> 2
- net /MCU_high/NRST: track 6.52 -> 49.2 mm, vias 1 -> 2
- net Net-(C10-Pad2): track 38.2 -> 0.00 mm
- net /MCU_high/SWD_CLK: track 6.13 -> 36.5 mm, vias 0 -> 1
- net Net-(R114-Pad2): track 9.35 -> 37.5 mm, vias 0 -> 1
- net /MCU_high/SWD_IO: track 10.9 -> 38.7 mm, vias 0 -> 1
- net /MCU_high/MCO: track 0.00 -> 27.4 mm, vias 0 -> 1
- net HVGND: track 37.6 -> 63.5 mm
- net KEY_PWR: track 4.21 -> 28.3 mm
- net Net-(L23-Pad1): track 0.00 -> 22.8 mm, vias 0 -> 1
- net PWR_LOCK: track 0.00 -> 20.6 mm
- net /MCU_high/SWD_SWO: track 8.36 -> 27.7 mm, vias 0 -> 1
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Other:
- board size 435 x 100 mm -> 315 x 100 mm
- board text added: "CH0"
- board text added: "CH1"
- board text added: "CH2"
- board text added: "CH3"
- board text added: "CH4"
- board text added: "CH5"
