File: uScope.kicad_pcb (KiCad board)
At the start: 2 copper layers, 315 x 100 mm, 594 parts, among them J1 Pump+, J10 Nucleo_SWD, J11 STLinkV2, J12 Nucleo_SWD, J13 Conn_02x09_Odd_Even, J14 Conn_02x09_Odd_Even, J15 Conn_02x03_Odd_Even, J16 Conn_02x03_Odd_Even, J2 Pump-, J3 U_E, J4 U_F, J5 Conn_01x02, J6 U_K, J7 Anode, J8 USB_B_Micro, J9 STLinkV2, Q10 BC817, Q11 BC807, Q12 BSS138, Q13 BSS138, Q14 BSS138, Q15 BSS138, Q16 BSS138, Q17 BSS138, Q18 BSS138, Q19 BSS138, Q20 BSS138, Q21 BC817, Q3 BC817, Q4 BC807, Q5 BUK98150-55A, Q6 BUK98150-55A, Q7 BUK98150-55A, Q8 BUK98150-55A, Q9 BSS84, SW10 ESC, SW11 RST, SW2 set_current, SW3 PWRON, SW4 RST, SW5 Encoder, SW7 UP, SW8 DOWN, SW9 ENTER, U1 K, U11 LMC6482, U12 LMC6482, U13 LM321, U14 DAC8564, U15 LM321, U16 LM321, U17 LM321, U18 LM317L_SOT89, U19 PAM242x, U2 E, U20 LM337L_SO8, U21 TPS613222ADBV, U22 LP2985-3.3, U23 BQ24079RGT, U24 Holder 2x18650, U25 LCD_I2C, U26 STM32L431RBTx, U27 ADS131M06, U28 OPTI128, U29 QSE159, U3 F, U30 SN74LVC1G14DRL, U31 QSE159, U32 SN74LVC1G14DRL, U33 ADS131M06, U34 STM32L431RBTx, U35 LM317L_SOT89, U36 LP2985-3.3, U37 TL432, U38 TC7660S, U39 LM337L_SO8, U4 Pump, U5 INA128, U6 RHV2-1212S/R20, U8 LMC6482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

Commit message: - PCB WiP
Parts:
- moved R150 52.3 mm to (51.4, 92.3), turned to 0 degrees
- moved R151 40.8 mm to (64.5, 92.3), turned to 0 degrees
- moved R152 29.4 mm to (77.5, 92.3), turned to 0 degrees
- moved R153 18.0 mm to (90.6, 92.3), turned to 0 degrees
- moved F3 5.54 mm to (99.4, 78.7)
- moved NTC2 2.25 mm to (78.0, 99.3), turned to 90 degrees
- moved C199 2.07 mm to (80.1, 62.6)
- moved C84 1.67 mm to (80.1, 61.1)
- moved C94 1.40 mm to (105.7, 65.5)
- moved C95 1.40 mm to (104.9, 63.5)
- moved D12 1.40 mm to (102.1, 65.5)
- moved D14 1.40 mm to (105.0, 69.1)
- moved R106 1.40 mm to (98.6, 63.8)
- moved C90 1.40 mm to (98.5, 65.3)
- moved C93 1.40 mm to (101.2, 75.1)
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Connections:
- C125 pad 2: /MCU_low/ENC_SW -> /MCU_low/ENC_SW_F
- C127 pad 2: /MCU_low/ENC_A -> /MCU_low/ENC_A_F
- C128 pad 2: /MCU_low/ENC_B -> /MCU_low/ENC_B_F
- C142 pad 2: /MCU_low/KEY_LEFT -> /MCU_low/LEFT
- C143 pad 2: /MCU_low/KEY_RIGHT -> /MCU_low/RIGHT
- C144 pad 2: /MCU_low/KEY_ENTER -> /MCU_low/ENTER
- C145 pad 2: /MCU_low/KEY_ESC -> /MCU_low/ESC
- J13 pad 10: KEY_PWR -> /MCU_low/ENC_SW
- J13 pad 12: /MCU_low/ENC_SW -> /MCU_low/ENC_B
- J13 pad 16: /MCU_low/ENC_B -> PWR_LOCK
- J13 pad 18: PWR_LOCK -> KEY_PWR
- J14 pad 11: /MCU_low/ENC_SW -> /MCU_low/ENC_B
- J14 pad 15: /MCU_low/ENC_B -> PWR_LOCK
- J14 pad 17: PWR_LOCK -> KEY_PWR
- J14 pad 9: KEY_PWR -> /MCU_low/ENC_SW
- R134 pad 2: Net-(R134-Pad2) -> /MCU_low/ENC_SW
- R135 pad 1: Net-(R134-Pad2) -> /MCU_low/ENC_SW
- R135 pad 2: /MCU_low/ENC_SW -> /MCU_low/ENC_SW_F
- R137 pad 2: Net-(R137-Pad2) -> /MCU_low/ENC_A
- R138 pad 1: Net-(R138-Pad1) -> /MCU_low/ENC_B
- R144 pad 1: Net-(R137-Pad2) -> /MCU_low/ENC_A
- R144 pad 2: /MCU_low/ENC_A -> /MCU_low/ENC_A_F
- R145 pad 1: Net-(R138-Pad1) -> /MCU_low/ENC_B
- R145 pad 2: /MCU_low/ENC_B -> /MCU_low/ENC_B_F
- R150 pad 2: Net-(R150-Pad2) -> /MCU_low/KEY_LEFT
- R151 pad 2: Net-(R151-Pad2) -> /MCU_low/KEY_RIGHT
- R152 pad 2: Net-(R152-Pad2) -> /MCU_low/KEY_ENTER
- R153 pad 2: Net-(R153-Pad2) -> /MCU_low/KEY_ESC
- R156 pad 1: Net-(R150-Pad2) -> /MCU_low/KEY_LEFT
- R156 pad 2: /MCU_low/KEY_LEFT -> /MCU_low/LEFT
- R157 pad 1: Net-(R151-Pad2) -> /MCU_low/KEY_RIGHT
- R157 pad 2: /MCU_low/KEY_RIGHT -> /MCU_low/RIGHT
- R158 pad 1: Net-(R152-Pad2) -> /MCU_low/KEY_ENTER
- R158 pad 2: /MCU_low/KEY_ENTER -> /MCU_low/ENTER
- R159 pad 1: Net-(R153-Pad2) -> /MCU_low/KEY_ESC
- R159 pad 2: /MCU_low/KEY_ESC -> /MCU_low/ESC
- SW10 pad 2: Net-(R153-Pad2) -> /MCU_low/KEY_ESC
- SW5 pad A: Net-(R137-Pad2) -> /MCU_low/ENC_A
- SW5 pad B: Net-(R138-Pad1) -> /MCU_low/ENC_B
- SW5 pad S2: Net-(R134-Pad2) -> /MCU_low/ENC_SW
- SW7 pad 2: Net-(R150-Pad2) -> /MCU_low/KEY_LEFT
- SW8 pad 2: Net-(R151-Pad2) -> /MCU_low/KEY_RIGHT
- SW9 pad 2: Net-(R152-Pad2) -> /MCU_low/KEY_ENTER
- U26 pad 26: /MCU_low/ENC_A -> /MCU_low/ENC_A_F
- U26 pad 27: /MCU_low/ENC_B -> /MCU_low/ENC_B_F
- U26 pad 28: /MCU_low/ENC_SW -> /MCU_low/ENC_SW_F
- U26 pad 37: /MCU_low/KEY_LEFT -> /MCU_low/LEFT
- U26 pad 38: /MCU_low/KEY_RIGHT -> /MCU_low/RIGHT
- U26 pad 39: /MCU_low/KEY_ENTER -> /MCU_low/ENTER
- U26 pad 40: /MCU_low/KEY_ESC -> /MCU_low/ESC
Routing:
- net +3V3: track 59.5 -> 218.3 mm, vias 7 -> 11
- net /MCU_low/ENC_SW: track 0.00 -> 101.9 mm
- net /MCU_low/ENC_A: track 0.00 -> 101.4 mm
- net /MCU_low/ENC_B: track 0.00 -> 93.5 mm
- net /MCU_low/KEY_LEFT: track 1.73 -> 74.8 mm
- net /MCU_low/KEY_RIGHT: track 2.24 -> 62.3 mm
- net +15V: track 13.1 -> 72.0 mm, vias 0 -> 1
- net /LV_UART_RX: track 9.96 -> 61.0 mm
- net Net-(C114-Pad2): track 10.4 -> 59.4 mm
- net /MCU_low/KEY_ENTER: track 2.24 -> 50.1 mm
- net +12V: track 30.4 -> 74.2 mm, vias 1 -> 4
- net /MCU_low/KEY_ESC: track 2.24 -> 37.7 mm
- net GND: track 127.3 -> 149.0 mm, vias 14 -> 24
- net /Battery_Charger/Vusb: track 92.7 -> 108.7 mm
- net KEY_PWR: track 28.3 -> 16.2 mm
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
Commit message: - PCB WiP - polygons on PCB small
Parts:
- C171, C181, C182, C183, C184, C185, C189, C194, C195, C196, D13, D30, D37, D38, L26, Q18, R167, R173, R192, R194, U36, U39: moved to B.Cu
- C175, C176, L25: moved to F.Cu
- moved C195 13.0 mm to (94.2, 33.0)
- moved R192 12.8 mm to (81.7, 36.6)
- moved R194 11.4 mm to (82.5, 33.3)
- moved C189 9.94 mm to (83.3, 36.6)
- moved C194 9.83 mm to (92.5, 36.3)
- moved C196 9.83 mm to (92.5, 33.0)
- moved R173 9.24 mm to (86.2, 25.0), turned to 180 degrees
- moved R164 7.87 mm to (57.5, 36.4), turned to 0 degrees
- moved U36 6.55 mm to (92.7, 20.7), turned to 270 degrees
- moved C171 6.13 mm to (19.7, 46.3), turned to 225 degrees
- moved R167 6.11 mm to (64.8, 34.4), turned to 270 degrees
- moved D37 6.08 mm to (85.4, 31.6), turned to 0 degrees
- moved R191 5.77 mm to (103.8, 33.4)
- moved D38 4.63 mm to (89.5, 31.6), turned to 180 degrees
- moved D30 4.44 mm to (82.7, 25.0), turned to 180 degrees
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Routing:
- net HV+3V3: track 30.6 -> 169.4 mm, vias 7 -> 11
- net HV+5V: track 20.6 -> 147.3 mm, vias 0 -> 2
- net HV-5V: track 16.9 -> 98.1 mm, vias 0 -> 2
- net HVGND: track 63.5 -> 97.9 mm, vias 11 -> 58
- net /HV_UART_TX: track 0.00 -> 23.2 mm, vias 0 -> 1
- net /HV_UART_RX: track 6.23 -> 22.8 mm
- net Net-(C191-Pad1): track 28.4 -> 44.1 mm, vias 0 -> 2
- net Net-(L22-Pad1): track 0.00 -> 13.2 mm
- net HV+12V: track 13.2 -> 22.9 mm
- net Net-(D30-Pad2): track 18.6 -> 27.1 mm
- net Net-(R191-Pad2): track 9.66 -> 2.30 mm
- net GND: track 149.0 -> 154.7 mm, vias 24 -> 59
- net /communication/K_HV: track 5.32 -> 9.87 mm
- net Net-(C171-Pad1): track 5.81 -> 1.74 mm, vias 1 -> 0
- net /MCU_high/ADC_MISO: track 10.8 -> 7.27 mm
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- added copper zone on B.Cu, net GND
- added copper zone on F.Cu, net GND
- added copper zone on B.Cu, net HVGND
- added copper zone on F.Cu, net HVGND

Commit message: - PCB WiP
Parts:
- removed C108: 1u, Capacitor_SMD:C_0603_1608Metric
- removed R201: 100k, Resistor_THT:R_Axial_DIN0207_L6.3mm_D2.5mm_P10.16mm_Horizontal
- removed the REF** at (327.8, 95.0)
- added C7: 100n, Capacitor_SMD:C_0603_1608Metric, F.Cu at (306.8, 111.4)
- added R10: 10k, Resistor_SMD:R_0603_1608Metric_Pad1.05x0.95mm_HandSolder, B.Cu at (250.4, 85.5)
- added R11: 10k, Resistor_SMD:R_0603_1608Metric_Pad1.05x0.95mm_HandSolder, B.Cu at (248.9, 85.5)
- added R12: 10k, Resistor_SMD:R_0603_1608Metric_Pad1.05x0.95mm_HandSolder, B.Cu at (247.4, 85.5)
- added R13: 10k, Resistor_SMD:R_0603_1608Metric_Pad1.05x0.95mm_HandSolder, B.Cu at (245.9, 85.5)
- C102, C103, C133, C134, C143, C145, C97, R110, R157, R159: moved to F.Cu
- C40, C41, C42, C53, JP1, JP2, L16, L19, L9, R200, SW4: moved to B.Cu
- D3, D4: footprint miscellaneous_my:D_SOD-323-523-SMA_Universal_Handsoldering -> miscellaneous_my:D_SOD-323-523_HandSoldering
- R35, R49, R72, R86: value 10k -> 0R
- moved R87 135.3 mm to (270.4, 91.7), turned to 180 degrees
- moved R73 82.6 mm to (270.4, 90.2), turned to 180 degrees
- moved SW4 49.5 mm to (251.6, 110.7), turned to 0 degrees
- moved R52 40.3 mm to (270.4, 93.2), turned to 180 degrees
- moved C109 37.9 mm to (312.8, 108.7), turned to 270 degrees
- moved C107 36.2 mm to (314.3, 108.7), turned to 270 degrees
- moved C102 35.6 mm to (320.0, 108.2), turned to 90 degrees
- moved L19 35.6 mm to (289.6, 105.2), turned to 180 degrees
- moved C103 35.0 mm to (318.5, 108.2), turned to 90 degrees
- moved L16 35.0 mm to (287.0, 101.6)
- moved U22 34.7 mm to (317.1, 108.7), turned to 180 degrees
- moved C105 34.3 mm to (321.4, 108.7), turned to 270 degrees
- moved C104 34.2 mm to (319.8, 108.7), turned to 270 degrees
- moved C97 34.2 mm to (315.7, 105.5)
- moved R110 34.2 mm to (312.5, 105.5)
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Connections:
- J13 pad 17: GND -> +BATT
- J13 pad 2: /MCU_low/KEY_LEFT -> /MCU_low/KEY_ESC
- J13 pad 4: /MCU_low/KEY_RIGHT -> /MCU_low/KEY_ENTER
- J13 pad 6: /MCU_low/KEY_ENTER -> /MCU_low/KEY_RIGHT
- J13 pad 8: /MCU_low/KEY_ESC -> /MCU_low/KEY_LEFT
- J13 pad 9: +BATT -> GND
- J14 pad 1: /MCU_low/KEY_LEFT -> /MCU_low/KEY_ESC
- J14 pad 10: +BATT -> GND
- J14 pad 18: GND -> +BATT
- J14 pad 3: /MCU_low/KEY_RIGHT -> /MCU_low/KEY_ENTER
- J14 pad 5: /MCU_low/KEY_ENTER -> /MCU_low/KEY_RIGHT
- J14 pad 7: /MCU_low/KEY_ESC -> /MCU_low/KEY_LEFT
- R35 pad 1: /drivers/DAC_A -> Net-(C31-Pad2)
- R49 pad 1: /drivers/DAC_B -> Net-(C44-Pad2)
- R72 pad 1: /drivers/DAC_C -> Net-(C55-Pad2)
- R86 pad 1: /drivers/DAC_D -> Net-(C65-Pad2)
Routing:
- net +12V: track 74.2 -> 269.5 mm, vias 4 -> 20
- net +15V: track 72.0 -> 248.9 mm, vias 1 -> 10
- net +BATT: track 22.3 -> 124.9 mm, vias 0 -> 1
- net /drivers/DAC_D: track 99.4 -> 0.00 mm
- net +5V: track 47.8 -> 143.1 mm, vias 2 -> 5
- net GND: track 154.7 -> 234.1 mm, vias 59 -> 115
- net /LV_UART_TX: track 0.00 -> 69.2 mm, vias 0 -> 2
- net /drivers/DAC_A: track 61.4 -> 2.73 mm
- net Net-(L19-Pad1): track 10.1 -> 62.6 mm, vias 2 -> 1
- net Net-(L17-Pad1): track 11.4 -> 58.6 mm, vias 0 -> 2
- net /MCU_low/ADC_MISO: track 13.3 -> 58.4 mm, vias 0 -> 2
- net /drivers/DAC_C: track 46.8 -> 2.75 mm
- net /MCU_low/ADC_DRDY: track 11.4 -> 55.2 mm, vias 0 -> 2
- net Net-(L21-Pad2): track 10.5 -> 52.3 mm
- net /MCU_low/LEFT: track 1.73 -> 43.6 mm, vias 1 -> 0
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
Commit message: - PCB WiP
Parts:
- added REF**: MountingHole_2.2mm_M2, MountingHole:MountingHole_2.2mm_M2, F.Cu at (265.2, 26.4)
- added REF**: Symbol_HighVoltage_Type2_CopperTop_VerySmall, Symbol:Symbol_HighVoltage_Type2_CopperTop_VerySmall, F.Cu at (183.5, 33.1)
- added REF**: Symbol_Highvoltage_Type2_CopperTop_Small, Symbol:Symbol_Highvoltage_Type2_CopperTop_Small, F.Cu at (178.6, 68.1)
- added REF**: Symbol_Highvoltage_Type2_CopperTop_Small, Symbol:Symbol_Highvoltage_Type2_CopperTop_Small, B.Cu at (78.6, 50.5)
- added REF**: Symbol_Highvoltage_Type2_CopperTop_Small, Symbol:Symbol_Highvoltage_Type2_CopperTop_Small, B.Cu at (31.5, 62.1)
- added REF**: Symbol_Highvoltage_Type2_CopperTop_Small, Symbol:Symbol_Highvoltage_Type2_CopperTop_Small, F.Cu at (78.6, 50.5)
- added REF**: Symbol_Highvoltage_Type2_CopperTop_Small, Symbol:Symbol_Highvoltage_Type2_CopperTop_Small, F.Cu at (31.5, 62.1)
- added REF**: MountingHole_2.2mm_M2, MountingHole:MountingHole_2.2mm_M2, F.Cu at (265.2, 21.8)
- added REF**: MountingHole_2.2mm_M2, MountingHole:MountingHole_2.2mm_M2, F.Cu at (223.5, 26.4)
- added REF**: MountingHole_2.2mm_M2, MountingHole:MountingHole_2.2mm_M2, F.Cu at (223.5, 21.8)
- added REF**: Symbol_HighVoltage_Type2_CopperTop_VerySmall, Symbol:Symbol_HighVoltage_Type2_CopperTop_VerySmall, F.Cu at (268.2, 33.1)
- added REF**: Symbol_HighVoltage_Type2_CopperTop_VerySmall, Symbol:Symbol_HighVoltage_Type2_CopperTop_VerySmall, B.Cu at (268.2, 33.1)
- added REF**: Symbol_HighVoltage_Type2_CopperTop_VerySmall, Symbol:Symbol_HighVoltage_Type2_CopperTop_VerySmall, F.Cu at (226.8, 33.1)
- added REF**: Symbol_HighVoltage_Type2_CopperTop_VerySmall, Symbol:Symbol_HighVoltage_Type2_CopperTop_VerySmall, B.Cu at (226.8, 33.1)
- added REF**: Symbol_HighVoltage_Type2_CopperTop_VerySmall, Symbol:Symbol_HighVoltage_Type2_CopperTop_VerySmall, B.Cu at (183.5, 33.1)
- added TP10: TestPoint, TestPoint:TestPoint_THTPad_D1.5mm_Drill0.7mm, F.Cu at (235.7, 24.6)
- added TP11: TestPoint, TestPoint:TestPoint_THTPad_D1.5mm_Drill0.7mm, F.Cu at (233.9, 25.7)
- added TP12: TestPoint, TestPoint:TestPoint_THTPad_D1.5mm_Drill0.7mm, F.Cu at (191.8, 25.7)
- added TP42: TestPoint, TestPoint:TestPoint_THTPad_D1.5mm_Drill0.7mm, F.Cu at (280.0, 24.1)
- added TP5: TestPoint, TestPoint:TestPoint_THTPad_D1.5mm_Drill0.7mm, F.Cu at (193.5, 22.5)
- added TP6: TestPoint, TestPoint:TestPoint_THTPad_D1.5mm_Drill0.7mm, F.Cu at (235.7, 22.5)
- added TP7: TestPoint, TestPoint:TestPoint_THTPad_D1.5mm_Drill0.7mm, F.Cu at (191.8, 23.5)
- added TP8: TestPoint, TestPoint:TestPoint_THTPad_D1.5mm_Drill0.7mm, F.Cu at (233.9, 23.5)
- added TP9: TestPoint, TestPoint:TestPoint_THTPad_D1.5mm_Drill0.7mm, F.Cu at (193.5, 24.6)
- J13, J14: value Conn_02x09_Odd_Even -> Conn_02x10_Odd_Even; footprint Connector_PinSocket_2.54mm:PinSocket_2x09_P2.54mm_Vertical -> Connector_PinSocket_2.54mm:PinSocket_2x10_P2.54mm_Vertical
- R122, R36, R52, R73, R87: moved to F.Cu
- moved R132 34.1 mm to (297.6, 106.2), turned to 270 degrees
- moved R128 34.0 mm to (297.6, 102.5), turned to 270 degrees
- moved Q16 30.5 mm to (300.1, 106.2), turned to 0 degrees
- moved Q15 30.4 mm to (300.1, 102.5), turned to 0 degrees
- moved R133 27.0 mm to (302.6, 106.2), turned to 90 degrees
- moved R129 26.8 mm to (302.6, 102.5), turned to 90 degrees
- moved U25 25.4 mm to (304.0, 110.0), turned to 270 degrees
- moved R63 12.6 mm to (263.4, 94.8), turned to 90 degrees
- moved R61 11.9 mm to (261.7, 94.8), turned to 90 degrees
- moved R51 11.7 mm to (260.1, 94.8), turned to 90 degrees
- moved R64 9.51 mm to (263.4, 92.3), turned to 0 degrees
- moved R50 8.28 mm to (260.1, 92.3), turned to 180 degrees
- moved C40 6.93 mm to (255.9, 90.6), turned to 0 degrees
- moved R52 4.84 mm to (272.3, 88.8)
- moved D22 4.60 mm to (240.0, 99.4)
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Connections:
- J13 pad 1: GND -> +12V
- J13 pad 10: /MCU_low/ENC_SW -> /MCU_low/KEY_LEFT
- J13 pad 11: +15V -> GND
- J13 pad 12: /MCU_low/ENC_B -> /MCU_low/ENC_SW
- J13 pad 13: +5V -> GND
- J13 pad 14: /MCU_low/ENC_A -> /MCU_low/ENC_B
- J13 pad 15: +3V3 -> +5V
- J13 pad 16: PWR_LOCK -> /MCU_low/ENC_A
- J13 pad 17: +BATT -> +3V3
- J13 pad 18: KEY_PWR -> PWR_LOCK
- J13 pad 2: /MCU_low/KEY_ESC -> -5V
- J13 pad 3: /LV_UART_TX -> +15V
- J13 pad 4: /MCU_low/KEY_ENTER -> GND
- J13 pad 5: /LV_UART_RX -> /LV_UART_TX
- J13 pad 6: /MCU_low/KEY_RIGHT -> /MCU_low/KEY_ESC
- J13 pad 7: GND -> /LV_UART_RX
- J13 pad 8: /MCU_low/KEY_LEFT -> /MCU_low/KEY_ENTER
- J13 pad 9: GND -> /MCU_low/KEY_RIGHT
- J14 pad 1: /MCU_low/KEY_ESC -> -5V
- J14 pad 10: GND -> /MCU_low/KEY_RIGHT
- J14 pad 11: /MCU_low/ENC_B -> /MCU_low/ENC_SW
- J14 pad 12: +15V -> GND
- J14 pad 13: /MCU_low/ENC_A -> /MCU_low/ENC_B
- J14 pad 14: +5V -> GND
- J14 pad 15: PWR_LOCK -> /MCU_low/ENC_A
- J14 pad 16: +3V3 -> +5V
- J14 pad 17: KEY_PWR -> PWR_LOCK
- J14 pad 18: +BATT -> +3V3
- J14 pad 2: GND -> +12V
- J14 pad 3: /MCU_low/KEY_ENTER -> GND
- J14 pad 4: /LV_UART_TX -> +15V
- J14 pad 5: /MCU_low/KEY_RIGHT -> /MCU_low/KEY_ESC
- J14 pad 6: /LV_UART_RX -> /LV_UART_TX
- J14 pad 7: /MCU_low/KEY_LEFT -> /MCU_low/KEY_ENTER
- J14 pad 8: GND -> /LV_UART_RX
- J14 pad 9: /MCU_low/ENC_SW -> /MCU_low/KEY_LEFT
- U26 pad 35: KEY_PWR -> PWR_LOCK
- U26 pad 36: Net-(U26-Pad36) -> KEY_PWR
- U26 pad 45: PWR_LOCK -> Net-(U26-Pad45)
Routing:
- net Net-(C65-Pad2): track 19.4 -> 120.8 mm
- net +5V: track 143.1 -> 239.1 mm, vias 5 -> 6
- net HVGND: track 97.9 -> 177.8 mm, vias 58 -> 71
- net -5V: track 9.78 -> 81.2 mm, vias 0 -> 1
- net +3V3: track 237.7 -> 299.4 mm, vias 12 -> 14
- net HV+5V: track 147.3 -> 208.8 mm, vias 2 -> 4
- net /LV_UART_TX: track 69.2 -> 128.5 mm, vias 2 -> 4
- net /LV_UART_RX: track 68.6 -> 126.9 mm, vias 2 -> 4
- net Net-(C55-Pad2): track 19.6 -> 68.2 mm
- net PWR_LOCK: track 42.5 -> 90.6 mm
- net KEY_PWR: track 36.7 -> 84.1 mm, vias 1 -> 0
- net HV-5V: track 98.1 -> 136.7 mm, vias 2 -> 4
- net /ADC_UF: track 16.8 -> 51.0 mm, vias 0 -> 1
- net /ADC_UE: track 19.8 -> 48.8 mm, vias 0 -> 1
- net /MCU_low/I2C_SCL: track 1.57 -> 29.1 mm, vias 0 -> 2
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Other:
- net class Default: clearance 0.2 -> 0.1778
- rule trace_clearance: 0.2 -> 0.1778
- rule trace_min: 0.2 -> 0.1778

Commit message: - PCB final !!!!! before DRC
Parts:
- removed the REF** at (178.6, 68.1)
- removed the REF** at (78.6, 50.5) (x2)
- removed the REF** at (268.2, 33.1) (x2)
- removed the REF** at (226.8, 33.1) (x2)
- added REF** (x2): Symbol_Attention_CopperTop_Big, Symbol:Symbol_Attention_CopperTop_Big, F.Cu at (188.0, 101.1)
- added REF**: Symbol_HighVoltage_Type2_CopperTop_VerySmall, Symbol:Symbol_HighVoltage_Type2_CopperTop_VerySmall, F.Cu at (268.2, 33.1)
- added REF**: Symbol_HighVoltage_Type2_CopperTop_VerySmall, Symbol:Symbol_HighVoltage_Type2_CopperTop_VerySmall, B.Cu at (268.2, 33.1)
- added REF**: Symbol_HighVoltage_Type2_CopperTop_VerySmall, Symbol:Symbol_HighVoltage_Type2_CopperTop_VerySmall, F.Cu at (226.8, 33.1)
- added REF**: Symbol_HighVoltage_Type2_CopperTop_VerySmall, Symbol:Symbol_HighVoltage_Type2_CopperTop_VerySmall, B.Cu at (226.8, 33.1)
- added REF**: Symbol_Highvoltage_Type2_CopperTop_Small, Symbol:Symbol_Highvoltage_Type2_CopperTop_Small, B.Cu at (78.6, 50.5)
- added REF**: Symbol_Highvoltage_Type2_CopperTop_Small, Symbol:Symbol_Highvoltage_Type2_CopperTop_Small, F.Cu at (78.6, 50.5)
- added REF**: OSHW-Logo2_14.6x12mm_Copper, Symbol:OSHW-Logo2_14.6x12mm_Copper, F.Cu at (207.8, 100.6)
- added REF**: Symbol_Highvoltage_Type2_CopperTop_Small, Symbol:Symbol_Highvoltage_Type2_CopperTop_Small, B.Cu at (290.4, 37.1)
- added REF**: OSHW-Logo2_14.6x12mm_SilkScreen, Symbol:OSHW-Logo2_14.6x12mm_SilkScreen, F.Cu at (207.8, 100.6)
- added REF**: Symbol_Highvoltage_Type2_CopperTop_Small, Symbol:Symbol_Highvoltage_Type2_CopperTop_Small, B.Cu at (227.0, 66.2)
- added REF**: Symbol_Highvoltage_Type2_CopperTop_Small, Symbol:Symbol_Highvoltage_Type2_CopperTop_Small, B.Cu at (178.1, 68.1)
- C126, D23: moved to F.Cu
- moved R136 15.2 mm to (302.1, 112.8)
- moved R143 15.2 mm to (298.6, 112.8)
- moved D23 14.8 mm to (302.1, 112.8)
- moved C126 14.8 mm to (298.6, 112.8)
- moved R153 4.19 mm to (85.0, 90.0)
- moved L21 1.54 mm to (294.1, 103.4), turned to 0 degrees
- moved C41 1.40 mm to (242.8, 91.7)
- moved C42 1.40 mm to (244.3, 91.7)
- moved C53 1.40 mm to (244.3, 94.7)
- moved L9 1.40 mm to (242.8, 94.7)
- moved R50 1.40 mm to (260.1, 93.7)
- moved R64 1.40 mm to (263.4, 93.7)
- moved C40 1.40 mm to (255.9, 91.9)
- moved D22 1.40 mm to (240.0, 100.8)
- moved JP1 1.40 mm to (255.1, 95.0)
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Routing:
- net +3V3: track 299.4 -> 398.3 mm, vias 14 -> 16
- net Net-(C55-Pad2): track 68.2 -> 122.1 mm, vias 0 -> 1
- net Net-(C65-Pad2): track 120.8 -> 174.3 mm, vias 0 -> 1
- net Net-(C44-Pad2): track 19.6 -> 64.9 mm, vias 0 -> 1
- net Net-(C31-Pad2): track 28.3 -> 51.1 mm, vias 1 -> 2
- net -5V: track 81.2 -> 100.4 mm
- net +12V: track 285.6 -> 304.1 mm, vias 20 -> 24
- net +15V: track 271.1 -> 255.0 mm
- net +BATT: track 124.9 -> 109.6 mm
- net GND: track 248.2 -> 263.0 mm, vias 141 -> 186
- net /MCU_low/BAT_ADC: track 18.6 -> 31.4 mm
- net /MCU_low/KEY_LEFT: track 82.2 -> 90.7 mm
- net /drivers/DAC_A: track 2.73 -> 8.74 mm
- net /MCU_low/KEY_ESC: track 52.4 -> 57.7 mm
- net /MCU_low/KEY_ENTER: track 58.5 -> 63.7 mm
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Other:
- board text added: "+Pump-"
- board text added: "+Volt -"
- board text added: "1:10 out 10MOhm multimeter"
- board text added: "Extract. UE"
- board text added: "Focus UF"
- board text added: "Kathode UK"
- board text added: "Microscope supply"
- board text added: "Wrocław University of Science and Technology"
- board text added: "Łukasz Sitarek 2020"
- board text removed: "- Volt+"
- board text removed: "-Pump+"
- board text removed: "10MOhm multimeter 1:10 out"
- board text removed: "UE Extract."
- board text removed: "UF Focus"
- board text removed: "UK (HVGND) Kathode"

Commit message: - PCB final before split
Parts:
- removed the REF** at (268.2, 33.1) (x2)
- removed the REF** at (226.8, 33.1) (x2)
- removed the REF** at (78.6, 50.5) (x2)
- added REF**: Symbol_HighVoltage_Type2_CopperTop_VerySmall, Symbol:Symbol_HighVoltage_Type2_CopperTop_VerySmall, F.Cu at (268.2, 33.1)
- added REF**: Symbol_HighVoltage_Type2_CopperTop_VerySmall, Symbol:Symbol_HighVoltage_Type2_CopperTop_VerySmall, B.Cu at (268.2, 33.1)
- added REF**: Symbol_HighVoltage_Type2_CopperTop_VerySmall, Symbol:Symbol_HighVoltage_Type2_CopperTop_VerySmall, F.Cu at (226.8, 33.1)
- added REF**: Symbol_HighVoltage_Type2_CopperTop_VerySmall, Symbol:Symbol_HighVoltage_Type2_CopperTop_VerySmall, B.Cu at (226.8, 33.1)
- added REF**: Symbol_Highvoltage_Type2_CopperTop_Small, Symbol:Symbol_Highvoltage_Type2_CopperTop_Small, B.Cu at (78.6, 50.5)
- added REF**: Symbol_Highvoltage_Type2_CopperTop_Small, Symbol:Symbol_Highvoltage_Type2_CopperTop_Small, F.Cu at (78.6, 50.5)
- moved U32 0.13 mm to (54.1, 36.1)
Routing:
- net HV+3V3: track 169.4 -> 170.3 mm
- net +12V: track 304.1 -> 303.2 mm, vias 24 -> 23
Other:
- rule via_min_size: 0.6 -> 0.8
