File: drivers.sch (KiCad schematic (older format))
At the start: 123 parts, among them Q5 BUK98150-55A, Q6 BUK98150-55A, Q7 BUK98150-55A, Q8 BUK98150-55A, U1 K, U13 LM321, U14 DAC8564, U15 LM321, U16 LM321, U17 LM321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

Commit message: - init PCB - fix last things in schematic
Parts:
- U1, U2, U3, U4: footprint Library_uScope:APD_P2_single -> Power_my:DCDC_APD_P2_single
- U14: footprint (none) -> Package_SO:TSSOP-16_4.4x5mm_P0.65mm
Changed lines of the file:
@@
 F 0 "U1" H 10128 1851 50  0000 L CNN
 F 1 "K" H 10128 1760 50  0000 L CNN
-F 2 "Library_uScope:APD_P2_single" H 9900 1800 50  0001 C CNN
+F 2 "Power_my:DCDC_APD_P2_single" H 9900 1800 50  0001 C CNN
 F 3 "" H 9900 1800 50  0001 C CNN
 	1    9900 1800
@@
 F 0 "U2" H 10128 3551 50  0000 L CNN
 F 1 "E" H 10128 3460 50  0000 L CNN
-F 2 "Library_uScope:APD_P2_single" H 9900 3500 50  0001 C CNN
+F 2 "Power_my:DCDC_APD_P2_single" H 9900 3500 50  0001 C CNN
 F 3 "" H 9900 3500 50  0001 C CNN
 	1    9900 3500
@@
 F 0 "U3" H 10128 5251 50  0000 L CNN
 F 1 "F" H 10128 5160 50  0000 L CNN
-F 2 "Library_uScope:APD_P2_single" H 9900 5200 50  0001 C CNN
+F 2 "Power_my:DCDC_APD_P2_single" H 9900 5200 50  0001 C CNN
 F 3 "" H 9900 5200 50  0001 C CNN
 	1    9900 5200
@@
 L power:+12V #PWR043
 U 1 1 5F61F5AB
-P 9600 1100
-F 0 "#PWR043" H 9600 950 50  0001 C CNN
-F 1 "+12V" H 9600 1216 39  0000 C CNN
-F 2 "" H 9600 1100 50  0001 C CNN
-F 3 "" H 9600 1100 50  0001 C CNN
-	1    9600 1100
+P 9600 1050
+F 0 "#PWR043" H 9600 900 50  0001 C CNN
+F 1 "+12V" H 9600 1166 39  0000 C CNN
+F 2 "" H 9600 1050 50  0001 C CNN
+F 3 "" H 9600 1050 50  0001 C CNN
+	1    9600 1050
 	1    0    0    -1
 $EndComp
@@
 L power:+12V #PWR053
 U 1 1 5F84F50D
-P 9600 2800
-F 0 "#PWR053" H 9600 2650 50  0001 C CNN
-F 1 "+12V" H 9600 2916 39  0000 C CNN
-F 2 "" H 9600 2800 50  0001 C CNN
-F 3 "" H 9600 2800 50  0001 C CNN
-	1    9600 2800
+P 9600 2750
+F 0 "#PWR053" H 9600 2600 50  0001 C CNN
+F 1 "+12V" H 9600 2866 39  0000 C CNN
+F 2 "" H 9600 2750 50  0001 C CNN
+F 3 "" H 9600 2750 50  0001 C CNN
+	1    9600 2750
 	1    0    0    -1
 $EndComp
@@
 L power:+12V #PWR065
 U 1 1 5F84FDEA
-P 9600 4500
-F 0 "#PWR065" H 9600 4350 50  0001 C CNN
-F 1 "+12V" H 9600 4616 39  0000 C CNN
-F 2 "" H 9600 4500 50  0001 C CNN
-F 3 "" H 9600 4500 50  0001 C CNN
-	1    9600 4500
+P 9600 4450
+F 0 "#PWR065" H 9600 4300 50  0001 C CNN
+F 1 "+12V" H 9600 4566 39  0000 C CNN
+F 2 "" H 9600 4450 50  0001 C CNN
+F 3 "" H 9600 4450 50  0001 C CNN
+	1    9600 4450
 	1    0    0    -1
 $EndComp
@@
 F 0 "U4" H 6228 7251 50  0000 L CNN
 F 1 "Pump" H 6228 7160 50  0000 L CNN
-F 2 "Library_uScope:APD_P2_single" H 6000 7200 50  0001 C CNN
+F 2 "Power_my:DCDC_APD_P2_single" H 6000 7200 50  0001 C CNN
 F 3 "" H 6000 7200 50  0001 C CNN
 	1    6000 7200
@@
 F 0 "U14" H 2600 3200 50  0000 C CNN
 F 1 "DAC8564" H 3300 3200 50  0000 C CNN
-F 2 "" H 4000 1850 50  0001 C CNN
+F 2 "Package_SO:TSSOP-16_4.4x5mm_P0.65mm" H 4000 1850 50  0001 C CNN
 F 3 "" H 4000 1850 50  0001 C CNN
 	1    3000 2900
@@
 Wire Wire Line
 	2350 2650 1950 2650
+$Comp
+L power:PWR_FLAG #FLG0103
+U 1 1 5FA28994
+P 3400 2100
+F 0 "#FLG0103" H 3400 2175 50  0001 C CNN
+F 1 "PWR_FLAG" H 3400 2274 50  0001 C CNN
+F 2 "" H 3400 2100 50  0001 C CNN
+F 3 "~" H 3400 2100 50  0001 C CNN
+	1    3400 2100
+	1    0    0    -1
+$EndComp
+Wire Wire Line
+	9600 1050 9600 1100
+Wire Wire Line
+	9600 2750 9600 2800
+Wire Wire Line
+	9600 4450 9600 4500
 $EndSCHEMATC

Commit message: - first segregation on pcb
Parts:
- C30, C39, C43, C52, C54, C63, C64, C73: footprint Capacitor_SMD:C_0805_2012Metric_Pad1.15x1.40mm_HandSolder -> Capacitor_SMD:C_0603_1608Metric_Pad1.05x0.95mm_HandSolder
Changed lines of the file:
@@
 F 0 "C39" H 8750 1650 50  0000 R CNN
 F 1 "100p" H 8750 1550 50  0000 R CNN
-F 2 "Capacitor_SMD:C_0805_2012Metric_Pad1.15x1.40mm_HandSolder" H 8800 1600 50  0001 C CNN
+F 2 "Capacitor_SMD:C_0603_1608Metric_Pad1.05x0.95mm_HandSolder" H 8800 1600 50  0001 C CNN
 F 3 "~" H 8800 1600 50  0001 C CNN
 	1    8800 1600
@@
 F 0 "C30" H 8400 950 50  0000 R CNN
 F 1 "100n" H 8400 850 50  0000 R CNN
-F 2 "Capacitor_SMD:C_0805_2012Metric_Pad1.15x1.40mm_HandSolder" H 8450 900 50  0001 C CNN
+F 2 "Capacitor_SMD:C_0603_1608Metric_Pad1.05x0.95mm_HandSolder" H 8450 900 50  0001 C CNN
 F 3 "~" H 8450 900 50  0001 C CNN
 	1    8450 900
@@
 F 0 "C52" H 8750 3350 50  0000 R CNN
 F 1 "100p" H 8750 3250 50  0000 R CNN
-F 2 "Capacitor_SMD:C_0805_2012Metric_Pad1.15x1.40mm_HandSolder" H 8800 3300 50  0001 C CNN
+F 2 "Capacitor_SMD:C_0603_1608Metric_Pad1.05x0.95mm_HandSolder" H 8800 3300 50  0001 C CNN
 F 3 "~" H 8800 3300 50  0001 C CNN
 	1    8800 3300
@@
 F 0 "C43" H 8400 2650 50  0000 R CNN
 F 1 "100n" H 8400 2550 50  0000 R CNN
-F 2 "Capacitor_SMD:C_0805_2012Metric_Pad1.15x1.40mm_HandSolder" H 8450 2600 50  0001 C CNN
+F 2 "Capacitor_SMD:C_0603_1608Metric_Pad1.05x0.95mm_HandSolder" H 8450 2600 50  0001 C CNN
 F 3 "~" H 8450 2600 50  0001 C CNN
 	1    8450 2600
@@
 F 0 "C63" H 8750 5050 50  0000 R CNN
 F 1 "100p" H 8750 4950 50  0000 R CNN
-F 2 "Capacitor_SMD:C_0805_2012Metric_Pad1.15x1.40mm_HandSolder" H 8800 5000 50  0001 C CNN
+F 2 "Capacitor_SMD:C_0603_1608Metric_Pad1.05x0.95mm_HandSolder" H 8800 5000 50  0001 C CNN
 F 3 "~" H 8800 5000 50  0001 C CNN
 	1    8800 5000
@@
 F 0 "C54" H 8400 4350 50  0000 R CNN
 F 1 "100n" H 8400 4250 50  0000 R CNN
-F 2 "Capacitor_SMD:C_0805_2012Metric_Pad1.15x1.40mm_HandSolder" H 8450 4300 50  0001 C CNN
+F 2 "Capacitor_SMD:C_0603_1608Metric_Pad1.05x0.95mm_HandSolder" H 8450 4300 50  0001 C CNN
 F 3 "~" H 8450 4300 50  0001 C CNN
 	1    8450 4300
@@
 F 0 "C73" H 4850 7050 50  0000 R CNN
 F 1 "100p" H 4850 6950 50  0000 R CNN
-F 2 "Capacitor_SMD:C_0805_2012Metric_Pad1.15x1.40mm_HandSolder" H 4900 7000 50  0001 C CNN
+F 2 "Capacitor_SMD:C_0603_1608Metric_Pad1.05x0.95mm_HandSolder" H 4900 7000 50  0001 C CNN
 F 3 "~" H 4900 7000 50  0001 C CNN
 	1    4900 7000
@@
 F 0 "C64" H 4500 6350 50  0000 R CNN
 F 1 "100n" H 4500 6250 50  0000 R CNN
-F 2 "Capacitor_SMD:C_0805_2012Metric_Pad1.15x1.40mm_HandSolder" H 4550 6300 50  0001 C CNN
+F 2 "Capacitor_SMD:C_0603_1608Metric_Pad1.05x0.95mm_HandSolder" H 4550 6300 50  0001 C CNN
 F 3 "~" H 4550 6300 50  0001 C CNN
 	1    4550 6300

Commit message: - PCB progress
Parts:
- C30, C39, C40, C41, C42, C43, C52, C53, C54, C63, C64, C73: footprint Capacitor_SMD:C_0603_1608Metric_Pad1.05x0.95mm_HandSolder -> Capacitor_SMD:C_0603_1608Metric
- L9: footprint Resistor_SMD:R_0805_2012Metric_Pad1.15x1.40mm_HandSolder -> Inductor_SMD:L_0603_1608Metric
Changed lines of the file:
@@
 F 0 "C39" H 8750 1650 50  0000 R CNN
 F 1 "100p" H 8750 1550 50  0000 R CNN
-F 2 "Capacitor_SMD:C_0603_1608Metric_Pad1.05x0.95mm_HandSolder" H 8800 1600 50  0001 C CNN
+F 2 "Capacitor_SMD:C_0603_1608Metric" H 8800 1600 50  0001 C CNN
 F 3 "~" H 8800 1600 50  0001 C CNN
 	1    8800 1600
@@
 F 0 "C30" H 8400 950 50  0000 R CNN
 F 1 "100n" H 8400 850 50  0000 R CNN
-F 2 "Capacitor_SMD:C_0603_1608Metric_Pad1.05x0.95mm_HandSolder" H 8450 900 50  0001 C CNN
+F 2 "Capacitor_SMD:C_0603_1608Metric" H 8450 900 50  0001 C CNN
 F 3 "~" H 8450 900 50  0001 C CNN
 	1    8450 900
@@
 F 0 "C52" H 8750 3350 50  0000 R CNN
 F 1 "100p" H 8750 3250 50  0000 R CNN
-F 2 "Capacitor_SMD:C_0603_1608Metric_Pad1.05x0.95mm_HandSolder" H 8800 3300 50  0001 C CNN
+F 2 "Capacitor_SMD:C_0603_1608Metric" H 8800 3300 50  0001 C CNN
 F 3 "~" H 8800 3300 50  0001 C CNN
 	1    8800 3300
@@
 F 0 "C43" H 8400 2650 50  0000 R CNN
 F 1 "100n" H 8400 2550 50  0000 R CNN
-F 2 "Capacitor_SMD:C_0603_1608Metric_Pad1.05x0.95mm_HandSolder" H 8450 2600 50  0001 C CNN
+F 2 "Capacitor_SMD:C_0603_1608Metric" H 8450 2600 50  0001 C CNN
 F 3 "~" H 8450 2600 50  0001 C CNN
 	1    8450 2600
@@
 F 0 "C63" H 8750 5050 50  0000 R CNN
 F 1 "100p" H 8750 4950 50  0000 R CNN
-F 2 "Capacitor_SMD:C_0603_1608Metric_Pad1.05x0.95mm_HandSolder" H 8800 5000 50  0001 C CNN
+F 2 "Capacitor_SMD:C_0603_1608Metric" H 8800 5000 50  0001 C CNN
 F 3 "~" H 8800 5000 50  0001 C CNN
 	1    8800 5000
@@
 F 0 "C54" H 8400 4350 50  0000 R CNN
 F 1 "100n" H 8400 4250 50  0000 R CNN
-F 2 "Capacitor_SMD:C_0603_1608Metric_Pad1.05x0.95mm_HandSolder" H 8450 4300 50  0001 C CNN
+F 2 "Capacitor_SMD:C_0603_1608Metric" H 8450 4300 50  0001 C CNN
 F 3 "~" H 8450 4300 50  0001 C CNN
 	1    8450 4300
@@
 F 0 "C73" H 4850 7050 50  0000 R CNN
 F 1 "100p" H 4850 6950 50  0000 R CNN
-F 2 "Capacitor_SMD:C_0603_1608Metric_Pad1.05x0.95mm_HandSolder" H 4900 7000 50  0001 C CNN
+F 2 "Capacitor_SMD:C_0603_1608Metric" H 4900 7000 50  0001 C CNN
 F 3 "~" H 4900 7000 50  0001 C CNN
 	1    4900 7000
@@
 F 0 "C64" H 4500 6350 50  0000 R CNN
 F 1 "100n" H 4500 6250 50  0000 R CNN
-F 2 "Capacitor_SMD:C_0603_1608Metric_Pad1.05x0.95mm_HandSolder" H 4550 6300 50  0001 C CNN
+F 2 "Capacitor_SMD:C_0603_1608Metric" H 4550 6300 50  0001 C CNN
 F 3 "~" H 4550 6300 50  0001 C CNN
 	1    4550 6300
@@
 F 0 "C40" H 2650 2300 50  0000 L BNN
 F 1 "100n" H 2650 2200 50  0000 L TNN
-F 2 "Capacitor_SMD:C_0603_1608Metric_Pad1.05x0.95mm_HandSolder" H 2600 2250 50  0001 C CNN
+F 2 "Capacitor_SMD:C_0603_1608Metric" H 2600 2250 50  0001 C CNN
 F 3 "~" H 2600 2250 50  0001 C CNN
 	1    2600 2250
@@
 F 0 "C42" H 3750 2300 50  0000 L BNN
 F 1 "100n" H 3750 2200 50  0000 L TNN
-F 2 "Capacitor_SMD:C_0603_1608Metric_Pad1.05x0.95mm_HandSolder" H 3700 2250 50  0001 C CNN
+F 2 "Capacitor_SMD:C_0603_1608Metric" H 3700 2250 50  0001 C CNN
 F 3 "~" H 3700 2250 50  0001 C CNN
 	1    3700 2250
@@
 F 0 "C41" H 3450 2300 50  0000 L BNN
 F 1 "1u" H 3450 2200 50  0000 L TNN
-F 2 "Capacitor_SMD:C_0603_1608Metric_Pad1.05x0.95mm_HandSolder" H 3400 2250 50  0001 C CNN
+F 2 "Capacitor_SMD:C_0603_1608Metric" H 3400 2250 50  0001 C CNN
 F 3 "~" H 3400 2250 50  0001 C CNN
 	1    3400 2250
@@
 F 0 "L9" V 3205 2100 50  0000 C CNN
 F 1 "BLM18RK102" V 3114 2100 50  0000 C CNN
-F 2 "Resistor_SMD:R_0805_2012Metric_Pad1.15x1.40mm_HandSolder" H 3000 2100 50  0001 C CNN
+F 2 "Inductor_SMD:L_0603_1608Metric" H 3000 2100 50  0001 C CNN
 F 3 "~" H 3000 2100 50  0001 C CNN
 	1    3000 2100
@@
 F 0 "C53" H 3800 3600 50  0000 L BNN
 F 1 "1u" H 3800 3500 50  0000 L TNN
-F 2 "Capacitor_SMD:C_0603_1608Metric_Pad1.05x0.95mm_HandSolder" H 3750 3550 50  0001 C CNN
+F 2 "Capacitor_SMD:C_0603_1608Metric" H 3750 3550 50  0001 C CNN
 F 3 "~" H 3750 3550 50  0001 C CNN
 	1    3750 3550

Commit message: - PCB WiP - Pump output aligned
Parts:
- R45, R47, R50, R51, R61, R62, R63, R64, R66, R82, R84, R96, R98: footprint Resistor_SMD:R_0603_1608Metric_Pad1.05x0.95mm_HandSolder -> Resistor_SMD:R_0603_1608Metric
Changed lines of the file:
@@
 F 0 "R45" V 9050 1300 50  0000 C BNN
 F 1 "1k" V 8850 1300 50  0000 C TNN
-F 2 "Resistor_SMD:R_0603_1608Metric_Pad1.05x0.95mm_HandSolder" V 8880 1300 50  0001 C CNN
+F 2 "Resistor_SMD:R_0603_1608Metric" V 8880 1300 50  0001 C CNN
 F 3 "~" H 8950 1300 50  0001 C CNN
 	1    8950 1300
@@
 F 0 "R47" V 9050 1800 50  0000 C BNN
 F 1 "100k" V 8850 1800 50  0000 C TNN
-F 2 "Resistor_SMD:R_0603_1608Metric_Pad1.05x0.95mm_HandSolder" V 8880 1800 50  0001 C CNN
+F 2 "Resistor_SMD:R_0603_1608Metric" V 8880 1800 50  0001 C CNN
 F 3 "~" H 8950 1800 50  0001 C CNN
 	1    8950 1800
@@
 F 0 "R62" V 9050 3000 50  0000 C BNN
 F 1 "1k" V 8850 3000 50  0000 C TNN
-F 2 "Resistor_SMD:R_0603_1608Metric_Pad1.05x0.95mm_HandSolder" V 8880 3000 50  0001 C CNN
+F 2 "Resistor_SMD:R_0603_1608Metric" V 8880 3000 50  0001 C CNN
 F 3 "~" H 8950 3000 50  0001 C CNN
 	1    8950 3000
@@
 F 0 "R66" V 9050 3500 50  0000 C BNN
 F 1 "100k" V 8850 3500 50  0000 C TNN
-F 2 "Resistor_SMD:R_0603_1608Metric_Pad1.05x0.95mm_HandSolder" V 8880 3500 50  0001 C CNN
+F 2 "Resistor_SMD:R_0603_1608Metric" V 8880 3500 50  0001 C CNN
 F 3 "~" H 8950 3500 50  0001 C CNN
 	1    8950 3500
@@
 F 0 "R82" V 9050 4700 50  0000 C BNN
 F 1 "1k" V 8850 4700 50  0000 C TNN
-F 2 "Resistor_SMD:R_0603_1608Metric_Pad1.05x0.95mm_HandSolder" V 8880 4700 50  0001 C CNN
+F 2 "Resistor_SMD:R_0603_1608Metric" V 8880 4700 50  0001 C CNN
 F 3 "~" H 8950 4700 50  0001 C CNN
 	1    8950 4700
@@
 F 0 "R84" V 9050 5200 50  0000 C BNN
 F 1 "100k" V 8850 5200 50  0000 C TNN
-F 2 "Resistor_SMD:R_0603_1608Metric_Pad1.05x0.95mm_HandSolder" V 8880 5200 50  0001 C CNN
+F 2 "Resistor_SMD:R_0603_1608Metric" V 8880 5200 50  0001 C CNN
 F 3 "~" H 8950 5200 50  0001 C CNN
 	1    8950 5200
@@
 F 0 "R96" V 5150 6700 50  0000 C BNN
 F 1 "1k" V 4950 6700 50  0000 C TNN
-F 2 "Resistor_SMD:R_0603_1608Metric_Pad1.05x0.95mm_HandSolder" V 4980 6700 50  0001 C CNN
+F 2 "Resistor_SMD:R_0603_1608Metric" V 4980 6700 50  0001 C CNN
 F 3 "~" H 5050 6700 50  0001 C CNN
 	1    5050 6700
@@
 F 0 "R98" V 5150 7200 50  0000 C BNN
 F 1 "100k" V 4950 7200 50  0000 C TNN
-F 2 "Resistor_SMD:R_0603_1608Metric_Pad1.05x0.95mm_HandSolder" V 4980 7200 50  0001 C CNN
+F 2 "Resistor_SMD:R_0603_1608Metric" V 4980 7200 50  0001 C CNN
 F 3 "~" H 5050 7200 50  0001 C CNN
 	1    5050 7200
@@
 F 0 "R64" V 1950 3250 50  0000 C BNN
 F 1 "10R" V 1750 3250 50  0000 C TNN
-F 2 "Resistor_SMD:R_0603_1608Metric_Pad1.05x0.95mm_HandSolder" V 1780 3250 50  0001 C CNN
+F 2 "Resistor_SMD:R_0603_1608Metric" V 1780 3250 50  0001 C CNN
 F 3 "~" H 1850 3250 50  0001 C CNN
 	1    1850 3250
@@
 F 0 "R50" V 1950 2650 50  0000 C BNN
 F 1 "10R" V 1750 2650 50  0000 C TNN
-F 2 "Resistor_SMD:R_0603_1608Metric_Pad1.05x0.95mm_HandSolder" V 1780 2650 50  0001 C CNN
+F 2 "Resistor_SMD:R_0603_1608Metric" V 1780 2650 50  0001 C CNN
 F 3 "~" H 1850 2650 50  0001 C CNN
 	1    1850 2650
@@
 F 0 "R51" V 2250 2800 50  0000 C BNN
 F 1 "10R" V 2050 2800 50  0000 C TNN
-F 2 "Resistor_SMD:R_0603_1608Metric_Pad1.05x0.95mm_HandSolder" V 2080 2800 50  0001 C CNN
+F 2 "Resistor_SMD:R_0603_1608Metric" V 2080 2800 50  0001 C CNN
 F 3 "~" H 2150 2800 50  0001 C CNN
 	1    2150 2800
@@
 F 0 "R61" V 1950 2950 50  0000 C BNN
 F 1 "10R" V 1750 2950 50  0000 C TNN
-F 2 "Resistor_SMD:R_0603_1608Metric_Pad1.05x0.95mm_HandSolder" V 1780 2950 50  0001 C CNN
+F 2 "Resistor_SMD:R_0603_1608Metric" V 1780 2950 50  0001 C CNN
 F 3 "~" H 1850 2950 50  0001 C CNN
 	1    1850 2950
@@
 F 0 "R63" V 2250 3100 50  0000 C BNN
 F 1 "10R" V 2050 3100 50  0000 C TNN
-F 2 "Resistor_SMD:R_0603_1608Metric_Pad1.05x0.95mm_HandSolder" V 2080 3100 50  0001 C CNN
+F 2 "Resistor_SMD:R_0603_1608Metric" V 2080 3100 50  0001 C CNN
 F 3 "~" H 2150 3100 50  0001 C CNN
 	1    2150 3100

Commit message: - PCB WiP
Parts:
- added C205, C206, C207, C208: 1u, Capacitor_SMD:C_0603_1608Metric, symbol Device:C_Small
Connections:
- net +12V: now also C205.2, C206.2, C207.2, C208.2
- net GND: now also C205.1, C206.1, C207.1, C208.1
Changed lines of the file:
@@
-	1    0    0    -1
-$EndComp
-$Comp
-L power:+12V #PWR043
-U 1 1 5F61F5AB
-P 9600 1050
-F 0 "#PWR043" H 9600 900 50  0001 C CNN
-F 1 "+12V" H 9600 1166 39  0000 C CNN
-F 2 "" H 9600 1050 50  0001 C CNN
-F 3 "" H 9600 1050 50  0001 C CNN
-	1    9600 1050
 	1    0    0    -1
 $EndComp
@@
 Wire Wire Line
 	8100 1800 8800 1800
-$Comp
-L power:+12V #PWR053
-U 1 1 5F84F50D
-P 9600 2750
-F 0 "#PWR053" H 9600 2600 50  0001 C CNN
-F 1 "+12V" H 9600 2866 39  0000 C CNN
-F 2 "" H 9600 2750 50  0001 C CNN
-F 3 "" H 9600 2750 50  0001 C CNN
-	1    9600 2750
-	1    0    0    -1
-$EndComp
 Wire Wire Line
 	8100 2900 8050 2900
@@
 Wire Wire Line
 	8100 3500 8800 3500
-$Comp
-L power:+12V #PWR065
-U 1 1 5F84FDEA
-P 9600 4450
-F 0 "#PWR065" H 9600 4300 50  0001 C CNN
-F 1 "+12V" H 9600 4566 39  0000 C CNN
-F 2 "" H 9600 4450 50  0001 C CNN
-F 3 "" H 9600 4450 50  0001 C CNN
-	1    9600 4450
-	1    0    0    -1
-$EndComp
 Wire Wire Line
 	8100 4600 8050 4600
@@
 L power:+12V #PWR071
 U 1 1 5F98552E
-P 5700 6500
-F 0 "#PWR071" H 5700 6350 50  0001 C CNN
-F 1 "+12V" H 5700 6616 39  0000 C CNN
-F 2 "" H 5700 6500 50  0001 C CNN
-F 3 "" H 5700 6500 50  0001 C CNN
-	1    5700 6500
+P 5700 6200
+F 0 "#PWR071" H 5700 6050 50  0001 C CNN
+F 1 "+12V" H 5700 6316 39  0000 C CNN
+F 2 "" H 5700 6200 50  0001 C CNN
+F 3 "" H 5700 6200 50  0001 C CNN
+	1    5700 6200
 	1    0    0    -1
 $EndComp
@@
 	1    0    0    -1
 $EndComp
-Wire Wire Line
-	9600 1050 9600 1100
-Wire Wire Line
-	9600 2750 9600 2800
-Wire Wire Line
-	9600 4450 9600 4500
+$Comp
+L Device:C_Small C208
+U 1 1 5FAF5CBE
+P 5400 6300
+F 0 "C208" H 5350 6350 50  0000 R CNN
+F 1 "1u" H 5350 6250 50  0000 R CNN
+F 2 "Capacitor_SMD:C_0603_1608Metric" H 5400 6300 50  0001 C CNN
+F 3 "~" H 5400 6300 50  0001 C CNN
+	1    5400 6300
+	-1   0    0    1
+$EndComp
+$Comp
+L power:GND #PWR?
+U 1 1 5FAF5F66
+P 5400 6400
+AR Path="/5F40DCB9/5FAF5F66" Ref="#PWR?"  Part="1"
+AR Path="/5F618AB9/5FAF5F66" Ref="#PWR?"  Part="1"
+AR Path="/5FAF5F66" Ref="#PWR?"  Part="1"
+AR Path="/5F61C123/5FAF5F66" Ref="#PWR0250"  Part="1"
+F 0 "#PWR0250" H 5400 6240 50  0001 C CNN
+F 1 "GND" H 5400 6300 39  0000 C TNN
+F 2 "" H 5400 6400 50  0001 C CNN
+F 3 "" H 5400 6400 50  0001 C CNN
+	1    5400 6400
+	1    0    0    -1
+$EndComp
+Wire Wire Line
+	5400 6200 5700 6200
+Wire Wire Line
+	5700 6500 5700 6200
+Connection ~ 5700 6200
+$Comp
+L power:+12V #PWR0207
+U 1 1 5FB4B56D
+P 9600 4200
+F 0 "#PWR0207" H 9600 4050 50  0001 C CNN
+F 1 "+12V" H 9600 4316 39  0000 C CNN
+F 2 "" H 9600 4200 50  0001 C CNN
+F 3 "" H 9600 4200 50  0001 C CNN
+	1    9600 4200
+	1    0    0    -1
+$EndComp
+$Comp
+L Device:C_Small C207
+U 1 1 5FB4B573
+P 9300 4300
+F 0 "C207" H 9250 4350 50  0000 R CNN
+F 1 "1u" H 9250 4250 50  0000 R CNN
+F 2 "Capacitor_SMD:C_0603_1608Metric" H 9300 4300 50  0001 C CNN
+F 3 "~" H 9300 4300 50  0001 C CNN
+	1    9300 4300
+	-1   0    0    1
+$EndComp
+$Comp
+L power:GND #PWR?
+U 1 1 5FB4B57A
+P 9300 4400
+AR Path="/5F40DCB9/5FB4B57A" Ref="#PWR?"  Part="1"
+AR Path="/5F618AB9/5FB4B57A" Ref="#PWR?"  Part="1"
+AR Path="/5FB4B57A" Ref="#PWR?"  Part="1"
+AR Path="/5F61C123/5FB4B57A" Ref="#PWR0212"  Part="1"
+F 0 "#PWR0212" H 9300 4240 50  0001 C CNN
+F 1 "GND" H 9300 4300 39  0000 C TNN
+F 2 "" H 9300 4400 50  0001 C CNN
+F 3 "" H 9300 4400 50  0001 C CNN
+	1    9300 4400
+	1    0    0    -1
+$EndComp
+Wire Wire Line
+	9300 4200 9600 4200
+Wire Wire Line
+	9600 4500 9600 4200
+Connection ~ 9600 4200
+$Comp
+L power:+12V #PWR065
+U 1 1 5FB67647
+P 9600 2500
+F 0 "#PWR065" H 9600 2350 50  0001 C CNN
+F 1 "+12V" H 9600 2616 39  0000 C CNN
+F 2 "" H 9600 2500 50  0001 C CNN
+F 3 "" H 9600 2500 50  0001 C CNN
+	1    9600 2500
+	1    0    0    -1
+$EndComp
+$Comp
+L Device:C_Small C206
+U 1 1 5FB6764D
+P 9300 2600
+F 0 "C206" H 9250 2650 50  0000 R CNN
+F 1 "1u" H 9250 2550 50  0000 R CNN
+F 2 "Capacitor_SMD:C_0603_1608Metric" H 9300 2600 50  0001 C CNN
+F 3 "~" H 9300 2600 50  0001 C CNN
+	1    9300 2600
+	-1   0    0    1
+$EndComp
+$Comp
+L power:GND #PWR?
+U 1 1 5FB67654
+P 9300 2700
+AR Path="/5F40DCB9/5FB67654" Ref="#PWR?"  Part="1"
+AR Path="/5F618AB9/5FB67654" Ref="#PWR?"  Part="1"
+AR Path="/5FB67654" Ref="#PWR?"  Part="1"
+AR Path="/5F61C123/5FB67654" Ref="#PWR0134"  Part="1"
+F 0 "#PWR0134" H 9300 2540 50  0001 C CNN
+F 1 "GND" H 9300 2600 39  0000 C TNN
+F 2 "" H 9300 2700 50  0001 C CNN
+F 3 "" H 9300 2700 50  0001 C CNN
+	1    9300 2700
+	1    0    0    -1
+$EndComp
+Wire Wire Line
+	9300 2500 9600 2500
+Wire Wire Line
+	9600 2800 9600 2500
+Connection ~ 9600 2500
+$Comp
+L power:+12V #PWR043
+U 1 1 5FB8393B
+P 9600 800
+F 0 "#PWR043" H 9600 650 50  0001 C CNN
+F 1 "+12V" H 9600 916 39  0000 C CNN
+F 2 "" H 9600 800 50  0001 C CNN
+F 3 "" H 9600 800 50  0001 C CNN
+	1    9600 800
+	1    0    0    -1
+$EndComp
+$Comp
+L Device:C_Small C205
+U 1 1 5FB83941
+P 9300 900
+F 0 "C205" H 9250 950 50  0000 R CNN
+F 1 "1u" H 9250 850 50  0000 R CNN
+F 2 "Capacitor_SMD:C_0603_1608Metric" H 9300 900 50  0001 C CNN
+F 3 "~" H 9300 900 50  0001 C CNN
+	1    9300 900
+	-1   0    0    1
+$EndComp
+$Comp
+L power:GND #PWR?
+U 1 1 5FB83948
+P 9300 1000
+AR Path="/5F40DCB9/5FB83948" Ref="#PWR?"  Part="1"
+AR Path="/5F618AB9/5FB83948" Ref="#PWR?"  Part="1"
+AR Path="/5FB83948" Ref="#PWR?"  Part="1"
+AR Path="/5F61C123/5FB83948" Ref="#PWR053"  Part="1"
+F 0 "#PWR053" H 9300 840 50  0001 C CNN
+F 1 "GND" H 9300 900 39  0000 C TNN
+F 2 "" H 9300 1000 50  0001 C CNN
+F 3 "" H 9300 1000 50  0001 C CNN
+	1    9300 1000
+	1    0    0    -1
+$EndComp
+Wire Wire Line
+	9300 800  9600 800
+Wire Wire Line
+	9600 1100 9600 800
+Connection ~ 9600 800
 $EndSCHEMATC
