File: drivers.sch (KiCad schematic (older format))
At the start: 127 parts, among them Q5 BUK98150-55A, Q6 BUK98150-55A, Q7 BUK98150-55A, Q8 BUK98150-55A, U1 K, U13 LM321, U14 DAC8564, U15 LM321, U16 LM321, U17 LM321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

Commit message: - PCB WiP
Parts:
- removed R68, R69, R70, R71: 10k, Resistor_SMD:R_0603_1608Metric_Pad1.05x0.95mm_HandSolder, symbol Device:R_Small
- added JP1, JP2: 10k, miscellaneous_my:Jumper_3P_0603_1608Metric_open, symbol Jumper:Jumper_3_Bridged12
Connections:
- net +3V3: now also JP1.3 (B), JP2.3 (B)
- net GND: now also JP1.1 (A), JP2.1 (A)
- net at U14.14 (A1): now also JP1.2 (C)
- net at U14.13 (A0): now also JP2.2 (C)
Changed lines of the file:
@@
 Connection ~ 8100 4600
 Connection ~ 8100 2900
-$Comp
-L Device:R_Small R70
-U 1 1 5FAFD80F
-P 1800 4000
-F 0 "R70" H 1859 4046 50  0000 L CNN
-F 1 "10k" H 1859 3955 50  0000 L CNN
-F 2 "Resistor_SMD:R_0603_1608Metric_Pad1.05x0.95mm_HandSolder" H 1800 4000 50  0001 C CNN
-F 3 "~" H 1800 4000 50  0001 C CNN
-	1    1800 4000
-	1    0    0    -1
-$EndComp
-$Comp
-L Device:R_Small R68
-U 1 1 5FAFF133
-P 1800 3800
-F 0 "R68" H 1859 3846 50  0000 L CNN
-F 1 "10k" H 1859 3755 50  0000 L CNN
-F 2 "Resistor_SMD:R_0603_1608Metric_Pad1.05x0.95mm_HandSolder" H 1800 3800 50  0001 C CNN
-F 3 "~" H 1800 3800 50  0001 C CNN
-	1    1800 3800
-	1    0    0    -1
-$EndComp
-Wire Wire Line
-	1800 3900 2050 3900
-Wire Wire Line
-	2050 3900 2050 3450
-Wire Wire Line
-	2050 3450 2400 3450
-Connection ~ 1800 3900
-$Comp
-L Device:R_Small R71
-U 1 1 5FB149DF
-P 2150 4000
-F 0 "R71" H 2209 4046 50  0000 L CNN
-F 1 "10k" H 2209 3955 50  0000 L CNN
-F 2 "Resistor_SMD:R_0603_1608Metric_Pad1.05x0.95mm_HandSolder" H 2150 4000 50  0001 C CNN
-F 3 "~" H 2150 4000 50  0001 C CNN
-	1    2150 4000
-	1    0    0    -1
-$EndComp
-$Comp
-L Device:R_Small R69
-U 1 1 5FB149E6
-P 2150 3800
-F 0 "R69" H 2209 3846 50  0000 L CNN
-F 1 "10k" H 2209 3755 50  0000 L CNN
-F 2 "Resistor_SMD:R_0603_1608Metric_Pad1.05x0.95mm_HandSolder" H 2150 3800 50  0001 C CNN
-F 3 "~" H 2150 3800 50  0001 C CNN
-	1    2150 3800
-	1    0    0    -1
-$EndComp
-Wire Wire Line
-	2150 3900 2400 3900
-Connection ~ 2150 3900
-Wire Wire Line
-	2400 3900 2400 3550
+Wire Wire Line
+	1950 3950 1950 3450
+Wire Wire Line
+	1950 3450 2400 3450
 $Comp
 L power:GND #PWR?
 U 1 1 5FB6B7BD
-P 2150 4100
+P 2250 4200
 AR Path="/5F40DCB9/5FB6B7BD" Ref="#PWR?"  Part="1"
 AR Path="/5F618AB9/5FB6B7BD" Ref="#PWR?"  Part="1"
@@
 AR Path="/5F7D6767/5FB6B7BD" Ref="#PWR?"  Part="1"
 AR Path="/5F61C123/5FB6B7BD" Ref="#PWR062"  Part="1"
-F 0 "#PWR062" H 2150 3940 50  0001 C CNN
-F 1 "GND" H 2150 4000 39  0000 C TNN
-F 2 "" H 2150 4100 50  0001 C CNN
-F 3 "" H 2150 4100 50  0001 C CNN
-	1    2150 4100
+F 0 "#PWR062" H 2250 4040 50  0001 C CNN
+F 1 "GND" H 2250 4100 39  0000 C TNN
+F 2 "" H 2250 4200 50  0001 C CNN
+F 3 "" H 2250 4200 50  0001 C CNN
+	1    2250 4200
 	1    0    0    -1
 $EndComp
@@
 L power:GND #PWR?
 U 1 1 5FB6B8A6
-P 1800 4100
+P 1800 4200
 AR Path="/5F40DCB9/5FB6B8A6" Ref="#PWR?"  Part="1"
 AR Path="/5F618AB9/5FB6B8A6" Ref="#PWR?"  Part="1"
@@
 AR Path="/5F7D6767/5FB6B8A6" Ref="#PWR?"  Part="1"
 AR Path="/5F61C123/5FB6B8A6" Ref="#PWR061"  Part="1"
-F 0 "#PWR061" H 1800 3940 50  0001 C CNN
-F 1 "GND" H 1800 4000 39  0000 C TNN
-F 2 "" H 1800 4100 50  0001 C CNN
-F 3 "" H 1800 4100 50  0001 C CNN
-	1    1800 4100
+F 0 "#PWR061" H 1800 4040 50  0001 C CNN
+F 1 "GND" H 1800 4100 39  0000 C TNN
+F 2 "" H 1800 4200 50  0001 C CNN
+F 3 "" H 1800 4200 50  0001 C CNN
+	1    1800 4200
 	1    0    0    -1
 $EndComp
@@
 L power:+3V3 #PWR?
 U 1 1 5FF3AAB8
-P 2150 3700
+P 2250 3700
 AR Path="/5F620813/5FF3AAB8" Ref="#PWR?"  Part="1"
 AR Path="/5F61C123/5FF3AAB8" Ref="#PWR058"  Part="1"
-F 0 "#PWR058" H 2150 3550 50  0001 C CNN
-F 1 "+3V3" H 2165 3873 50  0000 C CNN
-F 2 "" H 2150 3700 50  0001 C CNN
-F 3 "" H 2150 3700 50  0001 C CNN
-	1    2150 3700
+F 0 "#PWR058" H 2250 3550 50  0001 C CNN
+F 1 "+3V3" H 2265 3873 50  0000 C CNN
+F 2 "" H 2250 3700 50  0001 C CNN
+F 3 "" H 2250 3700 50  0001 C CNN
+	1    2250 3700
 	1    0    0    -1
 $EndComp
@@
 	9600 1100 9600 800
 Connection ~ 9600 800
+$Comp
+L Jumper:Jumper_3_Bridged12 JP1
+U 1 1 5FDBC5DF
+P 1800 3950
+F 0 "JP1" V 1846 4017 50  0000 L CNN
+F 1 "10k" V 1755 4017 50  0000 L CNN
+F 2 "miscellaneous_my:Jumper_3P_0603_1608Metric_open" H 1800 3950 50  0001 C CNN
+F 3 "~" H 1800 3950 50  0001 C CNN
+	1    1800 3950
+	0    -1   -1   0
+$EndComp
+$Comp
+L Jumper:Jumper_3_Bridged12 JP2
+U 1 1 5FE13BA2
+P 2250 3950
+F 0 "JP2" V 2296 4017 50  0000 L CNN
+F 1 "10k" V 2205 4017 50  0000 L CNN
+F 2 "miscellaneous_my:Jumper_3P_0603_1608Metric_open" H 2250 3950 50  0001 C CNN
+F 3 "~" H 2250 3950 50  0001 C CNN
+	1    2250 3950
+	0    -1   -1   0
+$EndComp
+Wire Wire Line
+	2400 3550 2400 3950
 $EndSCHEMATC

Commit message: - PCB WiP
Parts:
- added R10, R11, R12, R13: 10k, Resistor_SMD:R_0603_1608Metric_Pad1.05x0.95mm_HandSolder, symbol Device:R_Small
- R35, R49, R72, R86: value 10k -> 0R
Connections:
- net DAC_A: now also R10.1; no longer R35.1
- net DAC_B: now also R11.1; no longer R49.1
- net DAC_C: now also R12.1; no longer R72.1
- net DAC_D: now also R13.1; no longer R86.1
- net at C31.2, R36.2, R37.1: now also R35.1, R10.2
- net at C44.2, R52.2, R53.1: now also R49.1, R11.2
- net at C55.2, R73.2, R74.1: now also R72.1, R12.2
- net at C65.2, R87.2, R88.1: now also R86.1, R13.2
Changed lines of the file:
@@
 	5700 5000 5700 5050
 Connection ~ 5700 5000
-Text HLabel 5400 1200 0    50   Input ~ 0
+Text HLabel 5350 1200 0    50   Input ~ 0
 TIM_CH1
 Text HLabel 5100 2900 0    50   Input ~ 0
@@
 Text HLabel 5100 4600 0    50   Input ~ 0
 TIM_CH3
-Wire Wire Line
-	5450 1200 5400 1200
 $Comp
 L uScope:APD_P2_single U?
@@
 	1800 7000 1800 7050
 Connection ~ 1800 7000
-Text HLabel 1500 6600 0    50   Input ~ 0
+Text HLabel 1400 6600 0    50   Input ~ 0
 TIM_CH4
-Wire Wire Line
-	1550 6600 1500 6600
 $Comp
 L power:GND #PWR?
@@
 Text Label 3600 3200 0    50   ~ 0
 DAC_D
-Text Label 7550 900  0    50   ~ 0
+Text Label 5200 900  0    50   ~ 0
 DAC_A
-Wire Wire Line
-	7850 900  7550 900
 Wire Wire Line
 	8100 1200 8100 900
@@
 	8100 900  8050 900
 Connection ~ 8100 1200
-Text Label 7550 2600 0    50   ~ 0
+Text Label 5200 2600 0    50   ~ 0
 DAC_B
 Wire Wire Line
-	7850 2600 7550 2600
-Wire Wire Line
 	8100 2900 8100 2600
 Wire Wire Line
 	8100 2600 8050 2600
-Text Label 7550 4300 0    50   ~ 0
+Text Label 5200 4300 0    50   ~ 0
 DAC_C
 Wire Wire Line
-	7850 4300 7550 4300
-Wire Wire Line
 	8100 4600 8100 4300
 Wire Wire Line
 	8100 4300 8050 4300
-Text Label 3650 6300 0    50   ~ 0
+Text Label 1300 6300 0    50   ~ 0
 DAC_D
-Wire Wire Line
-	3950 6300 3650 6300
 Wire Wire Line
 	4200 6600 4200 6300
@@
 P 4050 6300
 F 0 "R86" V 4150 6300 50  0000 C BNN
-F 1 "10k" V 3950 6300 50  0000 C TNN
+F 1 "0R" V 3950 6300 50  0000 C TNN
 F 2 "Resistor_SMD:R_0603_1608Metric_Pad1.05x0.95mm_HandSolder" V 3980 6300 50  0001 C CNN
 F 3 "~" H 4050 6300 50  0001 C CNN
@@
 $EndComp
 Wire Wire Line
-	5100 4600 5450 4600
-Wire Wire Line
 	5750 2900 5700 2900
 Wire Wire Line
@@
 $EndComp
 Wire Wire Line
-	5100 2900 5450 2900
-Wire Wire Line
 	5750 1200 5700 1200
 Wire Wire Line
@@
 P 7950 900
 F 0 "R35" V 8050 900 50  0000 C BNN
-F 1 "10k" V 7850 900 50  0000 C TNN
+F 1 "0R" V 7850 900 50  0000 C TNN
 F 2 "Resistor_SMD:R_0603_1608Metric_Pad1.05x0.95mm_HandSolder" V 7880 900 50  0001 C CNN
 F 3 "~" H 7950 900 50  0001 C CNN
@@
 P 7950 2600
 F 0 "R49" V 8050 2600 50  0000 C BNN
-F 1 "10k" V 7850 2600 50  0000 C TNN
+F 1 "0R" V 7850 2600 50  0000 C TNN
 F 2 "Resistor_SMD:R_0603_1608Metric_Pad1.05x0.95mm_HandSolder" V 7880 2600 50  0001 C CNN
 F 3 "~" H 7950 2600 50  0001 C CNN
@@
 P 7950 4300
 F 0 "R72" V 8050 4300 50  0000 C BNN
-F 1 "10k" V 7850 4300 50  0000 C TNN
+F 1 "0R" V 7850 4300 50  0000 C TNN
 F 2 "Resistor_SMD:R_0603_1608Metric_Pad1.05x0.95mm_HandSolder" V 7880 4300 50  0001 C CNN
 F 3 "~" H 7950 4300 50  0001 C CNN
@@
 Wire Wire Line
 	2400 3550 2400 3950
+Wire Wire Line
+	5700 900  5700 1200
+Wire Wire Line
+	5700 2600 5700 2900
+Wire Wire Line
+	5700 4300 5700 4600
+Wire Wire Line
+	1800 6300 1800 6600
+$Comp
+L Device:R_Small R10
+U 1 1 5FC5AE2E
+P 5550 900
+F 0 "R10" V 5650 900 50  0000 C BNN
+F 1 "10k" V 5450 900 50  0000 C TNN
+F 2 "Resistor_SMD:R_0603_1608Metric_Pad1.05x0.95mm_HandSolder" V 5480 900 50  0001 C CNN
+F 3 "~" H 5550 900 50  0001 C CNN
+	1    5550 900
+	0    -1   -1   0
+$EndComp
+Wire Wire Line
+	5700 900  7850 900
+Wire Wire Line
+	5350 1200 5450 1200
+Wire Wire Line
+	5700 900  5650 900
+Connection ~ 5700 900
+Wire Wire Line
+	5450 900  5200 900
+Wire Wire Line
+	5700 2600 7850 2600
+Wire Wire Line
+	5100 2900 5450 2900
+$Comp
+L Device:R_Small R11
+U 1 1 5FCD23F9
+P 5550 2600
+F 0 "R11" V 5650 2600 50  0000 C BNN
+F 1 "10k" V 5450 2600 50  0000 C TNN
+F 2 "Resistor_SMD:R_0603_1608Metric_Pad1.05x0.95mm_HandSolder" V 5480 2600 50  0001 C CNN
+F 3 "~" H 5550 2600 50  0001 C CNN
+	1    5550 2600
+	0    -1   -1   0
+$EndComp
+Wire Wire Line
+	5700 2600 5650 2600
+Connection ~ 5700 2600
+Wire Wire Line
+	5450 2600 5200 2600
+Wire Wire Line
+	5700 4300 7850 4300
+Wire Wire Line
+	5100 4600 5450 4600
+$Comp
+L Device:R_Small R12
+U 1 1 5FD2C61F
+P 5550 4300
+F 0 "R12" V 5650 4300 50  0000 C BNN
+F 1 "10k" V 5450 4300 50  0000 C TNN
+F 2 "Resistor_SMD:R_0603_1608Metric_Pad1.05x0.95mm_HandSolder" V 5480 4300 50  0001 C CNN
+F 3 "~" H 5550 4300 50  0001 C CNN
+	1    5550 4300
+	0    -1   -1   0
+$EndComp
+Wire Wire Line
+	5200 4300 5450 4300
+Wire Wire Line
+	5650 4300 5700 4300
+Connection ~ 5700 4300
+Connection ~ 4200 6600
+Wire Wire Line
+	1800 6300 3950 6300
+Wire Wire Line
+	1400 6600 1550 6600
+$Comp
+L Device:R_Small R13
+U 1 1 5FD8A4D7
+P 1650 6300
+F 0 "R13" V 1750 6300 50  0000 C BNN
+F 1 "10k" V 1550 6300 50  0000 C TNN
+F 2 "Resistor_SMD:R_0603_1608Metric_Pad1.05x0.95mm_HandSolder" V 1580 6300 50  0001 C CNN
+F 3 "~" H 1650 6300 50  0001 C CNN
+	1    1650 6300
+	0    -1   -1   0
+$EndComp
+Wire Wire Line
+	1750 6300 1800 6300
+Connection ~ 1800 6300
+Wire Wire Line
+	1550 6300 1300 6300
 $EndSCHEMATC
