File: drivers.sch (KiCad schematic (older format))
At the start: 129 parts, among them Q5 BUK98150-55A, Q6 BUK98150-55A, Q7 BUK98150-55A, Q8 BUK98150-55A, U1 K, U13 LM321, U14 DAC8564, U15 LM321, U16 LM321, U17 LM321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

Commit message: - as-built changes - add custom library elements
Parts:
- R10: value 10k -> n.c.
- R35: value 0R -> n.c.
- R36, R37, R38, R39, R40, R41, R42, R43, R44, R59, R60: value 10k -> 51k
Changed lines of the file:
@@
 encoding utf-8
 Sheet 4 10
-Title ""
-Date ""
-Rev ""
-Comp ""
+Title "Sterowniki"
+Date "2021-01-18"
+Rev "1.0"
+Comp "Łukasz Sitarek"
 Comment1 ""
 Comment2 ""
@@
 P 7650 2900
 F 0 "R59" V 7750 2900 50  0000 C BNN
-F 1 "10k" V 7550 2900 50  0000 C TNN
+F 1 "51k" V 7550 2900 50  0000 C TNN
 F 2 "Resistor_SMD:R_0603_1608Metric_Pad1.05x0.95mm_HandSolder" V 7580 2900 50  0001 C CNN
 F 3 "~" H 7650 2900 50  0001 C CNN
@@
 P 7950 2900
 F 0 "R60" V 8050 2900 50  0000 C BNN
-F 1 "10k" V 7850 2900 50  0000 C TNN
+F 1 "51k" V 7850 2900 50  0000 C TNN
 F 2 "Resistor_SMD:R_0603_1608Metric_Pad1.05x0.95mm_HandSolder" V 7880 2900 50  0001 C CNN
 F 3 "~" H 7950 2900 50  0001 C CNN
@@
 P 5550 1200
 F 0 "R36" V 5650 1200 50  0000 C BNN
-F 1 "10k" V 5450 1200 50  0000 C TNN
+F 1 "51k" V 5450 1200 50  0000 C TNN
 F 2 "Resistor_SMD:R_0603_1608Metric_Pad1.05x0.95mm_HandSolder" V 5480 1200 50  0001 C CNN
 F 3 "~" H 5550 1200 50  0001 C CNN
@@
 P 5850 1200
 F 0 "R37" V 5950 1200 50  0000 C BNN
-F 1 "10k" V 5750 1200 50  0000 C TNN
+F 1 "51k" V 5750 1200 50  0000 C TNN
 F 2 "Resistor_SMD:R_0603_1608Metric_Pad1.05x0.95mm_HandSolder" V 5780 1200 50  0001 C CNN
 F 3 "~" H 5850 1200 50  0001 C CNN
@@
 P 6150 1200
 F 0 "R38" V 6250 1200 50  0000 C BNN
-F 1 "10k" V 6050 1200 50  0000 C TNN
+F 1 "51k" V 6050 1200 50  0000 C TNN
 F 2 "Resistor_SMD:R_0603_1608Metric_Pad1.05x0.95mm_HandSolder" V 6080 1200 50  0001 C CNN
 F 3 "~" H 6150 1200 50  0001 C CNN
@@
 P 6450 1200
 F 0 "R39" V 6550 1200 50  0000 C BNN
-F 1 "10k" V 6350 1200 50  0000 C TNN
+F 1 "51k" V 6350 1200 50  0000 C TNN
 F 2 "Resistor_SMD:R_0603_1608Metric_Pad1.05x0.95mm_HandSolder" V 6380 1200 50  0001 C CNN
 F 3 "~" H 6450 1200 50  0001 C CNN
@@
 P 6750 1200
 F 0 "R40" V 6850 1200 50  0000 C BNN
-F 1 "10k" V 6650 1200 50  0000 C TNN
+F 1 "51k" V 6650 1200 50  0000 C TNN
 F 2 "Resistor_SMD:R_0603_1608Metric_Pad1.05x0.95mm_HandSolder" V 6680 1200 50  0001 C CNN
 F 3 "~" H 6750 1200 50  0001 C CNN
@@
 P 7050 1200
 F 0 "R41" V 7150 1200 50  0000 C BNN
-F 1 "10k" V 6950 1200 50  0000 C TNN
+F 1 "51k" V 6950 1200 50  0000 C TNN
 F 2 "Resistor_SMD:R_0603_1608Metric_Pad1.05x0.95mm_HandSolder" V 6980 1200 50  0001 C CNN
 F 3 "~" H 7050 1200 50  0001 C CNN
@@
 P 7350 1200
 F 0 "R42" V 7450 1200 50  0000 C BNN
-F 1 "10k" V 7250 1200 50  0000 C TNN
+F 1 "51k" V 7250 1200 50  0000 C TNN
 F 2 "Resistor_SMD:R_0603_1608Metric_Pad1.05x0.95mm_HandSolder" V 7280 1200 50  0001 C CNN
 F 3 "~" H 7350 1200 50  0001 C CNN
@@
 P 7650 1200
 F 0 "R43" V 7750 1200 50  0000 C BNN
-F 1 "10k" V 7550 1200 50  0000 C TNN
+F 1 "51k" V 7550 1200 50  0000 C TNN
 F 2 "Resistor_SMD:R_0603_1608Metric_Pad1.05x0.95mm_HandSolder" V 7580 1200 50  0001 C CNN
 F 3 "~" H 7650 1200 50  0001 C CNN
@@
 P 7950 1200
 F 0 "R44" V 8050 1200 50  0000 C BNN
-F 1 "10k" V 7850 1200 50  0000 C TNN
+F 1 "51k" V 7850 1200 50  0000 C TNN
 F 2 "Resistor_SMD:R_0603_1608Metric_Pad1.05x0.95mm_HandSolder" V 7880 1200 50  0001 C CNN
 F 3 "~" H 7950 1200 50  0001 C CNN
@@
 P 7950 900
 F 0 "R35" V 8050 900 50  0000 C BNN
-F 1 "0R" V 7850 900 50  0000 C TNN
+F 1 "n.c." V 7850 900 50  0000 C TNN
 F 2 "Resistor_SMD:R_0603_1608Metric_Pad1.05x0.95mm_HandSolder" V 7880 900 50  0001 C CNN
 F 3 "~" H 7950 900 50  0001 C CNN
@@
 P 5550 900
 F 0 "R10" V 5650 900 50  0000 C BNN
-F 1 "10k" V 5450 900 50  0000 C TNN
+F 1 "n.c." V 5450 900 50  0000 C TNN
 F 2 "Resistor_SMD:R_0603_1608Metric_Pad1.05x0.95mm_HandSolder" V 5480 900 50  0001 C CNN
 F 3 "~" H 5550 900 50  0001 C CNN
