File: MCU_high.sch (KiCad schematic (older format))
At the start: 74 parts, among them J11 STLinkV2, J12 Nucleo_SWD, SW11 RST, U33 ADS131M06, U34 STM32L431RBTx, Y4 8.192, Y5 8.192, Y6 32.768

Commit message: - PCB WiP
Parts:
- removed TP42: TestPoint, TestPoint:TestPoint_THTPad_D1.5mm_Drill0.7mm, symbol Connector:TestPoint
- added J15, J16: Conn_02x03_Odd_Even, Connector_PinSocket_2.54mm:PinSocket_2x03_P2.54mm_Vertical, symbol Connector_Generic:Conn_02x03_Odd_Even
- added TP40: TestPoint, TestPoint:TestPoint_THTPad_D1.5mm_Drill0.7mm, symbol Connector:TestPoint
Connections:
- net ADC_CH0: now also J15.4 (Pin_4), J16.3 (Pin_3), TP40.1
- net ADC_CH1: now also TP41.1, J15.6 (Pin_6), J16.5 (Pin_5)
- net HVGND: now also J15.1 (Pin_1), J15.2 (Pin_2), J16.1 (Pin_1), J16.2 (Pin_2)
- net at U34.29 (PB10): no longer TP41.1
- new net HV+5V: J15.3 (Pin_3), J16.4 (Pin_4)
- new net HV-5V: J15.5 (Pin_5), J16.6 (Pin_6)
Changed lines of the file:
@@
 $Descr A4 11693 8268
 encoding utf-8
-Sheet 10 11
+Sheet 9 10
 Title ""
 Date ""
@@
 	0    -1   -1   0
 $EndComp
-Text HLabel 8050 2250 0    50   Input ~ 0
+Text HLabel 7700 2350 0    50   Input ~ 0
 ADC_CH0
-Text HLabel 8050 2550 0    50   Input ~ 0
+Text HLabel 7700 2650 0    50   Input ~ 0
 ADC_CH1
 $Comp
@@
 	8500 2250 8900 2250
 Wire Wire Line
-	8150 2250 8050 2250
+	8150 2250 8100 2250
 Wire Wire Line
 	8500 2450 8800 2450
@@
 	8500 2550 8900 2550
 Wire Wire Line
-	8150 2550 8050 2550
+	8150 2550 8100 2550
 Wire Wire Line
 	8500 2750 8800 2750
@@
 $Comp
 L Connector:TestPoint TP?
-U 1 1 5FA2656C
-P 5200 6200
-AR Path="/5F7A93EE/5FA2656C" Ref="TP?"  Part="1"
-AR Path="/5F8337DC/5FA2656C" Ref="TP41"  Part="1"
-AR Path="/5F7D6767/5FA2656C" Ref="TP?"  Part="1"
-F 0 "TP41" V 5200 6388 50  0000 L CNN
-F 1 "TestPoint" V 5245 6388 50  0001 L CNN
-F 2 "TestPoint:TestPoint_THTPad_D1.5mm_Drill0.7mm" H 5400 6200 50  0001 C CNN
-F 3 "~" H 5400 6200 50  0001 C CNN
-	1    5200 6200
-	0    1    1    0
-$EndComp
-$Comp
-L Connector:TestPoint TP?
-U 1 1 5FA265F6
-P 5200 6300
-AR Path="/5F7A93EE/5FA265F6" Ref="TP?"  Part="1"
-AR Path="/5F8337DC/5FA265F6" Ref="TP42"  Part="1"
-AR Path="/5F7D6767/5FA265F6" Ref="TP?"  Part="1"
-F 0 "TP42" V 5200 6488 50  0000 L CNN
-F 1 "TestPoint" V 5245 6488 50  0001 L CNN
-F 2 "TestPoint:TestPoint_THTPad_D1.5mm_Drill0.7mm" H 5400 6300 50  0001 C CNN
-F 3 "~" H 5400 6300 50  0001 C CNN
-	1    5200 6300
-	0    1    1    0
-$EndComp
-$Comp
-L Connector:TestPoint TP?
 U 1 1 5FA26682
 P 5200 6400
@@
 Wire Wire Line
 	3750 7000 3750 7250
+$Comp
+L Connector:TestPoint TP?
+U 1 1 5FB6AB77
+P 8050 2250
+AR Path="/5F7A93EE/5FB6AB77" Ref="TP?"  Part="1"
+AR Path="/5F8337DC/5FB6AB77" Ref="TP40"  Part="1"
+AR Path="/5F7D6767/5FB6AB77" Ref="TP?"  Part="1"
+F 0 "TP40" V 8050 2438 50  0000 L CNN
+F 1 "TestPoint" V 8095 2438 50  0001 L CNN
+F 2 "TestPoint:TestPoint_THTPad_D1.5mm_Drill0.7mm" H 8250 2250 50  0001 C CNN
+F 3 "~" H 8250 2250 50  0001 C CNN
+	1    8050 2250
+	0    -1   -1   0
+$EndComp
+$Comp
+L Connector:TestPoint TP?
+U 1 1 5FB73BA5
+P 8050 2550
+AR Path="/5F7A93EE/5FB73BA5" Ref="TP?"  Part="1"
+AR Path="/5F8337DC/5FB73BA5" Ref="TP41"  Part="1"
+AR Path="/5F7D6767/5FB73BA5" Ref="TP?"  Part="1"
+F 0 "TP41" V 8050 2738 50  0000 L CNN
+F 1 "TestPoint" V 8095 2738 50  0001 L CNN
+F 2 "TestPoint:TestPoint_THTPad_D1.5mm_Drill0.7mm" H 8250 2550 50  0001 C CNN
+F 3 "~" H 8250 2550 50  0001 C CNN
+	1    8050 2550
+	0    -1   -1   0
+$EndComp
+Wire Wire Line
+	8100 2650 8100 2550
+Connection ~ 8100 2550
+Wire Wire Line
+	8100 2550 8050 2550
+Wire Wire Line
+	8100 2350 8100 2250
+Connection ~ 8100 2250
+Wire Wire Line
+	8100 2250 8050 2250
+$Comp
+L Connector_Generic:Conn_02x03_Odd_Even J15
+U 1 1 5FB4E18D
+P 1750 6200
+F 0 "J15" H 1800 6517 50  0000 C CNN
+F 1 "Conn_02x03_Odd_Even" H 1800 6426 50  0000 C CNN
+F 2 "Connector_PinSocket_2.54mm:PinSocket_2x03_P2.54mm_Vertical" H 1750 6200 50  0001 C CNN
+F 3 "~" H 1750 6200 50  0001 C CNN
+	1    1750 6200
+	1    0    0    -1
+$EndComp
+$Comp
+L power_my:HVGND #PWR?
+U 1 1 5FB4E463
+P 1550 5950
+AR Path="/5FB4E463" Ref="#PWR?"  Part="1"
+AR Path="/5F8337DC/5FB4E463" Ref="#PWR0262"  Part="1"
+F 0 "#PWR0262" H 1550 5900 50  0001 C CNN
+F 1 "HVGND" H 1550 5777 50  0000 C CNN
+F 2 "" H 1550 5950 50  0001 C CNN
+F 3 "" H 1550 5950 50  0001 C CNN
+	1    1550 5950
+	-1   0    0    1
+$EndComp
+$Comp
+L power_my:HVGND #PWR?
+U 1 1 5FB4EF2E
+P 2050 5950
+AR Path="/5FB4EF2E" Ref="#PWR?"  Part="1"
+AR Path="/5F8337DC/5FB4EF2E" Ref="#PWR0263"  Part="1"
+F 0 "#PWR0263" H 2050 5900 50  0001 C CNN
+F 1 "HVGND" H 2050 5777 50  0000 C CNN
+F 2 "" H 2050 5950 50  0001 C CNN
+F 3 "" H 2050 5950 50  0001 C CNN
+	1    2050 5950
+	-1   0    0    1
+$EndComp
+Text Label 7750 2350 0    50   ~ 0
+ADC_CH0
+Text Label 7750 2650 0    50   ~ 0
+ADC_CH1
+Wire Wire Line
+	7700 2350 8100 2350
+Wire Wire Line
+	7700 2650 8100 2650
+Text Label 2050 6200 0    50   ~ 0
+ADC_CH0
+Text Label 2050 6300 0    50   ~ 0
+ADC_CH1
+$Comp
+L power_my:HV+5V #PWR?
+U 1 1 5FB85092
+P 1250 6200
+AR Path="/5FB035A9/5FB85092" Ref="#PWR?"  Part="1"
+AR Path="/5F479892/5FB85092" Ref="#PWR?"  Part="1"
+AR Path="/5F8337DC/5FB85092" Ref="#PWR0260"  Part="1"
+F 0 "#PWR0260" H 1250 6050 50  0001 C CNN
+F 1 "HV+5V" H 1255 6373 50  0000 C CNN
+F 2 "" H 1250 6200 50  0001 C CNN
+F 3 "" H 1250 6200 50  0001 C CNN
+	1    1250 6200
+	1    0    0    -1
+$EndComp
+$Comp
+L power_my:HV-5V #PWR?
+U 1 1 5FB85098
+P 1250 6300
+AR Path="/5FB035A9/5FB85098" Ref="#PWR?"  Part="1"
+AR Path="/5F479892/5FB85098" Ref="#PWR?"  Part="1"
+AR Path="/5F8337DC/5FB85098" Ref="#PWR0261"  Part="1"
+F 0 "#PWR0261" H 1250 6150 50  0001 C CNN
+F 1 "HV-5V" H 1255 6473 50  0000 C CNN
+F 2 "" H 1250 6300 50  0001 C CNN
+F 3 "" H 1250 6300 50  0001 C CNN
+	1    1250 6300
+	-1   0    0    1
+$EndComp
+Wire Wire Line
+	1250 6200 1550 6200
+Wire Wire Line
+	1550 6300 1250 6300
+$Comp
+L Connector_Generic:Conn_02x03_Odd_Even J16
+U 1 1 5FBA5274
+P 1850 7050
+F 0 "J16" H 1900 7367 50  0000 C CNN
+F 1 "Conn_02x03_Odd_Even" H 1900 7276 50  0000 C CNN
+F 2 "Connector_PinSocket_2.54mm:PinSocket_2x03_P2.54mm_Vertical" H 1850 7050 50  0001 C CNN
+F 3 "~" H 1850 7050 50  0001 C CNN
+	1    1850 7050
+	-1   0    0    -1
+$EndComp
+$Comp
+L power_my:HVGND #PWR?
+U 1 1 5FBA527B
+P 1550 6800
+AR Path="/5FBA527B" Ref="#PWR?"  Part="1"
+AR Path="/5F8337DC/5FBA527B" Ref="#PWR0266"  Part="1"
+F 0 "#PWR0266" H 1550 6750 50  0001 C CNN
+F 1 "HVGND" H 1550 6627 50  0000 C CNN
+F 2 "" H 1550 6800 50  0001 C CNN
+F 3 "" H 1550 6800 50  0001 C CNN
+	1    1550 6800
+	-1   0    0    1
+$EndComp
+$Comp
+L power_my:HVGND #PWR?
+U 1 1 5FBA5281
+P 2050 6800
+AR Path="/5FBA5281" Ref="#PWR?"  Part="1"
+AR Path="/5F8337DC/5FBA5281" Ref="#PWR0267"  Part="1"
+F 0 "#PWR0267" H 2050 6750 50  0001 C CNN
+F 1 "HVGND" H 2050 6627 50  0000 C CNN
+F 2 "" H 2050 6800 50  0001 C CNN
+F 3 "" H 2050 6800 50  0001 C CNN
+	1    2050 6800
+	-1   0    0    1
+$EndComp
+Text Label 2050 7050 0    50   ~ 0
+ADC_CH0
+Text Label 2050 7150 0    50   ~ 0
+ADC_CH1
+$Comp
+L power_my:HV+5V #PWR?
+U 1 1 5FBA5289
+P 1250 7050
+AR Path="/5FB035A9/5FBA5289" Ref="#PWR?"  Part="1"
+AR Path="/5F479892/5FBA5289" Ref="#PWR?"  Part="1"
+AR Path="/5F8337DC/5FBA5289" Ref="#PWR0264"  Part="1"
+F 0 "#PWR0264" H 1250 6900 50  0001 C CNN
+F 1 "HV+5V" H 1255 7223 50  0000 C CNN
+F 2 "" H 1250 7050 50  0001 C CNN
+F 3 "" H 1250 7050 50  0001 C CNN
+	1    1250 7050
+	1    0    0    -1
+$EndComp
+$Comp
+L power_my:HV-5V #PWR?
+U 1 1 5FBA528F
+P 1250 7150
+AR Path="/5FB035A9/5FBA528F" Ref="#PWR?"  Part="1"
+AR Path="/5F479892/5FBA528F" Ref="#PWR?"  Part="1"
+AR Path="/5F8337DC/5FBA528F" Ref="#PWR0265"  Part="1"
+F 0 "#PWR0265" H 1250 7000 50  0001 C CNN
+F 1 "HV-5V" H 1255 7323 50  0000 C CNN
+F 2 "" H 1250 7150 50  0001 C CNN
+F 3 "" H 1250 7150 50  0001 C CNN
+	1    1250 7150
+	-1   0    0    1
+$EndComp
+Wire Wire Line
+	1250 7050 1550 7050
+Wire Wire Line
+	1550 7150 1250 7150
+Wire Wire Line
+	1550 5950 1550 6100
+Wire Wire Line
+	2050 5950 2050 6100
+Wire Wire Line
+	2050 6950 2050 6800
+Wire Wire Line
+	1550 6950 1550 6800
 $EndSCHEMATC

Commit message: - PCB WiP
Parts:
- added TP10, TP11, TP12, TP42, TP5, TP6, TP7, TP8, TP9: TestPoint, TestPoint:TestPoint_THTPad_D1.5mm_Drill0.7mm, symbol Connector:TestPoint
Connections:
- net ADC_CH1: now also TP11.1, TP12.1
- net HV+5V: now also TP5.1, TP6.1
- net HV-5V: now also TP7.1, TP8.1
- net HVGND: now also TP10.1, TP42.1, TP9.1
Changed lines of the file:
@@
 Wire Wire Line
 	1550 6950 1550 6800
+$Comp
+L Connector:TestPoint TP?
+U 1 1 5FC005CB
+P 8450 5250
+AR Path="/5F7A93EE/5FC005CB" Ref="TP?"  Part="1"
+AR Path="/5F8337DC/5FC005CB" Ref="TP6"  Part="1"
+AR Path="/5F7D6767/5FC005CB" Ref="TP?"  Part="1"
+F 0 "TP6" V 8450 5438 50  0000 L CNN
+F 1 "TestPoint" V 8495 5438 50  0001 L CNN
+F 2 "TestPoint:TestPoint_THTPad_D1.5mm_Drill0.7mm" H 8650 5250 50  0001 C CNN
+F 3 "~" H 8650 5250 50  0001 C CNN
+	1    8450 5250
+	0    -1   -1   0
+$EndComp
+$Comp
+L Connector:TestPoint TP?
+U 1 1 5FC00A9D
+P 8450 5350
+AR Path="/5F7A93EE/5FC00A9D" Ref="TP?"  Part="1"
+AR Path="/5F8337DC/5FC00A9D" Ref="TP8"  Part="1"
+AR Path="/5F7D6767/5FC00A9D" Ref="TP?"  Part="1"
+F 0 "TP8" V 8450 5538 50  0000 L CNN
+F 1 "TestPoint" V 8495 5538 50  0001 L CNN
+F 2 "TestPoint:TestPoint_THTPad_D1.5mm_Drill0.7mm" H 8650 5350 50  0001 C CNN
+F 3 "~" H 8650 5350 50  0001 C CNN
+	1    8450 5350
+	0    -1   -1   0
+$EndComp
+$Comp
+L Connector:TestPoint TP?
+U 1 1 5FC00B43
+P 8450 5450
+AR Path="/5F7A93EE/5FC00B43" Ref="TP?"  Part="1"
+AR Path="/5F8337DC/5FC00B43" Ref="TP10"  Part="1"
+AR Path="/5F7D6767/5FC00B43" Ref="TP?"  Part="1"
+F 0 "TP10" V 8450 5638 50  0000 L CNN
+F 1 "TestPoint" V 8495 5638 50  0001 L CNN
+F 2 "TestPoint:TestPoint_THTPad_D1.5mm_Drill0.7mm" H 8650 5450 50  0001 C CNN
+F 3 "~" H 8650 5450 50  0001 C CNN
+	1    8450 5450
+	0    -1   -1   0
+$EndComp
+$Comp
+L Connector:TestPoint TP?
+U 1 1 5FC00BE7
+P 8450 5550
+AR Path="/5F7A93EE/5FC00BE7" Ref="TP?"  Part="1"
+AR Path="/5F8337DC/5FC00BE7" Ref="TP12"  Part="1"
+AR Path="/5F7D6767/5FC00BE7" Ref="TP?"  Part="1"
+F 0 "TP12" V 8450 5738 50  0000 L CNN
+F 1 "TestPoint" V 8495 5738 50  0001 L CNN
+F 2 "TestPoint:TestPoint_THTPad_D1.5mm_Drill0.7mm" H 8650 5550 50  0001 C CNN
+F 3 "~" H 8650 5550 50  0001 C CNN
+	1    8450 5550
+	0    -1   -1   0
+$EndComp
+$Comp
+L power_my:HVGND #PWR?
+U 1 1 5FC00E04
+P 8850 5450
+AR Path="/5FC00E04" Ref="#PWR?"  Part="1"
+AR Path="/5F8337DC/5FC00E04" Ref="#PWR0278"  Part="1"
+F 0 "#PWR0278" H 8850 5400 50  0001 C CNN
+F 1 "HVGND" H 8850 5277 50  0000 C CNN
+F 2 "" H 8850 5450 50  0001 C CNN
+F 3 "" H 8850 5450 50  0001 C CNN
+	1    8850 5450
+	1    0    0    -1
+$EndComp
+$Comp
+L power_my:HV+5V #PWR?
+U 1 1 5FC01AB4
+P 9100 5250
+AR Path="/5FB035A9/5FC01AB4" Ref="#PWR?"  Part="1"
+AR Path="/5F479892/5FC01AB4" Ref="#PWR?"  Part="1"
+AR Path="/5F8337DC/5FC01AB4" Ref="#PWR013"  Part="1"
+F 0 "#PWR013" H 9100 5100 50  0001 C CNN
+F 1 "HV+5V" H 9105 5423 50  0000 C CNN
+F 2 "" H 9100 5250 50  0001 C CNN
+F 3 "" H 9100 5250 50  0001 C CNN
+	1    9100 5250
+	1    0    0    -1
+$EndComp
+$Comp
+L power_my:HV-5V #PWR?
+U 1 1 5FC01ABA
+P 9100 5350
+AR Path="/5FB035A9/5FC01ABA" Ref="#PWR?"  Part="1"
+AR Path="/5F479892/5FC01ABA" Ref="#PWR?"  Part="1"
+AR Path="/5F8337DC/5FC01ABA" Ref="#PWR0276"  Part="1"
+F 0 "#PWR0276" H 9100 5200 50  0001 C CNN
+F 1 "HV-5V" H 9105 5523 50  0000 C CNN
+F 2 "" H 9100 5350 50  0001 C CNN
+F 3 "" H 9100 5350 50  0001 C CNN
+	1    9100 5350
+	-1   0    0    1
+$EndComp
+$Comp
+L Connector:TestPoint TP?
+U 1 1 5FC2367C
+P 7550 5550
+AR Path="/5F7A93EE/5FC2367C" Ref="TP?"  Part="1"
+AR Path="/5F8337DC/5FC2367C" Ref="TP11"  Part="1"
+AR Path="/5F7D6767/5FC2367C" Ref="TP?"  Part="1"
+F 0 "TP11" V 7550 5738 50  0000 L CNN
+F 1 "TestPoint" V 7595 5738 50  0001 L CNN
+F 2 "TestPoint:TestPoint_THTPad_D1.5mm_Drill0.7mm" H 7750 5550 50  0001 C CNN
+F 3 "~" H 7750 5550 50  0001 C CNN
+	1    7550 5550
+	0    1    1    0
+$EndComp
+$Comp
+L Connector:TestPoint TP?
+U 1 1 5FC23683
+P 7550 5450
+AR Path="/5F7A93EE/5FC23683" Ref="TP?"  Part="1"
+AR Path="/5F8337DC/5FC23683" Ref="TP9"  Part="1"
+AR Path="/5F7D6767/5FC23683" Ref="TP?"  Part="1"
+F 0 "TP9" V 7550 5638 50  0000 L CNN
+F 1 "TestPoint" V 7595 5638 50  0001 L CNN
+F 2 "TestPoint:TestPoint_THTPad_D1.5mm_Drill0.7mm" H 7750 5450 50  0001 C CNN
+F 3 "~" H 7750 5450 50  0001 C CNN
+	1    7550 5450
+	0    1    1    0
+$EndComp
+$Comp
+L Connector:TestPoint TP?
+U 1 1 5FC2368A
+P 7550 5350
+AR Path="/5F7A93EE/5FC2368A" Ref="TP?"  Part="1"
+AR Path="/5F8337DC/5FC2368A" Ref="TP7"  Part="1"
+AR Path="/5F7D6767/5FC2368A" Ref="TP?"  Part="1"
+F 0 "TP7" V 7550 5538 50  0000 L CNN
+F 1 "TestPoint" V 7595 5538 50  0001 L CNN
+F 2 "TestPoint:TestPoint_THTPad_D1.5mm_Drill0.7mm" H 7750 5350 50  0001 C CNN
+F 3 "~" H 7750 5350 50  0001 C CNN
+	1    7550 5350
+	0    1    1    0
+$EndComp
+$Comp
+L Connector:TestPoint TP?
+U 1 1 5FC23691
+P 7550 5250
+AR Path="/5F7A93EE/5FC23691" Ref="TP?"  Part="1"
+AR Path="/5F8337DC/5FC23691" Ref="TP5"  Part="1"
+AR Path="/5F7D6767/5FC23691" Ref="TP?"  Part="1"
+F 0 "TP5" V 7550 5438 50  0000 L CNN
+F 1 "TestPoint" V 7595 5438 50  0001 L CNN
+F 2 "TestPoint:TestPoint_THTPad_D1.5mm_Drill0.7mm" H 7750 5250 50  0001 C CNN
+F 3 "~" H 7750 5250 50  0001 C CNN
+	1    7550 5250
+	0    1    1    0
+$EndComp
+$Comp
+L power_my:HVGND #PWR?
+U 1 1 5FC4E67E
+P 7150 5450
+AR Path="/5FC4E67E" Ref="#PWR?"  Part="1"
+AR Path="/5F8337DC/5FC4E67E" Ref="#PWR0277"  Part="1"
+F 0 "#PWR0277" H 7150 5400 50  0001 C CNN
+F 1 "HVGND" H 7150 5277 50  0000 C CNN
+F 2 "" H 7150 5450 50  0001 C CNN
+F 3 "" H 7150 5450 50  0001 C CNN
+	1    7150 5450
+	1    0    0    -1
+$EndComp
+$Comp
+L power_my:HV+5V #PWR?
+U 1 1 5FC4E684
+P 6900 5250
+AR Path="/5FB035A9/5FC4E684" Ref="#PWR?"  Part="1"
+AR Path="/5F479892/5FC4E684" Ref="#PWR?"  Part="1"
+AR Path="/5F8337DC/5FC4E684" Ref="#PWR012"  Part="1"
+F 0 "#PWR012" H 6900 5100 50  0001 C CNN
+F 1 "HV+5V" H 6905 5423 50  0000 C CNN
+F 2 "" H 6900 5250 50  0001 C CNN
+F 3 "" H 6900 5250 50  0001 C CNN
+	1    6900 5250
+	1    0    0    -1
+$EndComp
+$Comp
+L power_my:HV-5V #PWR?
+U 1 1 5FC4E68A
+P 6900 5350
+AR Path="/5FB035A9/5FC4E68A" Ref="#PWR?"  Part="1"
+AR Path="/5F479892/5FC4E68A" Ref="#PWR?"  Part="1"
+AR Path="/5F8337DC/5FC4E68A" Ref="#PWR014"  Part="1"
+F 0 "#PWR014" H 6900 5200 50  0001 C CNN
+F 1 "HV-5V" H 6905 5523 50  0000 C CNN
+F 2 "" H 6900 5350 50  0001 C CNN
+F 3 "" H 6900 5350 50  0001 C CNN
+	1    6900 5350
+	-1   0    0    1
+$EndComp
+Wire Wire Line
+	7550 5250 6900 5250
+Wire Wire Line
+	6900 5350 7550 5350
+Wire Wire Line
+	7550 5450 7150 5450
+Wire Wire Line
+	9100 5250 8450 5250
+Wire Wire Line
+	8450 5350 9100 5350
+Wire Wire Line
+	8850 5450 8450 5450
+$Comp
+L Connector:TestPoint TP?
+U 1 1 5FCBE9EF
+P 9800 5450
+AR Path="/5F7A93EE/5FCBE9EF" Ref="TP?"  Part="1"
+AR Path="/5F8337DC/5FCBE9EF" Ref="TP42"  Part="1"
+AR Path="/5F7D6767/5FCBE9EF" Ref="TP?"  Part="1"
+F 0 "TP42" V 9800 5638 50  0000 L CNN
+F 1 "TestPoint" V 9845 5638 50  0001 L CNN
+F 2 "TestPoint:TestPoint_THTPad_D1.5mm_Drill0.7mm" H 10000 5450 50  0001 C CNN
+F 3 "~" H 10000 5450 50  0001 C CNN
+	1    9800 5450
+	0    -1   -1   0
+$EndComp
+$Comp
+L power_my:HVGND #PWR?
+U 1 1 5FCBEACD
+P 9900 5450
+AR Path="/5FCBEACD" Ref="#PWR?"  Part="1"
+AR Path="/5F8337DC/5FCBEACD" Ref="#PWR0279"  Part="1"
+F 0 "#PWR0279" H 9900 5400 50  0001 C CNN
+F 1 "HVGND" H 9900 5277 50  0000 C CNN
+F 2 "" H 9900 5450 50  0001 C CNN
+F 3 "" H 9900 5450 50  0001 C CNN
+	1    9900 5450
+	1    0    0    -1
+$EndComp
+Wire Wire Line
+	9800 5450 9900 5450
+Text Label 8450 5550 0    50   ~ 0
+ADC_CH1
+Text Label 7550 5550 2    50   ~ 0
+ADC_CH1
 $EndSCHEMATC
