File: communication.sch (KiCad schematic (older format))
At the start: 0 parts

Commit message: - high side (supply, MCU) - low side MCU - much small changes
Parts:
- added C? (x3): 100n, Capacitor_SMD:C_0603_1608Metric_Pad1.05x0.95mm_HandSolder, symbol Device:C_Small
- added D? (x2): QEE113, miscellaneous_my:ONsemi_QEE113, symbol Device:LED_ALT
- added Q? (x4): BSS138, Package_TO_SOT_SMD:SOT-23, symbol Transistor_FET:BSS138
- added R? (x4): 470R, Resistor_SMD:R_0603_1608Metric_Pad1.05x0.95mm_HandSolder, symbol Device:R_Small
- added R? (x4): 1k, Resistor_SMD:R_0603_1608Metric_Pad1.05x0.95mm_HandSolder, symbol Device:R_Small
- added R? (x2): 0R, Resistor_SMD:R_0603_1608Metric_Pad1.05x0.95mm_HandSolder, symbol Device:R_Small
- added U? (x2): QSE159, OptoDevice:ONSemi_QSE15x, symbol Interface_Optical:QSE159
- added U? (x2): SN74LVC1G14DRL, Package_TO_SOT_SMD:SOT-553, symbol 74xGxx:SN74LVC1G14DRL
- added U?: OPTI128, miscellaneous_my:OPTI12x, symbol miscellaneous:OPTI128
Connections:
- net HV_UART_RX: now also Q?.3 (D), R?.2, R?.2, U?.4
- net HV_UART_TX: now also R?.1
- net UART_RX: now also Q?.3 (D), R?.2, R?.2, U?.4
- net UART_TX: now also R?.2
- new net: D?.1 (K), Q?.3 (D)
- new net: D?.2 (A), R?.2
- new net: Q?.1 (G), R?.1, R?.2, U?.2, U?.2 (Out)
- new net: Q?.1 (G), R?.1
- new net: Q?.1 (G), R?.2
- new net +3V3: R?.1, R?.1, U?.5 (VCC)
- new net +5V: C?.2, C?.2, R?.1, U?.3 (Vcc), U?.4 (VCC)
- new net A_HV: D?.2 (A), R?.2, U?.1 (A)
- new net GND: C?.1, C?.1, C?.1, Q?.2 (S), Q?.2 (S), U?.1 (GND), U?.3 (GND), U?.5 (GND)
- new net HV+3V3: R?.1, R?.1, U?.5 (VCC)
- new net HV+5V: C?.2, R?.1, U?.3 (Vcc)
- new net HVGND: Q?.2 (S), Q?.2 (S), U?.1 (GND), U?.3 (GND)
- new net K_HV: D?.1 (K), Q?.3 (D), U?.2 (K)
- new net RX_LV: Q?.1 (G), R?.1, R?.2, U?.2, U?.2 (Out), U?.3 (OUT)
Other:
- note added: "OPTI128\nIf typ. 7.5 mA Uf max 1.5 V\nOpen collector output\nOutput supply 5V +/- 0.5V"

Commit message: - final schematic
Parts:
- gave numbers to parts that had none: 24

Commit message: - PCB progress
Parts:
- C150, C151, C152: footprint Capacitor_SMD:C_0603_1608Metric_Pad1.05x0.95mm_HandSolder -> Capacitor_SMD:C_0603_1608Metric
Connections:
- net GND: now also Q20.2 (S); no longer C152.1, Q19.2 (S)
- net HVGND: now also C152.1, Q19.2 (S); no longer Q20.2 (S)
Other:
- moved on the sheet: C150, C152, U28
Changed lines of the file:
@@
 L power:GND #PWR?
 U 1 1 5FC526B7
-P 4800 2050
+P 4950 2050
 AR Path="/5F40DCB9/5FC526B7" Ref="#PWR?"  Part="1"
 AR Path="/5F618AB9/5FC526B7" Ref="#PWR?"  Part="1"
@@
 AR Path="/5F620813/5FC526B7" Ref="#PWR?"  Part="1"
 AR Path="/5F82F010/5FC526B7" Ref="#PWR0193"  Part="1"
-F 0 "#PWR0193" H 4800 1890 50  0001 C CNN
-F 1 "GND" H 4800 1950 39  0000 C TNN
-F 2 "" H 4800 2050 50  0001 C CNN
-F 3 "" H 4800 2050 50  0001 C CNN
-	1    4800 2050
+F 0 "#PWR0193" H 4950 1890 50  0001 C CNN
+F 1 "GND" H 4950 1950 39  0000 C TNN
+F 2 "" H 4950 2050 50  0001 C CNN
+F 3 "" H 4950 2050 50  0001 C CNN
+	1    4950 2050
 	1    0    0    -1
 $EndComp
@@
 L Device:C_Small C?
 U 1 1 5FC52923
-P 5000 1050
+P 5150 1050
 AR Path="/5F40DCB9/5FC52923" Ref="C?"  Part="1"
 AR Path="/5F463F4C/5FC52923" Ref="C?"  Part="1"
@@
 AR Path="/5FB035A9/5FC52923" Ref="C?"  Part="1"
 AR Path="/5F82F010/5FC52923" Ref="C150"  Part="1"
-F 0 "C150" H 5000 950 50  0000 R BNN
-F 1 "100n" H 5000 1150 50  0000 R TNN
-F 2 "Capacitor_SMD:C_0603_1608Metric_Pad1.05x0.95mm_HandSolder" H 5000 1050 50  0001 C CNN
-F 3 "~" H 5000 1050 50  0001 C CNN
-	1    5000 1050
+F 0 "C150" H 5150 950 50  0000 R BNN
+F 1 "100n" H 5150 1150 50  0000 R TNN
+F 2 "Capacitor_SMD:C_0603_1608Metric" H 5150 1050 50  0001 C CNN
+F 3 "~" H 5150 1050 50  0001 C CNN
+	1    5150 1050
 	-1   0    0    1
 $EndComp
@@
 L power:GND #PWR?
 U 1 1 5FC52934
-P 5000 1150
+P 5150 1150
 AR Path="/5F40DCB9/5FC52934" Ref="#PWR?"  Part="1"
 AR Path="/5F618AB9/5FC52934" Ref="#PWR?"  Part="1"
@@
 AR Path="/5F620813/5FC52934" Ref="#PWR?"  Part="1"
 AR Path="/5F82F010/5FC52934" Ref="#PWR0192"  Part="1"
-F 0 "#PWR0192" H 5000 990 50  0001 C CNN
-F 1 "GND" H 5000 1050 39  0000 C TNN
-F 2 "" H 5000 1150 50  0001 C CNN
-F 3 "" H 5000 1150 50  0001 C CNN
-	1    5000 1150
-	1    0    0    -1
-$EndComp
-Wire Wire Line
-	4800 1250 4800 900
-Wire Wire Line
-	4800 900  5000 900
-Wire Wire Line
-	5000 900  5000 950
+F 0 "#PWR0192" H 5150 990 50  0001 C CNN
+F 1 "GND" H 5150 1050 39  0000 C TNN
+F 2 "" H 5150 1150 50  0001 C CNN
+F 3 "" H 5150 1150 50  0001 C CNN
+	1    5150 1150
+	1    0    0    -1
+$EndComp
+Wire Wire Line
+	4950 1250 4950 900
+Wire Wire Line
+	4950 900  5150 900
+Wire Wire Line
+	5150 900  5150 950
 $Comp
 L power:+3V3 #PWR?
@@
 $EndComp
 Wire Wire Line
-	4800 850  4800 900
-Connection ~ 4800 900
+	4950 850  4950 900
+Connection ~ 4950 900
 $Comp
 L power_my:HV+5V #PWR?
@@
 L power:+5V #PWR?
 U 1 1 5FC7B7D3
-P 4800 850
+P 4950 850
 AR Path="/5F40DCB9/5FC7B7D3" Ref="#PWR?"  Part="1"
 AR Path="/5F479892/5FC7B7D3" Ref="#PWR?"  Part="1"
 AR Path="/5F620813/5FC7B7D3" Ref="#PWR?"  Part="1"
 AR Path="/5F82F010/5FC7B7D3" Ref="#PWR0191"  Part="1"
-F 0 "#PWR0191" H 4800 700 50  0001 C CNN
-F 1 "+5V" H 4815 1023 50  0000 C CNN
-F 2 "" H 4800 850 50  0001 C CNN
-F 3 "" H 4800 850 50  0001 C CNN
-	1    4800 850
+F 0 "#PWR0191" H 4950 700 50  0001 C CNN
+F 1 "+5V" H 4965 1023 50  0000 C CNN
+F 2 "" H 4950 850 50  0001 C CNN
+F 3 "" H 4950 850 50  0001 C CNN
+	1    4950 850
 	1    0    0    -1
 $EndComp
@@
 L miscellaneous:OPTI128 U28
 U 1 1 5FC8BE03
-P 4800 1650
-F 0 "U28" H 5300 1900 50  0000 L CNN
-F 1 "OPTI128" H 5300 1800 50  0000 L CNN
-F 2 "miscellaneous_my:OPTI12x" H 4850 950 50  0001 C CNN
-F 3 "https://toshiba.semicon-storage.com/info/docget.jsp?did=53548&prodName=TLP2770" H 5850 500 50  0001 C CNN
-	1    4800 1650
+P 4950 1650
+F 0 "U28" H 5450 1900 50  0000 L CNN
+F 1 "OPTI128" H 5450 1800 50  0000 L CNN
+F 2 "miscellaneous_my:OPTI12x" H 5000 950 50  0001 C CNN
+F 3 "https://toshiba.semicon-storage.com/info/docget.jsp?did=53548&prodName=TLP2770" H 6000 500 50  0001 C CNN
+	1    4950 1650
 	1    0    0    -1
 $EndComp
@@
 $EndComp
 $Comp
-L power_my:HVGND #PWR?
-U 1 1 5F9EDFF6
-P 5450 6650
-AR Path="/5F9EDFF6" Ref="#PWR?"  Part="1"
-AR Path="/5F82F010/5F9EDFF6" Ref="#PWR0212"  Part="1"
-F 0 "#PWR0212" H 5450 6600 50  0001 C CNN
-F 1 "HVGND" H 5450 6477 50  0000 C CNN
-F 2 "" H 5450 6650 50  0001 C CNN
-F 3 "" H 5450 6650 50  0001 C CNN
-	1    5450 6650
-	1    0    0    -1
-$EndComp
-$Comp
 L Device:R_Small R?
 U 1 1 5F9EE003
@@
 Text Label 3800 3850 0    50   ~ 0
 K_HV
-Text Label 5950 1650 0    50   ~ 0
+Text Label 6100 1650 0    50   ~ 0
 RX_LV
 Wire Wire Line
 	3800 3450 3800 3550
-Text Label 3900 1500 0    50   ~ 0
+Text Label 4050 1500 0    50   ~ 0
 A_HV
-Text Label 3900 1800 0    50   ~ 0
+Text Label 4050 1800 0    50   ~ 0
 K_HV
 Wire Wire Line
-	4100 1500 3900 1500
-Wire Wire Line
-	4100 1800 3900 1800
+	4250 1500 4050 1500
+Wire Wire Line
+	4250 1800 4050 1800
 $Comp
 L Device:C_Small C?
@@
 F 0 "C151" H 5900 3100 50  0000 R BNN
 F 1 "100n" H 5900 3300 50  0000 R TNN
-F 2 "Capacitor_SMD:C_0603_1608Metric_Pad1.05x0.95mm_HandSolder" H 5900 3200 50  0001 C CNN
+F 2 "Capacitor_SMD:C_0603_1608Metric" H 5900 3200 50  0001 C CNN
 F 3 "~" H 5900 3200 50  0001 C CNN
 	1    5900 3200
@@
 RX_LV
 Wire Wire Line
-	5350 1650 5950 1650
+	5500 1650 6100 1650
 Connection ~ 6300 3700
 Wire Wire Line
@@
 	1    0    0    -1
 $EndComp
-$Comp
-L power:GND #PWR?
-U 1 1 5FA3BE46
-P 2600 5750
-AR Path="/5F40DCB9/5FA3BE46" Ref="#PWR?"  Part="1"
-AR Path="/5F618AB9/5FA3BE46" Ref="#PWR?"  Part="1"
-AR Path="/5FA3BE46" Ref="#PWR?"  Part="1"
-AR Path="/5F620813/5FA3BE46" Ref="#PWR?"  Part="1"
-AR Path="/5F82F010/5FA3BE46" Ref="#PWR0207"  Part="1"
-F 0 "#PWR0207" H 2600 5590 50  0001 C CNN
-F 1 "GND" H 2600 5650 39  0000 C TNN
-F 2 "" H 2600 5750 50  0001 C CNN
-F 3 "" H 2600 5750 50  0001 C CNN
-	1    2600 5750
-	1    0    0    -1
-$EndComp
 Wire Wire Line
 	2150 5350 2600 5350
@@
 L Device:C_Small C?
 U 1 1 5FA3C84B
-P 4000 5600
+P 4000 5550
 AR Path="/5F40DCB9/5FA3C84B" Ref="C?"  Part="1"
 AR Path="/5F463F4C/5FA3C84B" Ref="C?"  Part="1"
@@
 AR Path="/5FB035A9/5FA3C84B" Ref="C?"  Part="1"
 AR Path="/5F82F010/5FA3C84B" Ref="C152"  Part="1"
-F 0 "C152" H 4000 5500 50  0000 R BNN
-F 1 "100n" H 4000 5700 50  0000 R TNN
-F 2 "Capacitor_SMD:C_0603_1608Metric_Pad1.05x0.95mm_HandSolder" H 4000 5600 50  0001 C CNN
-F 3 "~" H 4000 5600 50  0001 C CNN
-	1    4000 5600
+F 0 "C152" H 4000 5450 50  0000 R BNN
+F 1 "100n" H 4000 5650 50  0000 R TNN
+F 2 "Capacitor_SMD:C_0603_1608Metric" H 4000 5550 50  0001 C CNN
+F 3 "~" H 4000 5550 50  0001 C CNN
+	1    4000 5550
 	-1   0    0    1
 $EndComp
-$Comp
-L power:GND #PWR?
-U 1 1 5FA3C852
-P 4000 5700
-AR Path="/5F40DCB9/5FA3C852" Ref="#PWR?"  Part="1"
-AR Path="/5F618AB9/5FA3C852" Ref="#PWR?"  Part="1"
-AR Path="/5FA3C852" Ref="#PWR?"  Part="1"
-AR Path="/5F620813/5FA3C852" Ref="#PWR?"  Part="1"
-AR Path="/5F82F010/5FA3C852" Ref="#PWR0206"  Part="1"
-F 0 "#PWR0206" H 4000 5540 50  0001 C CNN
-F 1 "GND" H 4000 5600 39  0000 C TNN
-F 2 "" H 4000 5700 50  0001 C CNN
-F 3 "" H 4000 5700 50  0001 C CNN
-	1    4000 5700
-	1    0    0    -1
-$EndComp
-Wire Wire Line
-	3800 5800 3800 5450
-Wire Wire Line
-	3800 5450 4000 5450
-Wire Wire Line
-	4000 5450 4000 5500
-Wire Wire Line
-	3800 5400 3800 5450
-Connection ~ 3800 5450
+Wire Wire Line
+	3800 5800 3800 5400
+Wire Wire Line
+	3800 5400 4000 5400
+Wire Wire Line
+	4000 5400 4000 5450
 $Comp
 L power_my:HV+5V #PWR?
@@
 Wire Notes Line
 	4200 6250 5300 6250
+$Comp
+L power_my:HVGND #PWR?
+U 1 1 5FAF3C3F
+P 4000 5650
+AR Path="/5FAF3C3F" Ref="#PWR?"  Part="1"
+AR Path="/5F82F010/5FAF3C3F" Ref="#PWR033"  Part="1"
+F 0 "#PWR033" H 4000 5600 50  0001 C CNN
+F 1 "HVGND" H 4000 5477 50  0000 C CNN
+F 2 "" H 4000 5650 50  0001 C CNN
+F 3 "" H 4000 5650 50  0001 C CNN
+	1    4000 5650
+	1    0    0    -1
+$EndComp
+Connection ~ 3800 5400
+$Comp
+L power_my:HVGND #PWR?
+U 1 1 5FAF749C
+P 2600 5750
+AR Path="/5FAF749C" Ref="#PWR?"  Part="1"
+AR Path="/5F82F010/5FAF749C" Ref="#PWR039"  Part="1"
+F 0 "#PWR039" H 2600 5700 50  0001 C CNN
+F 1 "HVGND" H 2600 5577 50  0000 C CNN
+F 2 "" H 2600 5750 50  0001 C CNN
+F 3 "" H 2600 5750 50  0001 C CNN
+	1    2600 5750
+	1    0    0    -1
+$EndComp
+$Comp
+L power:GND #PWR?
+U 1 1 5FAF97D0
+P 5450 6650
+AR Path="/5F40DCB9/5FAF97D0" Ref="#PWR?"  Part="1"
+AR Path="/5F618AB9/5FAF97D0" Ref="#PWR?"  Part="1"
+AR Path="/5FAF97D0" Ref="#PWR?"  Part="1"
+AR Path="/5F620813/5FAF97D0" Ref="#PWR?"  Part="1"
+AR Path="/5F82F010/5FAF97D0" Ref="#PWR0206"  Part="1"
+F 0 "#PWR0206" H 5450 6490 50  0001 C CNN
+F 1 "GND" H 5450 6550 39  0000 C TNN
+F 2 "" H 5450 6650 50  0001 C CNN
+F 3 "" H 5450 6650 50  0001 C CNN
+	1    5450 6650
+	1    0    0    -1
+$EndComp
+Wire Notes Line
+	4750 3550 4750 500
+Wire Notes Line
+	4750 5950 4750 3850
+Wire Notes Line
+	4750 7800 4750 6250
 $EndSCHEMATC

Commit message: - PCB WiP - Pump output aligned
Parts:
- R163, R164, R165, R166, R167, R168, R169, R170, R171, R172: footprint Resistor_SMD:R_0603_1608Metric_Pad1.05x0.95mm_HandSolder -> Resistor_SMD:R_0603_1608Metric
Changed lines of the file:
@@
 F 0 "R164" H 3859 3396 50  0000 L CNN
 F 1 "470R" H 3859 3305 50  0000 L CNN
-F 2 "Resistor_SMD:R_0603_1608Metric_Pad1.05x0.95mm_HandSolder" H 3800 3350 50  0001 C CNN
+F 2 "Resistor_SMD:R_0603_1608Metric" H 3800 3350 50  0001 C CNN
 F 3 "~" H 3800 3350 50  0001 C CNN
 	1    3800 3350
@@
 F 0 "R167" V 3500 4050 50  0000 C BNN
 F 1 "1k" V 3300 4050 50  0000 C TNN
-F 2 "Resistor_SMD:R_0603_1608Metric_Pad1.05x0.95mm_HandSolder" V 3330 4050 50  0001 C CNN
+F 2 "Resistor_SMD:R_0603_1608Metric" V 3330 4050 50  0001 C CNN
 F 3 "~" H 3400 4050 50  0001 C CNN
 	1    3400 4050
@@
 F 0 "R165" H 6359 3546 50  0000 L CNN
 F 1 "470R" H 6359 3455 50  0000 L CNN
-F 2 "Resistor_SMD:R_0603_1608Metric_Pad1.05x0.95mm_HandSolder" H 6300 3500 50  0001 C CNN
+F 2 "Resistor_SMD:R_0603_1608Metric" H 6300 3500 50  0001 C CNN
 F 3 "~" H 6300 3500 50  0001 C CNN
 	1    6300 3500
@@
 F 0 "R169" H 5509 5896 50  0000 L CNN
 F 1 "470R" H 5509 5805 50  0000 L CNN
-F 2 "Resistor_SMD:R_0603_1608Metric_Pad1.05x0.95mm_HandSolder" H 5450 5850 50  0001 C CNN
+F 2 "Resistor_SMD:R_0603_1608Metric" H 5450 5850 50  0001 C CNN
 F 3 "~" H 5450 5850 50  0001 C CNN
 	1    5450 5850
@@
 F 0 "R172" V 5950 6450 50  0000 C BNN
 F 1 "1k" V 5750 6450 50  0000 C TNN
-F 2 "Resistor_SMD:R_0603_1608Metric_Pad1.05x0.95mm_HandSolder" V 5780 6450 50  0001 C CNN
+F 2 "Resistor_SMD:R_0603_1608Metric" V 5780 6450 50  0001 C CNN
 F 3 "~" H 5850 6450 50  0001 C CNN
 	1    5850 6450
@@
 F 0 "R166" V 7050 3700 50  0000 C BNN
 F 1 "0R" V 6850 3700 50  0000 C TNN
-F 2 "Resistor_SMD:R_0603_1608Metric_Pad1.05x0.95mm_HandSolder" V 6880 3700 50  0001 C CNN
+F 2 "Resistor_SMD:R_0603_1608Metric" V 6880 3700 50  0001 C CNN
 F 3 "~" H 6950 3700 50  0001 C CNN
 	1    6950 3700
@@
 F 0 "R163" H 7059 2896 50  0000 L CNN
 F 1 "1k" H 7059 2805 50  0000 L CNN
-F 2 "Resistor_SMD:R_0603_1608Metric_Pad1.05x0.95mm_HandSolder" H 7000 2850 50  0001 C CNN
+F 2 "Resistor_SMD:R_0603_1608Metric" H 7000 2850 50  0001 C CNN
 F 3 "~" H 7000 2850 50  0001 C CNN
 	1    7000 2850
@@
 F 0 "R170" H 3409 5946 50  0000 L CNN
 F 1 "470R" H 3409 5855 50  0000 L CNN
-F 2 "Resistor_SMD:R_0603_1608Metric_Pad1.05x0.95mm_HandSolder" H 3350 5900 50  0001 C CNN
+F 2 "Resistor_SMD:R_0603_1608Metric" H 3350 5900 50  0001 C CNN
 F 3 "~" H 3350 5900 50  0001 C CNN
 	1    3350 5900
@@
 F 0 "R171" V 2750 6100 50  0000 C BNN
 F 1 "0R" V 2550 6100 50  0000 C TNN
-F 2 "Resistor_SMD:R_0603_1608Metric_Pad1.05x0.95mm_HandSolder" V 2580 6100 50  0001 C CNN
+F 2 "Resistor_SMD:R_0603_1608Metric" V 2580 6100 50  0001 C CNN
 F 3 "~" H 2650 6100 50  0001 C CNN
 	1    2650 6100
@@
 F 0 "R168" H 2659 5296 50  0000 L CNN
 F 1 "1k" H 2659 5205 50  0000 L CNN
-F 2 "Resistor_SMD:R_0603_1608Metric_Pad1.05x0.95mm_HandSolder" H 2600 5250 50  0001 C CNN
+F 2 "Resistor_SMD:R_0603_1608Metric" H 2600 5250 50  0001 C CNN
 F 3 "~" H 2600 5250 50  0001 C CNN
 	1    2600 5250
