File: voltmeters.sch (KiCad schematic (older format))
At the start: 27 parts

Commit message: - final schematic
Parts:
- removed C? (x2): 100p, Capacitor_SMD:C_0805_2012Metric_Pad1.15x1.40mm_HandSolder, symbol Device:C_Small
- removed R?: 500M, resistors_moje:MHR0317_0422_0424_0624SA, symbol Device:R
- removed R? (x3): 47k, Resistor_SMD:R_0603_1608Metric_Pad1.05x0.95mm_HandSolder, symbol Device:R_Small
- removed U? (x3): LMC6482, symbol Amplifier_Operational:LMC6482
- added C13, C14, C17, C18, C21, C22: 100n, Capacitor_SMD:C_0603_1608Metric_Pad1.05x0.95mm_HandSolder, symbol Device:C_Small
- added C23, C24: 100p, Capacitor_SMD:C_0805_2012Metric_Pad1.15x1.40mm_HandSolder, symbol Device:C_Small
- added L1, L2, L3, L4, L5, L6: BLM18RK102, Resistor_SMD:R_0805_2012Metric_Pad1.15x1.40mm_HandSolder, symbol Device:L_Core_Ferrite_Small
- added R25: 500M, resistors_moje:MHR0317_0422_0424_0624SA, symbol Device:R
- added R26, R27, R28: 47k, Resistor_SMD:R_0603_1608Metric_Pad1.05x0.95mm_HandSolder, symbol Device:R_Small
- added U11: LMC6482, symbol Amplifier_Operational:LMC6482
- gave numbers to parts that had none: 14
Connections:
- net +5V: now also L5.2; no longer U8.8 (V+), U9.8 (V+)
- net -5V: now also L6.1; no longer U8.4 (V-), U9.4 (V-)
- net GND: now also C21.1, C22.2, U11.3 (+), U11.5 (+); no longer U8.3 (+), U8.5 (+), U9.3 (+), U9.5 (+)
- net U_K renamed U_Extract
- net U_adcK renamed U_adcExtract
- new net: C14.1, L2.2, U8.4 (V-)
- new net: C13.2, L1.1, U8.8 (V+)
- new net: C18.1, L4.2, U9.4 (V-)
- new net: C17.2, L3.1, U9.8 (V+)
- new net: C23.1, R26.2, R27.1, U11.1
- new net: C23.2, R25.2, R26.1, U11.2 (-)
- new net: C24.2, R27.2, R28.1, U11.6 (-)
- new net: C22.1, L6.2, U11.4 (V-)
- new net: C21.2, L5.1, U11.8 (V+)
- new net HV+5V: L1.2, L3.2
- new net HV-5V: L2.1, L4.1
- new net HVGND: C13.1, C14.2, C17.1, C18.2, U8.3 (+), U8.5 (+), U9.3 (+), U9.5 (+)
- new net U_Kathode: R25.1
- new net U_adcKathode: C24.1, R28.2, U11.7
Other:
- note added: "High side:\nmeas U_E and U_F"
- note added: "Low side: meas U_K"
- moved on the sheet: C15, C16, C19, C20, R17, R18, R19, R20, R21, R22, R23, R24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

Commit message: - init PCB - fix last things in schematic
Parts:
- U11, U8, U9: footprint (none) -> miscellaneous_my:SO8-MSOP8_3x3mm_P0.65mm
Changed lines of the file:
@@
 F 0 "U8" H 3900 2017 50  0000 C CNN
 F 1 "LMC6482" H 3900 1926 50  0000 C CNN
-F 2 "" H 3900 1650 50  0001 C CNN
+F 2 "miscellaneous_my:SO8-MSOP8_3x3mm_P0.65mm" H 3900 1650 50  0001 C CNN
 F 3 "http://www.ti.com/lit/ds/symlink/lmc6482.pdf" H 3900 1650 50  0001 C CNN
 	1    3900 1650
@@
 F 0 "U8" H 5000 1917 50  0000 C CNN
 F 1 "LMC6482" H 5000 1826 50  0000 C CNN
-F 2 "" H 5000 1550 50  0001 C CNN
+F 2 "miscellaneous_my:SO8-MSOP8_3x3mm_P0.65mm" H 5000 1550 50  0001 C CNN
 F 3 "http://www.ti.com/lit/ds/symlink/lmc6482.pdf" H 5000 1550 50  0001 C CNN
 	2    5000 1550
@@
 F 0 "U8" H 7058 1646 50  0000 L CNN
 F 1 "LMC6482" H 7058 1555 50  0000 L CNN
-F 2 "" H 7100 1600 50  0001 C CNN
+F 2 "miscellaneous_my:SO8-MSOP8_3x3mm_P0.65mm" H 7100 1600 50  0001 C CNN
 F 3 "http://www.ti.com/lit/ds/symlink/lmc6482.pdf" H 7100 1600 50  0001 C CNN
 	3    7100 1600
@@
 F 0 "U9" H 3900 3317 50  0000 C CNN
 F 1 "LMC6482" H 3900 3226 50  0000 C CNN
-F 2 "" H 3900 2950 50  0001 C CNN
+F 2 "miscellaneous_my:SO8-MSOP8_3x3mm_P0.65mm" H 3900 2950 50  0001 C CNN
 F 3 "http://www.ti.com/lit/ds/symlink/lmc6482.pdf" H 3900 2950 50  0001 C CNN
 	1    3900 2950
@@
 F 0 "U9" H 5000 3217 50  0000 C CNN
 F 1 "LMC6482" H 5000 3126 50  0000 C CNN
-F 2 "" H 5000 2850 50  0001 C CNN
+F 2 "miscellaneous_my:SO8-MSOP8_3x3mm_P0.65mm" H 5000 2850 50  0001 C CNN
 F 3 "http://www.ti.com/lit/ds/symlink/lmc6482.pdf" H 5000 2850 50  0001 C CNN
 	2    5000 2850
@@
 F 0 "U9" H 7008 3046 50  0000 L CNN
 F 1 "LMC6482" H 7008 2955 50  0000 L CNN
-F 2 "" H 7050 3000 50  0001 C CNN
+F 2 "miscellaneous_my:SO8-MSOP8_3x3mm_P0.65mm" H 7050 3000 50  0001 C CNN
 F 3 "http://www.ti.com/lit/ds/symlink/lmc6482.pdf" H 7050 3000 50  0001 C CNN
 	3    7050 3000
@@
 F 0 "U11" H 4100 5867 50  0000 C CNN
 F 1 "LMC6482" H 4100 5776 50  0000 C CNN
-F 2 "" H 4100 5500 50  0001 C CNN
+F 2 "miscellaneous_my:SO8-MSOP8_3x3mm_P0.65mm" H 4100 5500 50  0001 C CNN
 F 3 "http://www.ti.com/lit/ds/symlink/lmc6482.pdf" H 4100 5500 50  0001 C CNN
 	1    4100 5500
@@
 F 0 "U11" H 5000 5867 50  0000 C CNN
 F 1 "LMC6482" H 5000 5776 50  0000 C CNN
-F 2 "" H 5000 5500 50  0001 C CNN
+F 2 "miscellaneous_my:SO8-MSOP8_3x3mm_P0.65mm" H 5000 5500 50  0001 C CNN
 F 3 "http://www.ti.com/lit/ds/symlink/lmc6482.pdf" H 5000 5500 50  0001 C CNN
 	2    5000 5500
@@
 F 0 "U11" H 7158 5696 50  0000 L CNN
 F 1 "LMC6482" H 7158 5605 50  0000 L CNN
-F 2 "" H 7200 5650 50  0001 C CNN
+F 2 "miscellaneous_my:SO8-MSOP8_3x3mm_P0.65mm" H 7200 5650 50  0001 C CNN
 F 3 "http://www.ti.com/lit/ds/symlink/lmc6482.pdf" H 7200 5650 50  0001 C CNN
 	3    7200 5650
@@
 Text HLabel 5400 5500 2    50   Output ~ 0
 U_adcKathode
+$Comp
+L power:PWR_FLAG #FLG01
+U 1 1 5FA4F000
+P 6850 1300
+F 0 "#FLG01" H 6850 1375 50  0001 C CNN
+F 1 "PWR_FLAG" H 6850 1474 50  0001 C CNN
+F 2 "" H 6850 1300 50  0001 C CNN
+F 3 "~" H 6850 1300 50  0001 C CNN
+	1    6850 1300
+	1    0    0    -1
+$EndComp
+Connection ~ 6850 1300
+$Comp
+L power:PWR_FLAG #FLG02
+U 1 1 5FA4F292
+P 6850 1900
+F 0 "#FLG02" H 6850 1975 50  0001 C CNN
+F 1 "PWR_FLAG" H 6850 2074 50  0001 C CNN
+F 2 "" H 6850 1900 50  0001 C CNN
+F 3 "~" H 6850 1900 50  0001 C CNN
+	1    6850 1900
+	-1   0    0    1
+$EndComp
+Connection ~ 6850 1900
+$Comp
+L power:PWR_FLAG #FLG03
+U 1 1 5FA4F3D5
+P 6800 2700
+F 0 "#FLG03" H 6800 2775 50  0001 C CNN
+F 1 "PWR_FLAG" H 6800 2874 50  0001 C CNN
+F 2 "" H 6800 2700 50  0001 C CNN
+F 3 "~" H 6800 2700 50  0001 C CNN
+	1    6800 2700
+	1    0    0    -1
+$EndComp
+Connection ~ 6800 2700
+$Comp
+L power:PWR_FLAG #FLG05
+U 1 1 5FA4F677
+P 6950 5350
+F 0 "#FLG05" H 6950 5425 50  0001 C CNN
+F 1 "PWR_FLAG" H 6950 5524 50  0001 C CNN
+F 2 "" H 6950 5350 50  0001 C CNN
+F 3 "~" H 6950 5350 50  0001 C CNN
+	1    6950 5350
+	1    0    0    -1
+$EndComp
+Connection ~ 6950 5350
+$Comp
+L power:PWR_FLAG #FLG04
+U 1 1 5FA4FB89
+P 6800 3300
+F 0 "#FLG04" H 6800 3375 50  0001 C CNN
+F 1 "PWR_FLAG" H 6800 3474 50  0001 C CNN
+F 2 "" H 6800 3300 50  0001 C CNN
+F 3 "~" H 6800 3300 50  0001 C CNN
+	1    6800 3300
+	-1   0    0    1
+$EndComp
+Connection ~ 6800 3300
+$Comp
+L power:PWR_FLAG #FLG06
+U 1 1 5FA4FE2B
+P 6950 5950
+F 0 "#FLG06" H 6950 6025 50  0001 C CNN
+F 1 "PWR_FLAG" H 6950 6124 50  0001 C CNN
+F 2 "" H 6950 5950 50  0001 C CNN
+F 3 "~" H 6950 5950 50  0001 C CNN
+	1    6950 5950
+	-1   0    0    1
+$EndComp
+Connection ~ 6950 5950
 $EndSCHEMATC

Commit message: - PCB progress
Parts:
- C13, C14, C17, C18, C21, C22: footprint Capacitor_SMD:C_0603_1608Metric_Pad1.05x0.95mm_HandSolder -> Capacitor_SMD:C_0603_1608Metric
- C15, C16, C19, C20, C23, C24: footprint Capacitor_SMD:C_0805_2012Metric_Pad1.15x1.40mm_HandSolder -> Capacitor_SMD:C_0603_1608Metric
- L1, L2, L3, L4, L5, L6: footprint Resistor_SMD:R_0805_2012Metric_Pad1.15x1.40mm_HandSolder -> Inductor_SMD:L_0603_1608Metric
- R18, R19, R20, R22, R23, R24, R26, R27, R28: footprint Resistor_SMD:R_0603_1608Metric_Pad1.05x0.95mm_HandSolder -> Resistor_SMD:R_0603_1608Metric
Changed lines of the file:
@@
 F 0 "C15" V 3950 2150 50  0000 R CNN
 F 1 "100p" V 3950 2250 50  0000 L CNN
-F 2 "Capacitor_SMD:C_0805_2012Metric_Pad1.15x1.40mm_HandSolder" H 3900 2200 50  0001 C CNN
+F 2 "Capacitor_SMD:C_0603_1608Metric" H 3900 2200 50  0001 C CNN
 F 3 "~" H 3900 2200 50  0001 C CNN
 	1    3900 2200
@@
 F 0 "C16" V 5050 2150 50  0000 R CNN
 F 1 "100p" V 5050 2250 50  0000 L CNN
-F 2 "Capacitor_SMD:C_0805_2012Metric_Pad1.15x1.40mm_HandSolder" H 5000 2200 50  0001 C CNN
+F 2 "Capacitor_SMD:C_0603_1608Metric" H 5000 2200 50  0001 C CNN
 F 3 "~" H 5000 2200 50  0001 C CNN
 	1    5000 2200
@@
 F 0 "C20" V 5050 3450 50  0000 R CNN
 F 1 "100p" V 5050 3550 50  0000 L CNN
-F 2 "Capacitor_SMD:C_0805_2012Metric_Pad1.15x1.40mm_HandSolder" H 5000 3500 50  0001 C CNN
+F 2 "Capacitor_SMD:C_0603_1608Metric" H 5000 3500 50  0001 C CNN
 F 3 "~" H 5000 3500 50  0001 C CNN
 	1    5000 3500
@@
 F 0 "C19" V 3950 3450 50  0000 R CNN
 F 1 "100p" V 3950 3550 50  0000 L CNN
-F 2 "Capacitor_SMD:C_0805_2012Metric_Pad1.15x1.40mm_HandSolder" H 3900 3500 50  0001 C CNN
+F 2 "Capacitor_SMD:C_0603_1608Metric" H 3900 3500 50  0001 C CNN
 F 3 "~" H 3900 3500 50  0001 C CNN
 	1    3900 3500
@@
 F 0 "R18" V 4000 1950 50  0000 C CNN
 F 1 "47k" V 3800 1950 50  0000 C CNN
-F 2 "Resistor_SMD:R_0603_1608Metric_Pad1.05x0.95mm_HandSolder" V 3830 1950 50  0001 C CNN
+F 2 "Resistor_SMD:R_0603_1608Metric" V 3830 1950 50  0001 C CNN
 F 3 "~" H 3900 1950 50  0001 C CNN
 	1    3900 1950
@@
 F 0 "R19" V 4550 1950 50  0000 C CNN
 F 1 "47k" V 4350 1950 50  0000 C CNN
-F 2 "Resistor_SMD:R_0603_1608Metric_Pad1.05x0.95mm_HandSolder" V 4380 1950 50  0001 C CNN
+F 2 "Resistor_SMD:R_0603_1608Metric" V 4380 1950 50  0001 C CNN
 F 3 "~" H 4450 1950 50  0001 C CNN
 	1    4450 1950
@@
 F 0 "R20" V 5100 1950 50  0000 C CNN
 F 1 "47k" V 4900 1950 50  0000 C CNN
-F 2 "Resistor_SMD:R_0603_1608Metric_Pad1.05x0.95mm_HandSolder" V 4930 1950 50  0001 C CNN
+F 2 "Resistor_SMD:R_0603_1608Metric" V 4930 1950 50  0001 C CNN
 F 3 "~" H 5000 1950 50  0001 C CNN
 	1    5000 1950
@@
 F 0 "R22" V 4000 3250 50  0000 C CNN
 F 1 "47k" V 3800 3250 50  0000 C CNN
-F 2 "Resistor_SMD:R_0603_1608Metric_Pad1.05x0.95mm_HandSolder" V 3830 3250 50  0001 C CNN
+F 2 "Resistor_SMD:R_0603_1608Metric" V 3830 3250 50  0001 C CNN
 F 3 "~" H 3900 3250 50  0001 C CNN
 	1    3900 3250
@@
 F 0 "R23" V 4550 3250 50  0000 C CNN
 F 1 "47k" V 4350 3250 50  0000 C CNN
-F 2 "Resistor_SMD:R_0603_1608Metric_Pad1.05x0.95mm_HandSolder" V 4380 3250 50  0001 C CNN
+F 2 "Resistor_SMD:R_0603_1608Metric" V 4380 3250 50  0001 C CNN
 F 3 "~" H 4450 3250 50  0001 C CNN
 	1    4450 3250
@@
 F 0 "R24" V 5100 3250 50  0000 C CNN
 F 1 "47k" V 4900 3250 50  0000 C CNN
-F 2 "Resistor_SMD:R_0603_1608Metric_Pad1.05x0.95mm_HandSolder" V 4930 3250 50  0001 C CNN
+F 2 "Resistor_SMD:R_0603_1608Metric" V 4930 3250 50  0001 C CNN
 F 3 "~" H 5000 3250 50  0001 C CNN
 	1    5000 3250
@@
 F 0 "C13" H 6900 1450 50  0000 L BNN
 F 1 "100n" H 6900 1350 50  0000 L TNN
-F 2 "Capacitor_SMD:C_0603_1608Metric_Pad1.05x0.95mm_HandSolder" H 6850 1400 50  0001 C CNN
+F 2 "Capacitor_SMD:C_0603_1608Metric" H 6850 1400 50  0001 C CNN
 F 3 "~" H 6850 1400 50  0001 C CNN
 	1    6850 1400
@@
 F 0 "L1" V 7455 1300 50  0000 C CNN
 F 1 "BLM18RK102" V 7364 1300 50  0000 C CNN
-F 2 "Resistor_SMD:R_0805_2012Metric_Pad1.15x1.40mm_HandSolder" H 7250 1300 50  0001 C CNN
+F 2 "Inductor_SMD:L_0603_1608Metric" H 7250 1300 50  0001 C CNN
 F 3 "~" H 7250 1300 50  0001 C CNN
 	1    7250 1300
@@
 F 0 "C14" H 6900 1850 50  0000 L BNN
 F 1 "100n" H 6900 1750 50  0000 L TNN
-F 2 "Capacitor_SMD:C_0603_1608Metric_Pad1.05x0.95mm_HandSolder" H 6850 1800 50  0001 C CNN
+F 2 "Capacitor_SMD:C_0603_1608Metric" H 6850 1800 50  0001 C CNN
 F 3 "~" H 6850 1800 50  0001 C CNN
 	1    6850 1800
@@
 F 0 "L2" V 7455 1900 50  0000 C CNN
 F 1 "BLM18RK102" V 7364 1900 50  0000 C CNN
-F 2 "Resistor_SMD:R_0805_2012Metric_Pad1.15x1.40mm_HandSolder" H 7250 1900 50  0001 C CNN
+F 2 "Inductor_SMD:L_0603_1608Metric" H 7250 1900 50  0001 C CNN
 F 3 "~" H 7250 1900 50  0001 C CNN
 	1    7250 1900
@@
 F 0 "C17" H 6850 2850 50  0000 L BNN
 F 1 "100n" H 6850 2750 50  0000 L TNN
-F 2 "Capacitor_SMD:C_0603_1608Metric_Pad1.05x0.95mm_HandSolder" H 6800 2800 50  0001 C CNN
+F 2 "Capacitor_SMD:C_0603_1608Metric" H 6800 2800 50  0001 C CNN
 F 3 "~" H 6800 2800 50  0001 C CNN
 	1    6800 2800
@@
 F 0 "L3" V 7405 2700 50  0000 C CNN
 F 1 "BLM18RK102" V 7314 2700 50  0000 C CNN
-F 2 "Resistor_SMD:R_0805_2012Metric_Pad1.15x1.40mm_HandSolder" H 7200 2700 50  0001 C CNN
+F 2 "Inductor_SMD:L_0603_1608Metric" H 7200 2700 50  0001 C CNN
 F 3 "~" H 7200 2700 50  0001 C CNN
 	1    7200 2700
@@
 F 0 "C18" H 6850 3250 50  0000 L BNN
 F 1 "100n" H 6850 3150 50  0000 L TNN
-F 2 "Capacitor_SMD:C_0603_1608Metric_Pad1.05x0.95mm_HandSolder" H 6800 3200 50  0001 C CNN
+F 2 "Capacitor_SMD:C_0603_1608Metric" H 6800 3200 50  0001 C CNN
 F 3 "~" H 6800 3200 50  0001 C CNN
 	1    6800 3200
@@
 F 0 "L4" V 7405 3300 50  0000 C CNN
 F 1 "BLM18RK102" V 7314 3300 50  0000 C CNN
-F 2 "Resistor_SMD:R_0805_2012Metric_Pad1.15x1.40mm_HandSolder" H 7200 3300 50  0001 C CNN
+F 2 "Inductor_SMD:L_0603_1608Metric" H 7200 3300 50  0001 C CNN
 F 3 "~" H 7200 3300 50  0001 C CNN
 	1    7200 3300
@@
 F 0 "C23" V 4150 6000 50  0000 R CNN
 F 1 "100p" V 4150 6100 50  0000 L CNN
-F 2 "Capacitor_SMD:C_0805_2012Metric_Pad1.15x1.40mm_HandSolder" H 4100 6050 50  0001 C CNN
+F 2 "Capacitor_SMD:C_0603_1608Metric" H 4100 6050 50  0001 C CNN
 F 3 "~" H 4100 6050 50  0001 C CNN
 	1    4100 6050
@@
 F 0 "C24" V 5050 6000 50  0000 R CNN
 F 1 "100p" V 5050 6100 50  0000 L CNN
-F 2 "Capacitor_SMD:C_0805_2012Metric_Pad1.15x1.40mm_HandSolder" H 5000 6050 50  0001 C CNN
+F 2 "Capacitor_SMD:C_0603_1608Metric" H 5000 6050 50  0001 C CNN
 F 3 "~" H 5000 6050 50  0001 C CNN
 	1    5000 6050
@@
 F 0 "R26" V 4200 5800 50  0000 C CNN
 F 1 "47k" V 4000 5800 50  0000 C CNN
-F 2 "Resistor_SMD:R_0603_1608Metric_Pad1.05x0.95mm_HandSolder" V 4030 5800 50  0001 C CNN
+F 2 "Resistor_SMD:R_0603_1608Metric" V 4030 5800 50  0001 C CNN
 F 3 "~" H 4100 5800 50  0001 C CNN
 	1    4100 5800
@@
 F 0 "R27" V 4650 5800 50  0000 C CNN
 F 1 "47k" V 4450 5800 50  0000 C CNN
-F 2 "Resistor_SMD:R_0603_1608Metric_Pad1.05x0.95mm_HandSolder" V 4480 5800 50  0001 C CNN
+F 2 "Resistor_SMD:R_0603_1608Metric" V 4480 5800 50  0001 C CNN
 F 3 "~" H 4550 5800 50  0001 C CNN
 	1    4550 5800
@@
 F 0 "R28" V 5100 5800 50  0000 C CNN
 F 1 "47k" V 4900 5800 50  0000 C CNN
-F 2 "Resistor_SMD:R_0603_1608Metric_Pad1.05x0.95mm_HandSolder" V 4930 5800 50  0001 C CNN
+F 2 "Resistor_SMD:R_0603_1608Metric" V 4930 5800 50  0001 C CNN
 F 3 "~" H 5000 5800 50  0001 C CNN
 	1    5000 5800
@@
 F 0 "C21" H 7000 5500 50  0000 L BNN
 F 1 "100n" H 7000 5400 50  0000 L TNN
-F 2 "Capacitor_SMD:C_0603_1608Metric_Pad1.05x0.95mm_HandSolder" H 6950 5450 50  0001 C CNN
+F 2 "Capacitor_SMD:C_0603_1608Metric" H 6950 5450 50  0001 C CNN
 F 3 "~" H 6950 5450 50  0001 C CNN
 	1    6950 5450
@@
 F 0 "L5" V 7555 5350 50  0000 C CNN
 F 1 "BLM18RK102" V 7464 5350 50  0000 C CNN
-F 2 "Resistor_SMD:R_0805_2012Metric_Pad1.15x1.40mm_HandSolder" H 7350 5350 50  0001 C CNN
+F 2 "Inductor_SMD:L_0603_1608Metric" H 7350 5350 50  0001 C CNN
 F 3 "~" H 7350 5350 50  0001 C CNN
 	1    7350 5350
@@
 F 0 "C22" H 7000 5900 50  0000 L BNN
 F 1 "100n" H 7000 5800 50  0000 L TNN
-F 2 "Capacitor_SMD:C_0603_1608Metric_Pad1.05x0.95mm_HandSolder" H 6950 5850 50  0001 C CNN
+F 2 "Capacitor_SMD:C_0603_1608Metric" H 6950 5850 50  0001 C CNN
 F 3 "~" H 6950 5850 50  0001 C CNN
 	1    6950 5850
@@
 F 0 "L6" V 7555 5950 50  0000 C CNN
 F 1 "BLM18RK102" V 7464 5950 50  0000 C CNN
-F 2 "Resistor_SMD:R_0805_2012Metric_Pad1.15x1.40mm_HandSolder" H 7350 5950 50  0001 C CNN
+F 2 "Inductor_SMD:L_0603_1608Metric" H 7350 5950 50  0001 C CNN
 F 3 "~" H 7350 5950 50  0001 C CNN
 	1    7350 5950
